Commit message: add grid heightmap

File: src/mr2_rover_description/urdf/rover_base.xacro (robot description, xacro)
@@ -89,5 +89,5 @@
     <link name="front_camera"/>
     <joint name="base_to_front_camera" type="fixed">
-	    <origin xyz="${length/2.0} 0 0" rpy="0 ${front_camera_pitch} 0"/>
+	    <origin xyz="${length/2.0} 0 ${height}" rpy="0 ${front_camera_pitch} 0"/>
       <parent link="base_link"/>
       <child link="front_camera"/>
