Commit message: attempt to add gnss

File: src/mr2_rover_description/urdf/rover.urdf.xacro (robot description, xacro)
@@ -18,4 +18,13 @@
     <parameters>$(find mr2_rover_description)/config/controllers.yaml</parameters>
   </plugin>
+</gazebo>
+<gazebo reference="base_link">
+  <sensor name="left_gnss_sensor" type="navsat">
+    <always_on>1</always_on>
+    <update_rate>1</update_rate>
+    <visualize>true</visualize>
+            <topic>left_gnss/fix</topic>
+            <ignition_frame_id>base_link</ignition_frame_id>
+  </sensor>
 </gazebo>
       <ros2_control name="GazeboSimSystem" type="system">
@@ -42,8 +51,8 @@
         <joint name="rr_steering_joint"><command_interface name="position"/><state_interface name="position"/></joint>
         <!-- Wheel velocity interfaces -->
-        <joint name="fl_wheel_joint"><command_interface name="velocity"/><state_interface name="velocity"/></joint>
-        <joint name="fr_wheel_joint"><command_interface name="velocity"/><state_interface name="velocity"/></joint>
-        <joint name="rl_wheel_joint"><command_interface name="velocity"/><state_interface name="velocity"/></joint>
-        <joint name="rr_wheel_joint"><command_interface name="velocity"/><state_interface name="velocity"/></joint>
+        <joint name="fl_wheel_joint"><command_interface name="velocity"/><state_interface name="velocity"/><state_interface name="position"/></joint>
+        <joint name="fr_wheel_joint"><command_interface name="velocity"/><state_interface name="velocity"/><state_interface name="position"/></joint>
+        <joint name="rl_wheel_joint"><command_interface name="velocity"/><state_interface name="velocity"/><state_interface name="position"/></joint>
+        <joint name="rr_wheel_joint"><command_interface name="velocity"/><state_interface name="velocity"/><state_interface name="position"/></joint>
       </ros2_control>
 </robot>

File: src/mr2_rover_description/urdf/rover_base.xacro (robot description, xacro)
@@ -72,5 +72,12 @@
       <dynamics damping="0.1" friction="0.0"/>
       <limit lower="-${joint_lim}" upper="${joint_lim}" effort="${joint_effort}" velocity="${joint_vel}"/>
+      <mimic joint="left_rocker_joint" multiplier="-1" offset="0"/>
     </joint>
+    <link name="left_gnss"/>
+    <joint name="base_to_sensor" type="fixed">
+	    <origin xyz="0 ${-width/2.0} 0" rpy="0 0 0"/>
+  <parent link="base_link"/>
+  <child  link="left_gnss"/>
+</joint>
   </xacro:macro>
 </robot>

Commit message: add rgbd camera

File: src/mr2_rover_description/urdf/rover.urdf.xacro (robot description, xacro)
@@ -13,46 +13,135 @@
   <!-- ros2_control plugin -->
   <gazebo>
-	  <plugin filename="gz_ros2_control-system" name="gz_ros2_control::GazeboSimROS2ControlPlugin">
-	  <robot_param>robot_description</robot_param>
-	  <robot_param_node>robot_state_publisher</robot_param_node>
-    <parameters>$(find mr2_rover_description)/config/controllers.yaml</parameters>
-  </plugin>
-</gazebo>
-<gazebo reference="base_link">
-  <sensor name="left_gnss_sensor" type="navsat">
-    <always_on>1</always_on>
-    <update_rate>1</update_rate>
-    <visualize>true</visualize>
-            <topic>left_gnss/fix</topic>
-            <ignition_frame_id>base_link</ignition_frame_id>
-  </sensor>
-</gazebo>
-      <ros2_control name="GazeboSimSystem" type="system">
-        <hardware>
-          <plugin>gz_ros2_control/GazeboSimSystem</plugin>
-        </hardware>
-	<!-- Mimic Joint -->
-	<joint name="left_rocker_joint">
-	  <state_interface name="position"/>
-	  <state_interface name="velocity"/>
-	  <state_interface name="effort"/>
-	</joint>
-	<joint name="right_rocker_joint">
-	  <param name="mimic">left_rocker_joint</param>
-	  <param name="multiplier">-1</param>
-	  <state_interface name="position"/>
-	  <state_interface name="velocity"/>
-	  <state_interface name="effort"/>
-	</joint>
-        <!-- Steering position interfaces -->
-        <joint name="fl_steering_joint"><command_interface name="position"/><state_interface name="position"/></joint>
-        <joint name="fr_steering_joint"><command_interface name="position"/><state_interface name="position"/></joint>
-        <joint name="rl_steering_joint"><command_interface name="position"/><state_interface name="position"/></joint>
-        <joint name="rr_steering_joint"><command_interface name="position"/><state_interface name="position"/></joint>
-        <!-- Wheel velocity interfaces -->
-        <joint name="fl_wheel_joint"><command_interface name="velocity"/><state_interface name="velocity"/><state_interface name="position"/></joint>
-        <joint name="fr_wheel_joint"><command_interface name="velocity"/><state_interface name="velocity"/><state_interface name="position"/></joint>
-        <joint name="rl_wheel_joint"><command_interface name="velocity"/><state_interface name="velocity"/><state_interface name="position"/></joint>
-        <joint name="rr_wheel_joint"><command_interface name="velocity"/><state_interface name="velocity"/><state_interface name="position"/></joint>
-      </ros2_control>
+    <plugin filename="gz_ros2_control-system" name="gz_ros2_control::GazeboSimROS2ControlPlugin">
+      <robot_param>robot_description</robot_param>
+      <robot_param_node>robot_state_publisher</robot_param_node>
+      <parameters>$(find mr2_rover_description)/config/controllers.yaml</parameters>
+    </plugin>
+  </gazebo>
+  <gazebo reference="left_gnss">
+    <sensor name="left_gnss_sensor" type="navsat">
+      <always_on>1</always_on>
+      <update_rate>1</update_rate>
+      <visualize>true</visualize>
+      <topic>left_gnss/navsat</topic>
+      <ignition_frame_id>left_gnss</ignition_frame_id>
+    </sensor>
+  </gazebo>
+  <gazebo reference="right_gnss">
+    <sensor name="right_gnss_sensor" type="navsat">
+      <always_on>1</always_on>
+      <update_rate>1</update_rate>
+      <visualize>true</visualize>
+      <topic>right_gnss/navsat</topic>
+      <ignition_frame_id>right_gnss</ignition_frame_id>
+    </sensor>
+  </gazebo>
+  <gazebo reference="front_camera">
+    <sensor name="front_camera_sensor" type="rgbd_camera">
+	<update_rate>60</update_rate>
+	<always_on>1</always_on>
+        <visualize>true</visualize>
+	<topic>rgbd_camera</topic>
+        <ignition_frame_id>front_camera</ignition_frame_id>
+        <camera>
+          <horizontal_fov>1.0472</horizontal_fov>
+          <lens>
+            <intrinsics>
+              <!-- fx = fy = width / ( 2 * tan (hfov / 2 ) ) -->
+              <fx>554.25469</fx>
+              <fy>554.25469</fy>
+              <!-- cx = ( width + 1 ) / 2 -->
+              <cx>320.5</cx>
+              <!-- cy = ( height + 1 ) / 2 -->
+              <cy>240.5</cy>
+              <s>0</s>
+            </intrinsics>
+          </lens>
+          <distortion>
+            <k1>0.0</k1>
+            <k2>0.0</k2>
+            <k3>0.0</k3>
+            <p1>0.0</p1>
+            <p2>0.0</p2>
+            <center>0.5 0.5</center>
+          </distortion>
+          <image>
+            <width>640</width>
+            <height>480</height>
+            <format>R8G8B8</format>
+          </image>
+          <clip>
+            <near>0.01</near>
+            <far>300</far>
+          </clip>
+          <depth_camera>
+            <clip>
+              <near>0.1</near>
+              <far>10</far>
+            </clip>
+          </depth_camera>
+          <noise>
+            <type>gaussian</type>
+            <mean>0</mean>
+            <stddev>0.007</stddev>
+          </noise>
+        </camera>
+    </sensor>
+  </gazebo>
+  <ros2_control name="GazeboSimSystem" type="system">
+    <hardware>
+      <plugin>gz_ros2_control/GazeboSimSystem</plugin>
+    </hardware>
+    <!-- Mimic Joint -->
+    <joint name="left_rocker_joint">
+      <state_interface name="position"/>
+      <state_interface name="velocity"/>
+      <state_interface name="effort"/>
+    </joint>
+    <joint name="right_rocker_joint">
+      <param name="mimic">left_rocker_joint</param>
+      <param name="multiplier">-1</param>
+      <state_interface name="position"/>
+      <state_interface name="velocity"/>
+      <state_interface name="effort"/>
+    </joint>
+    <!-- Steering position interfaces -->
+    <joint name="fl_steering_joint">
+      <command_interface name="position"/>
+      <state_interface name="position"/>
+    </joint>
+    <joint name="fr_steering_joint">
+      <command_interface name="position"/>
+      <state_interface name="position"/>
+    </joint>
+    <joint name="rl_steering_joint">
+      <command_interface name="position"/>
+      <state_interface name="position"/>
+    </joint>
+    <joint name="rr_steering_joint">
+      <command_interface name="position"/>
+      <state_interface name="position"/>
+    </joint>
+    <!-- Wheel velocity interfaces -->
+    <joint name="fl_wheel_joint">
+      <command_interface name="velocity"/>
+      <state_interface name="velocity"/>
+      <state_interface name="position"/>
+    </joint>
+    <joint name="fr_wheel_joint">
+      <command_interface name="velocity"/>
+      <state_interface name="velocity"/>
+      <state_interface name="position"/>
+    </joint>
+    <joint name="rl_wheel_joint">
+      <command_interface name="velocity"/>
+      <state_interface name="velocity"/>
+      <state_interface name="position"/>
+    </joint>
+    <joint name="rr_wheel_joint">
+      <command_interface name="velocity"/>
+      <state_interface name="velocity"/>
+      <state_interface name="position"/>
+    </joint>
+  </ros2_control>
 </robot>

File: src/mr2_rover_description/urdf/rover_base.xacro (robot description, xacro)
@@ -1,39 +1,39 @@
 <?xml version="1.0"?>
 <robot xmlns:xacro="http://www.ros.org/wiki/xacro">
-  <xacro:macro name="rover_base"
-               params="length:=0.73 width:=0.49 height:=0.19 mass:=10 rocker_size:=0.1 rocker_mass:=0.5 joint_effort:=50 joint_vel:=2.0 joint_lim:=1.57">
-    <!-- ===== Base ===== -->
+  <xacro:macro name="rover_base" params="length:=0.73 width:=0.49 height:=0.19 mass:=10 rocker_size:=0.1 rocker_mass:=0.5 joint_effort:=50 joint_vel:=2.0 joint_lim:=1.57 front_camera_pitch:=0.3491">
     <link name="base_link">
       <inertial>
         <mass value="${mass}"/>
-        <inertia ixx="${mass*(width*width + height*height)/12.0}"
-                 iyy="${mass*(length*length + height*height)/12.0}"
-                 izz="${mass*(length*length + width*width)/12.0}"
-                 ixy="0" ixz="0" iyz="0"/>
+        <inertia ixx="${mass*(width*width + height*height)/12.0}" iyy="${mass*(length*length + height*height)/12.0}" izz="${mass*(length*length + width*width)/12.0}" ixy="0" ixz="0" iyz="0"/>
       </inertial>
       <visual>
-        <geometry><box size="${length} ${width} ${height}"/></geometry>
+        <geometry>
+          <box size="${length} ${width} ${height}"/>
+        </geometry>
         <origin xyz="0 0 ${height/2.0}"/>
       </visual>
       <collision>
-        <geometry><box size="${length} ${width} ${height}"/></geometry>
+        <geometry>
+          <box size="${length} ${width} ${height}"/>
+        </geometry>
         <origin xyz="0 0 ${height/2.0}"/>
       </collision>
     </link>
-    <!-- ===== Left rocker ===== -->
     <link name="left_rocker">
       <inertial>
         <origin xyz="0 -${width/2.0} 0"/>
         <mass value="${rocker_mass}"/>
-        <inertia ixx="1e-3" ixy="0" ixz="0"
-                 iyy="1e-3" iyz="0"
-                 izz="1e-3"/>
+        <inertia ixx="1e-3" ixy="0" ixz="0" iyy="1e-3" iyz="0" izz="1e-3"/>
       </inertial>
       <visual>
-        <geometry><box size="${rocker_size} ${rocker_size} ${rocker_size}"/></geometry>
+        <geometry>
+          <box size="${rocker_size} ${rocker_size} ${rocker_size}"/>
+        </geometry>
         <origin xyz="0 0 ${rocker_size/2.0}"/>
       </visual>
       <collision>
-        <geometry><box size="${rocker_size} ${rocker_size} ${rocker_size}"/></geometry>
+        <geometry>
+          <box size="${rocker_size} ${rocker_size} ${rocker_size}"/>
+        </geometry>
         <origin xyz="0 0 ${rocker_size/2.0}"/>
       </collision>
@@ -41,5 +41,5 @@
     <joint name="left_rocker_joint" type="revolute">
       <parent link="base_link"/>
-      <child  link="left_rocker"/>
+      <child link="left_rocker"/>
       <origin xyz="0 -${width/2.0} 0" rpy="0 0 0"/>
       <axis xyz="0 1 0"/>
@@ -47,19 +47,20 @@
       <limit lower="-${joint_lim}" upper="${joint_lim}" effort="${joint_effort}" velocity="${joint_vel}"/>
     </joint>
-    <!-- ===== Right rocker ===== -->
     <link name="right_rocker">
       <inertial>
         <origin xyz="0 ${width/2.0} 0"/>
         <mass value="${rocker_mass}"/>
-        <inertia ixx="1e-3" ixy="0" ixz="0"
-                 iyy="1e-3" iyz="0"
-                 izz="1e-3"/>
+        <inertia ixx="1e-3" ixy="0" ixz="0" iyy="1e-3" iyz="0" izz="1e-3"/>
       </inertial>
       <visual>
-        <geometry><box size="${rocker_size} ${rocker_size} ${rocker_size}"/></geometry>
+        <geometry>
+          <box size="${rocker_size} ${rocker_size} ${rocker_size}"/>
+        </geometry>
         <origin xyz="0 0 ${rocker_size/2.0}"/>
       </visual>
       <collision>
-        <geometry><box size="${rocker_size} ${rocker_size} ${rocker_size}"/></geometry>
+        <geometry>
+          <box size="${rocker_size} ${rocker_size} ${rocker_size}"/>
+        </geometry>
         <origin xyz="0 0 ${rocker_size/2.0}"/>
       </collision>
@@ -67,5 +68,5 @@
     <joint name="right_rocker_joint" type="revolute">
       <parent link="base_link"/>
-      <child  link="right_rocker"/>
+      <child link="right_rocker"/>
       <origin xyz="0 ${width/2.0} 0" rpy="0 0 0"/>
       <axis xyz="0 1 0"/>
@@ -75,9 +76,21 @@
     </joint>
     <link name="left_gnss"/>
-    <joint name="base_to_sensor" type="fixed">
-	    <origin xyz="0 ${-width/2.0} 0" rpy="0 0 0"/>
-  <parent link="base_link"/>
-  <child  link="left_gnss"/>
-</joint>
+    <joint name="base_to_left_gnss" type="fixed">
+      <origin xyz="0 ${-width/2.0} 0" rpy="0 0 0"/>
+      <parent link="base_link"/>
+      <child link="left_gnss"/>
+    </joint>
+    <link name="right_gnss"/>
+    <joint name="base_to_right_gnss" type="fixed">
+      <origin xyz="0 ${width/2.0} 0" rpy="0 0 0"/>
+      <parent link="base_link"/>
+      <child link="right_gnss"/>
+    </joint>
+    <link name="front_camera"/>
+    <joint name="base_to_front_camera" type="fixed">
+	    <origin xyz="${length/2.0} 0 0" rpy="0 ${front_camera_pitch} 0"/>
+      <parent link="base_link"/>
+      <child link="front_camera"/>
+    </joint>
   </xacro:macro>
 </robot>

File: src/mr2_rover_description/urdf/swerve_module.xacro (robot description, xacro)
@@ -3,15 +3,13 @@
   <xacro:macro name="swerve_module" params="prefix parent xyz">
     <!-- local constants -->
-    <xacro:property name="steer_limit"  value="3.14"/>
-    <xacro:property name="wheel_limit"  value="20.0"/>
+    <xacro:property name="steer_limit" value="3.14"/>
+    <xacro:property name="wheel_limit" value="20.0"/>
     <xacro:property name="wheel_radius" value="0.11"/>
-    <xacro:property name="wheel_width"  value="0.11"/>
+    <xacro:property name="wheel_width" value="0.11"/>
     <!-- Steering link -->
     <link name="${prefix}_mount">
       <inertial>
         <mass value="0.5"/>
-	<inertia ixx="1e-3" ixy="0"  ixz="0"
-            iyy="1e-3" iyz="0"
-            izz="1e-3"/>
+        <inertia ixx="1e-3" ixy="0" ixz="0" iyy="1e-3" iyz="0" izz="1e-3"/>
       </inertial>
       <visual>
@@ -28,28 +26,26 @@
     <!-- Wheel link -->
     <link name="${prefix}_wheel">
-<inertial>
-	    <mass value="0.2"/>
-	    <inertia ixx="1e-3" ixy="0" ixz="0"
-		     iyy="1e-3" iyz="0"
-		     izz="1e-3"/>
-	  </inertial>
-	  <visual>
-	    <origin xyz="0 0 0" rpy="1.5708 0 0"/> <!-- Z축->X축으로 눕힘 -->
-	    <geometry>
-	      <cylinder radius="${wheel_radius}" length="${wheel_width}"/>
-	    </geometry>
-	    <material name="Rubber"/>
-	  </visual>
-	  <collision>
-	    <origin xyz="0 0 0" rpy="1.5708 0 0"/> <!-- 동일하게 적용 -->
-	    <geometry>
-	      <cylinder radius="${wheel_radius}" length="${wheel_width}"/>
-	    </geometry>
-	  </collision>
-	</link>
+      <inertial>
+        <mass value="0.2"/>
+        <inertia ixx="1e-3" ixy="0" ixz="0" iyy="1e-3" iyz="0" izz="1e-3"/>
+      </inertial>
+      <visual>
+        <origin xyz="0 0 0" rpy="1.5708 0 0"/>
+        <geometry>
+          <cylinder radius="${wheel_radius}" length="${wheel_width}"/>
+        </geometry>
+        <material name="Rubber"/>
+      </visual>
+      <collision>
+        <origin xyz="0 0 0" rpy="1.5708 0 0"/>
+        <geometry>
+          <cylinder radius="${wheel_radius}" length="${wheel_width}"/>
+        </geometry>
+      </collision>
+    </link>
     <!-- Steering joint -->
     <joint name="${prefix}_steering_joint" type="continuous">
       <parent link="${parent}"/>
-      <child  link="${prefix}_mount"/>
+      <child link="${prefix}_mount"/>
       <origin xyz="${xyz}" rpy="0 0 0"/>
       <axis xyz="0 0 1"/>
@@ -59,5 +55,5 @@
     <joint name="${prefix}_wheel_joint" type="continuous">
       <parent link="${prefix}_mount"/>
-      <child  link="${prefix}_wheel"/>
+      <child link="${prefix}_wheel"/>
       <origin xyz="0 0 -${wheel_radius}" rpy="0 0 0"/>
       <axis xyz="0 1 0"/>

Commit message: Add IMU sensor to rover

File: src/mr2_rover_description/urdf/rover.urdf.xacro (robot description, xacro)
@@ -89,4 +89,13 @@
     </sensor>
   </gazebo>
+  <gazebo reference="imu_link">
+    <sensor name="imu_sensor" type="imu">
+      <always_on>1</always_on>
+      <update_rate>100</update_rate>
+      <visualize>false</visualize>
+      <topic>imu</topic>
+      <ignition_frame_id>imu_link</ignition_frame_id>
+    </sensor>
+  </gazebo>
   <ros2_control name="GazeboSimSystem" type="system">
     <hardware>

File: src/mr2_rover_description/urdf/rover_base.xacro (robot description, xacro)
@@ -89,8 +89,15 @@
     <link name="front_camera"/>
     <joint name="base_to_front_camera" type="fixed">
-	    <origin xyz="${length/2.0} 0 ${height}" rpy="0 ${front_camera_pitch} 0"/>
+            <origin xyz="${length/2.0} 0 ${height}" rpy="0 ${front_camera_pitch} 0"/>
       <parent link="base_link"/>
       <child link="front_camera"/>
     </joint>
+    <!-- IMU mounted at the top of the base box -->
+    <link name="imu_link"/>
+    <joint name="base_to_imu" type="fixed">
+      <origin xyz="0 0 ${height}" rpy="0 0 0"/>
+      <parent link="base_link"/>
+      <child link="imu_link"/>
+    </joint>
   </xacro:macro>
 </robot>

Commit message: add arm functionality to main (#23)
* add arm

* Expose arm joints to ros2_control

* fix joint axis direction

* moveit setup

* Add manipulator joint trajectory controller

* update moveit

* Spawn manipulator trajectory controller

* fix mimic warning

* increase velocity cap

* Include autonomous and MoveIt nodes in sim launch

File: src/mr2_rover_description/urdf/rover.urdf.xacro (robot description, xacro)
@@ -4,4 +4,5 @@
   <xacro:include filename="$(find mr2_rover_description)/urdf/rover_base.xacro"/>
   <xacro:include filename="$(find mr2_rover_description)/urdf/swerve_module.xacro"/>
+  <xacro:include filename="$(find mr2_rover_description)/urdf/manipulator.xacro"/>
   <!-- Chassis -->
   <xacro:rover_base/>
@@ -11,4 +12,6 @@
   <xacro:swerve_module prefix="rl" parent="left_rocker" xyz="-0.47 -0.08 -0.18"/>
   <xacro:swerve_module prefix="rr" parent="right_rocker" xyz="-0.47 0.08 -0.18"/>
+  <!-- Manipulator -->
+  <xacro:manipulator/>
   <!-- ros2_control plugin that loads the TwistToCommands controller -->
   <gazebo>
@@ -153,4 +156,35 @@
       <state_interface name="position"/>
     </joint>
+    <!-- Arm joint interfaces -->
+    <joint name="arm_j1">
+      <command_interface name="position"/>
+      <state_interface name="position"/>
+      <state_interface name="velocity"/>
+    </joint>
+    <joint name="arm_j2">
+      <command_interface name="position"/>
+      <state_interface name="position"/>
+      <state_interface name="velocity"/>
+    </joint>
+    <joint name="arm_j3">
+      <command_interface name="position"/>
+      <state_interface name="position"/>
+      <state_interface name="velocity"/>
+    </joint>
+    <joint name="arm_j4">
+      <command_interface name="position"/>
+      <state_interface name="position"/>
+      <state_interface name="velocity"/>
+    </joint>
+    <joint name="arm_j5">
+      <command_interface name="position"/>
+      <state_interface name="position"/>
+      <state_interface name="velocity"/>
+    </joint>
+    <joint name="arm_j6">
+      <command_interface name="position"/>
+      <state_interface name="position"/>
+      <state_interface name="velocity"/>
+    </joint>
   </ros2_control>
 </robot>

File: src/mr2_rover_description/urdf/rover_base.xacro (robot description, xacro)
@@ -75,4 +75,9 @@
       <mimic joint="left_rocker_joint" multiplier="-1" offset="0"/>
     </joint>
+    <joint name="right_rocker_joint_mimic" type="fixed">
+      <parent link="base_link" />
+      <child link="dummy_link" />
+    </joint>
+    <link name="dummy_link"/>
     <link name="left_gnss"/>
     <joint name="base_to_left_gnss" type="fixed">
