Commit message: Add motor 6 transmission to manipulator ros2_control

File: src/mr2_rover_description/urdf/single_joint.urdf.xacro (robot description, xacro)
@@ -1,4 +1,5 @@
 <?xml version="1.0"?>
 <robot xmlns:xacro="http://www.ros.org/wiki/xacro" name="single_joint">
+  <xacro:arg name="can_iface" default="can0"/>
   <link name="base_link"/>
   <link name="link1"/>
@@ -17,11 +18,18 @@
       <command_interface name="position"/>
       <state_interface name="position"/>
-      <state_interface name="velocity"/>
-      <state_interface name="effort"/>
-      <param name="device_plugin">mr2_devices_ak_servo/AkServoDevice</param>
-      <param name="motor_id">4</param>
-      <param name="gear_ratio">1.0</param>
-      <param name="can_iface">can0</param>
     </joint>
+    <transmission name="joint1_transmission">
+      <plugin>transmission_interface/SimpleTransmission</plugin>
+      <actuator name="motor4" role="motor4">
+        <command_interface name="position"/>
+        <state_interface name="position"/>
+        <param name="device_plugin">mr2_devices_ak_servo/AkServoDevice</param>
+        <param name="motor_id">4</param>
+        <param name="can_iface">$(arg can_iface)</param>
+      </actuator>
+      <joint name="joint1" role="joint1">
+        <mechanical_reduction>1.0</mechanical_reduction>
+      </joint>
+    </transmission>
   </ros2_control>
 </robot>

Commit message: Propagate velocity and effort through CAN transmissions

File: src/mr2_rover_description/urdf/single_joint.urdf.xacro (robot description, xacro)
@@ -1,4 +1,5 @@
 <?xml version="1.0"?>
 <robot xmlns:xacro="http://www.ros.org/wiki/xacro" name="single_joint">
+  <xacro:arg name="can_iface" default="can0"/>
   <link name="base_link"/>
   <link name="link1"/>
@@ -19,9 +20,21 @@
       <state_interface name="velocity"/>
       <state_interface name="effort"/>
+      <param name="actuator">motor4</param>
       <param name="device_plugin">mr2_devices_ak_servo/AkServoDevice</param>
       <param name="motor_id">4</param>
-      <param name="gear_ratio">1.0</param>
-      <param name="can_iface">can0</param>
+      <param name="can_iface">$(arg can_iface)</param>
     </joint>
+    <transmission name="joint1_transmission">
+      <plugin>transmission_interface/SimpleTransmission</plugin>
+      <actuator name="motor4" role="motor4">
+        <command_interface name="position"/>
+        <state_interface name="position"/>
+        <state_interface name="velocity"/>
+        <state_interface name="effort"/>
+      </actuator>
+      <joint name="joint1" role="joint1">
+        <mechanical_reduction>1.0</mechanical_reduction>
+      </joint>
+    </transmission>
   </ros2_control>
 </robot>

Commit message: Map motor 6 to arm joint 6 in manipulator ros2_control (#24)
* Add motor 6 transmission to manipulator ros2_control

* Load CAN actuators from joint parameters

* Fix escaping in CAN hardware error message

* Expose CAN interface selection via launch arguments

* Remove AK servo gear ratio scaling

File: src/mr2_rover_description/urdf/single_joint.urdf.xacro (robot description, xacro)
@@ -1,4 +1,5 @@
 <?xml version="1.0"?>
 <robot xmlns:xacro="http://www.ros.org/wiki/xacro" name="single_joint">
+  <xacro:arg name="can_iface" default="can0"/>
   <link name="base_link"/>
   <link name="link1"/>
@@ -17,11 +18,19 @@
       <command_interface name="position"/>
       <state_interface name="position"/>
-      <state_interface name="velocity"/>
-      <state_interface name="effort"/>
+      <param name="actuator">motor4</param>
       <param name="device_plugin">mr2_devices_ak_servo/AkServoDevice</param>
       <param name="motor_id">4</param>
-      <param name="gear_ratio">1.0</param>
-      <param name="can_iface">can0</param>
+      <param name="can_iface">$(arg can_iface)</param>
     </joint>
+    <transmission name="joint1_transmission">
+      <plugin>transmission_interface/SimpleTransmission</plugin>
+      <actuator name="motor4" role="motor4">
+        <command_interface name="position"/>
+        <state_interface name="position"/>
+      </actuator>
+      <joint name="joint1" role="joint1">
+        <mechanical_reduction>1.0</mechanical_reduction>
+      </joint>
+    </transmission>
   </ros2_control>
 </robot>

Commit message: Add mock AK servo emulator and polish single joint demo

File: src/mr2_rover_description/urdf/single_joint.urdf.xacro (robot description, xacro)
@@ -2,6 +2,26 @@
 <robot xmlns:xacro="http://www.ros.org/wiki/xacro" name="single_joint">
   <xacro:arg name="can_iface" default="can0"/>
-  <link name="base_link"/>
-  <link name="link1"/>
+  <link name="base_link">
+    <visual>
+      <origin xyz="0 0 0.025" rpy="0 0 0"/>
+      <geometry>
+        <box size="0.2 0.2 0.05"/>
+      </geometry>
+      <material name="base_blue">
+        <color rgba="0.2 0.2 0.8 1.0"/>
+      </material>
+    </visual>
+  </link>
+  <link name="link1">
+    <visual>
+      <origin xyz="0.15 0 0" rpy="0 0 0"/>
+      <geometry>
+        <box size="0.3 0.05 0.05"/>
+      </geometry>
+      <material name="link_orange">
+        <color rgba="0.9 0.5 0.2 1.0"/>
+      </material>
+    </visual>
+  </link>
   <joint name="joint1" type="revolute">
     <parent link="base_link"/>

Commit message: Support velocity and effort feedback for AK servos (#26)
* Support velocity and effort feedback for AK servos

* Add mock AK servo emulator and polish single joint demo

File: src/mr2_rover_description/urdf/single_joint.urdf.xacro (robot description, xacro)
@@ -2,6 +2,26 @@
 <robot xmlns:xacro="http://www.ros.org/wiki/xacro" name="single_joint">
   <xacro:arg name="can_iface" default="can0"/>
-  <link name="base_link"/>
-  <link name="link1"/>
+  <link name="base_link">
+    <visual>
+      <origin xyz="0 0 0.025" rpy="0 0 0"/>
+      <geometry>
+        <box size="0.2 0.2 0.05"/>
+      </geometry>
+      <material name="base_blue">
+        <color rgba="0.2 0.2 0.8 1.0"/>
+      </material>
+    </visual>
+  </link>
+  <link name="link1">
+    <visual>
+      <origin xyz="0.15 0 0" rpy="0 0 0"/>
+      <geometry>
+        <box size="0.3 0.05 0.05"/>
+      </geometry>
+      <material name="link_orange">
+        <color rgba="0.9 0.5 0.2 1.0"/>
+      </material>
+    </visual>
+  </link>
   <joint name="joint1" type="revolute">
     <parent link="base_link"/>
@@ -18,4 +38,6 @@
       <command_interface name="position"/>
       <state_interface name="position"/>
+      <state_interface name="velocity"/>
+      <state_interface name="effort"/>
       <param name="actuator">motor4</param>
       <param name="device_plugin">mr2_devices_ak_servo/AkServoDevice</param>
@@ -28,4 +50,6 @@
         <command_interface name="position"/>
         <state_interface name="position"/>
+        <state_interface name="velocity"/>
+        <state_interface name="effort"/>
       </actuator>
       <joint name="joint1" role="joint1">
