Commit message: Expose arm joints to ros2_control

File: src/mr2_rover_description/urdf/manipulator.xacro (robot description, xacro)
@@ -1,5 +1,5 @@
 <?xml version="1.0"?>
 <robot xmlns:xacro="http://www.ros.org/wiki/xacro">
-    <xacro:macro name="manipulator" params="length:=0.73 width:=0.49 height:=0.19">
+  <xacro:macro name="manipulator" params="length:=0.73 width:=0.49 height:=0.19">
     <link name="arm_l1">
       <inertial>
@@ -9,5 +9,5 @@
       <visual>
         <geometry>
-		<cylinder radius="0.15" length="0.1"/>
+          <cylinder radius="0.15" length="0.1"/>
         </geometry>
         <origin xyz="0 0 0.05"/>
@@ -15,5 +15,5 @@
       <collision>
         <geometry>
-		<cylinder radius="0.15" length="0.1"/>
+          <cylinder radius="0.15" length="0.1"/>
         </geometry>
         <origin xyz="0 0 0.05"/>
@@ -27,5 +27,5 @@
       <visual>
         <geometry>
-		<cylinder radius="0.05" length="0.4"/>
+          <cylinder radius="0.05" length="0.4"/>
         </geometry>
         <origin xyz="0 0 0.2"/>
@@ -33,5 +33,5 @@
       <collision>
         <geometry>
-		<cylinder radius="0.05" length="0.4"/>
+          <cylinder radius="0.05" length="0.4"/>
         </geometry>
         <origin xyz="0 0 0.2"/>
@@ -45,5 +45,5 @@
       <visual>
         <geometry>
-		<cylinder radius="0.05" length="0.05"/>
+          <cylinder radius="0.05" length="0.05"/>
         </geometry>
         <origin xyz="0.025 0 0" rpy="0 -1.571 0"/>
@@ -51,5 +51,5 @@
       <collision>
         <geometry>
-		<cylinder radius="0.05" length="0.05"/>
+          <cylinder radius="0.05" length="0.05"/>
         </geometry>
         <origin xyz="0.025 0 0" rpy="0 -1.571 0"/>
@@ -63,5 +63,5 @@
       <visual>
         <geometry>
-		<cylinder radius="0.05" length="0.2"/>
+          <cylinder radius="0.05" length="0.2"/>
         </geometry>
         <origin xyz="0 0 -0.1"/>
@@ -69,5 +69,5 @@
       <collision>
         <geometry>
-		<cylinder radius="0.05" length="0.2"/>
+          <cylinder radius="0.05" length="0.2"/>
         </geometry>
         <origin xyz="0 0 -0.1"/>
@@ -81,5 +81,5 @@
       <visual>
         <geometry>
-		<cylinder radius="0.05" length="0.1"/>
+          <cylinder radius="0.05" length="0.1"/>
         </geometry>
         <origin xyz="0.05 0 0" rpy="0 -1.571 0"/>
@@ -87,5 +87,5 @@
       <collision>
         <geometry>
-		<cylinder radius="0.05" length="0.1"/>
+          <cylinder radius="0.05" length="0.1"/>
         </geometry>
         <origin xyz="0.05 0 0" rpy="0 -1.571 0"/>
@@ -99,5 +99,5 @@
       <visual>
         <geometry>
-		<box size="0.1 0.1 0.1"/>
+          <box size="0.1 0.1 0.1"/>
         </geometry>
         <origin xyz="0.05 0 0" rpy="0 0 0"/>
@@ -105,10 +105,10 @@
       <collision>
         <geometry>
-		<box size="0.1 0.1 0.1"/>
+          <box size="0.1 0.1 0.1"/>
         </geometry>
         <origin xyz="0.05 0 0" rpy="0 0 0"/>
       </collision>
     </link>
-    <joint name="arm_j1" type="fixed">
+    <joint name="arm_j1" type="revolute">
       <parent link="base_link"/>
       <child link="arm_l1"/>
@@ -117,5 +117,5 @@
       <limit lower="0" upper="1" effort="50" velocity="0.01"/>
     </joint>
-    <joint name="arm_j2" type="fixed">
+    <joint name="arm_j2" type="revolute">
       <parent link="arm_l1"/>
       <child link="arm_l2"/>
@@ -124,5 +124,5 @@
       <limit lower="0" upper="1" effort="50" velocity="0.01"/>
     </joint>
-    <joint name="arm_j3" type="fixed">
+    <joint name="arm_j3" type="revolute">
       <parent link="arm_l2"/>
       <child link="arm_l3"/>
@@ -131,5 +131,5 @@
       <limit lower="0" upper="1" effort="50" velocity="0.01"/>
     </joint>
-    <joint name="arm_j4" type="fixed">
+    <joint name="arm_j4" type="revolute">
       <parent link="arm_l3"/>
       <child link="arm_l4"/>
@@ -138,5 +138,5 @@
       <limit lower="0" upper="1" effort="50" velocity="0.01"/>
     </joint>
-    <joint name="arm_j5" type="fixed">
+    <joint name="arm_j5" type="revolute">
       <parent link="arm_l4"/>
       <child link="arm_l5"/>
@@ -145,5 +145,5 @@
       <limit lower="0" upper="1" effort="50" velocity="0.01"/>
     </joint>
-    <joint name="arm_j6" type="fixed">
+    <joint name="arm_j6" type="revolute">
       <parent link="arm_l5"/>
       <child link="arm_l6"/>

File: src/mr2_rover_description/urdf/rover.urdf.xacro (robot description, xacro)
@@ -156,4 +156,35 @@
       <state_interface name="position"/>
     </joint>
+    <!-- Arm joint interfaces -->
+    <joint name="arm_j1">
+      <command_interface name="position"/>
+      <state_interface name="position"/>
+      <state_interface name="velocity"/>
+    </joint>
+    <joint name="arm_j2">
+      <command_interface name="position"/>
+      <state_interface name="position"/>
+      <state_interface name="velocity"/>
+    </joint>
+    <joint name="arm_j3">
+      <command_interface name="position"/>
+      <state_interface name="position"/>
+      <state_interface name="velocity"/>
+    </joint>
+    <joint name="arm_j4">
+      <command_interface name="position"/>
+      <state_interface name="position"/>
+      <state_interface name="velocity"/>
+    </joint>
+    <joint name="arm_j5">
+      <command_interface name="position"/>
+      <state_interface name="position"/>
+      <state_interface name="velocity"/>
+    </joint>
+    <joint name="arm_j6">
+      <command_interface name="position"/>
+      <state_interface name="position"/>
+      <state_interface name="velocity"/>
+    </joint>
   </ros2_control>
 </robot>

Commit message: fix joint axis direction

File: src/mr2_rover_description/urdf/manipulator.xacro (robot description, xacro)
@@ -27,5 +27,5 @@
       <visual>
         <geometry>
-          <cylinder radius="0.05" length="0.4"/>
+          <cylinder radius="0.02" length="0.4"/>
         </geometry>
         <origin xyz="0 0 0.2"/>
@@ -33,5 +33,5 @@
       <collision>
         <geometry>
-          <cylinder radius="0.05" length="0.4"/>
+          <cylinder radius="0.02" length="0.4"/>
         </geometry>
         <origin xyz="0 0 0.2"/>
@@ -63,5 +63,5 @@
       <visual>
         <geometry>
-          <cylinder radius="0.05" length="0.2"/>
+          <cylinder radius="0.02" length="0.2"/>
         </geometry>
         <origin xyz="0 0 -0.1"/>
@@ -69,5 +69,5 @@
       <collision>
         <geometry>
-          <cylinder radius="0.05" length="0.2"/>
+          <cylinder radius="0.02" length="0.2"/>
         </geometry>
         <origin xyz="0 0 -0.1"/>
@@ -115,5 +115,5 @@
       <origin xyz="${length/2.0} 0 ${height}" rpy="0 0 0"/>
       <axis xyz="0 0 1"/>
-      <limit lower="0" upper="1" effort="50" velocity="0.01"/>
+      <limit lower="-1" upper="1" effort="50" velocity="0.01"/>
     </joint>
     <joint name="arm_j2" type="revolute">
@@ -122,5 +122,5 @@
       <origin xyz="0.070 0 0.136" rpy="0 0 0"/>
       <axis xyz="0 1 0"/>
-      <limit lower="0" upper="1" effort="50" velocity="0.01"/>
+      <limit lower="-1" upper="1" effort="50" velocity="0.01"/>
     </joint>
     <joint name="arm_j3" type="revolute">
@@ -129,5 +129,5 @@
       <origin xyz="0 0 0.495" rpy="0 0 0"/>
       <axis xyz="0 1 0"/>
-      <limit lower="0" upper="1" effort="50" velocity="0.01"/>
+      <limit lower="" upper="1" effort="50" velocity="0.01"/>
     </joint>
     <joint name="arm_j4" type="revolute">
@@ -142,5 +142,5 @@
       <child link="arm_l5"/>
       <origin xyz="0 0 -0.260" rpy="0 0 0"/>
-      <axis xyz="0 0 1"/>
+      <axis xyz="0 1 0"/>
       <limit lower="0" upper="1" effort="50" velocity="0.01"/>
     </joint>
@@ -149,5 +149,5 @@
       <child link="arm_l6"/>
       <origin xyz="0.116 0 0" rpy="0 0 0"/>
-      <axis xyz="0 0 1"/>
+      <axis xyz="1 0 0"/>
       <limit lower="0" upper="1" effort="50" velocity="0.01"/>
     </joint>

Commit message: moveit setup

File: src/mr2_rover_description/urdf/manipulator.xacro (robot description, xacro)
@@ -129,5 +129,5 @@
       <origin xyz="0 0 0.495" rpy="0 0 0"/>
       <axis xyz="0 1 0"/>
-      <limit lower="" upper="1" effort="50" velocity="0.01"/>
+      <limit lower="-1" upper="1" effort="50" velocity="0.01"/>
     </joint>
     <joint name="arm_j4" type="revolute">
@@ -136,5 +136,5 @@
       <origin xyz="0.070 0 -0.138" rpy="0 0 0"/>
       <axis xyz="0 0 1"/>
-      <limit lower="0" upper="1" effort="50" velocity="0.01"/>
+      <limit lower="-1" upper="1" effort="50" velocity="0.01"/>
     </joint>
     <joint name="arm_j5" type="revolute">
@@ -143,5 +143,5 @@
       <origin xyz="0 0 -0.260" rpy="0 0 0"/>
       <axis xyz="0 1 0"/>
-      <limit lower="0" upper="1" effort="50" velocity="0.01"/>
+      <limit lower="-1" upper="1" effort="50" velocity="0.01"/>
     </joint>
     <joint name="arm_j6" type="revolute">
@@ -150,5 +150,5 @@
       <origin xyz="0.116 0 0" rpy="0 0 0"/>
       <axis xyz="1 0 0"/>
-      <limit lower="0" upper="1" effort="50" velocity="0.01"/>
+      <limit lower="-1" upper="1" effort="50" velocity="0.01"/>
     </joint>
   </xacro:macro>

Commit message: increase velocity cap

File: src/mr2_rover_description/urdf/manipulator.xacro (robot description, xacro)
@@ -115,5 +115,5 @@
       <origin xyz="${length/2.0} 0 ${height}" rpy="0 0 0"/>
       <axis xyz="0 0 1"/>
-      <limit lower="-1" upper="1" effort="50" velocity="0.01"/>
+      <limit lower="-1" upper="1" effort="50" velocity="1.0"/>
     </joint>
     <joint name="arm_j2" type="revolute">
@@ -122,5 +122,5 @@
       <origin xyz="0.070 0 0.136" rpy="0 0 0"/>
       <axis xyz="0 1 0"/>
-      <limit lower="-1" upper="1" effort="50" velocity="0.01"/>
+      <limit lower="-1" upper="1" effort="50" velocity="1.0"/>
     </joint>
     <joint name="arm_j3" type="revolute">
@@ -129,5 +129,5 @@
       <origin xyz="0 0 0.495" rpy="0 0 0"/>
       <axis xyz="0 1 0"/>
-      <limit lower="-1" upper="1" effort="50" velocity="0.01"/>
+      <limit lower="-1" upper="1" effort="50" velocity="1.0"/>
     </joint>
     <joint name="arm_j4" type="revolute">
@@ -136,5 +136,5 @@
       <origin xyz="0.070 0 -0.138" rpy="0 0 0"/>
       <axis xyz="0 0 1"/>
-      <limit lower="-1" upper="1" effort="50" velocity="0.01"/>
+      <limit lower="-1" upper="1" effort="50" velocity="1.0"/>
     </joint>
     <joint name="arm_j5" type="revolute">
@@ -143,5 +143,5 @@
       <origin xyz="0 0 -0.260" rpy="0 0 0"/>
       <axis xyz="0 1 0"/>
-      <limit lower="-1" upper="1" effort="50" velocity="0.01"/>
+      <limit lower="-1" upper="1" effort="50" velocity="1.0"/>
     </joint>
     <joint name="arm_j6" type="revolute">
@@ -150,5 +150,5 @@
       <origin xyz="0.116 0 0" rpy="0 0 0"/>
       <axis xyz="1 0 0"/>
-      <limit lower="-1" upper="1" effort="50" velocity="0.01"/>
+      <limit lower="-1" upper="1" effort="50" velocity="1.0"/>
     </joint>
   </xacro:macro>

Commit message: homing sensor overhaul and moveit2 changes

File: src/mr2_rover_description/urdf/manipulator.xacro (robot description, xacro)
@@ -1,4 +1,17 @@
 <?xml version="1.0"?>
 <robot xmlns:xacro="http://www.ros.org/wiki/xacro">
+  <!-- Joint limits (shared with ros2_control config) -->
+  <xacro:property name="arm_j1_lower_limit" value="-1"/>
+  <xacro:property name="arm_j1_upper_limit" value="1"/>
+  <xacro:property name="arm_j2_lower_limit" value="-1"/>
+  <xacro:property name="arm_j2_upper_limit" value="1"/>
+  <xacro:property name="arm_j3_lower_limit" value="-1"/>
+  <xacro:property name="arm_j3_upper_limit" value="1"/>
+  <xacro:property name="arm_j4_lower_limit" value="-1"/>
+  <xacro:property name="arm_j4_upper_limit" value="1"/>
+  <xacro:property name="arm_j5_lower_limit" value="-1"/>
+  <xacro:property name="arm_j5_upper_limit" value="1"/>
+  <xacro:property name="arm_j6_lower_limit" value="-1"/>
+  <xacro:property name="arm_j6_upper_limit" value="1"/>
   <xacro:macro name="manipulator" params="length:=0.73 width:=0.49 height:=0.19">
     <link name="arm_l1">
@@ -115,5 +128,5 @@
       <origin xyz="${length/2.0} 0 ${height}" rpy="0 0 0"/>
       <axis xyz="0 0 1"/>
-      <limit lower="-1" upper="1" effort="50" velocity="1.0"/>
+      <limit lower="${arm_j1_lower_limit}" upper="${arm_j1_upper_limit}" effort="50" velocity="1.0"/>
     </joint>
     <joint name="arm_j2" type="revolute">
@@ -122,5 +135,5 @@
       <origin xyz="0.070 0 0.136" rpy="0 0 0"/>
       <axis xyz="0 1 0"/>
-      <limit lower="-1" upper="1" effort="50" velocity="1.0"/>
+      <limit lower="${arm_j2_lower_limit}" upper="${arm_j2_upper_limit}" effort="50" velocity="1.0"/>
     </joint>
     <joint name="arm_j3" type="revolute">
@@ -129,5 +142,5 @@
       <origin xyz="0 0 0.495" rpy="0 0 0"/>
       <axis xyz="0 1 0"/>
-      <limit lower="-1" upper="1" effort="50" velocity="1.0"/>
+      <limit lower="${arm_j3_lower_limit}" upper="${arm_j3_upper_limit}" effort="50" velocity="1.0"/>
     </joint>
     <joint name="arm_j4" type="revolute">
@@ -136,5 +149,5 @@
       <origin xyz="0.070 0 -0.138" rpy="0 0 0"/>
       <axis xyz="0 0 1"/>
-      <limit lower="-1" upper="1" effort="50" velocity="1.0"/>
+      <limit lower="${arm_j4_lower_limit}" upper="${arm_j4_upper_limit}" effort="50" velocity="1.0"/>
     </joint>
     <joint name="arm_j5" type="revolute">
@@ -143,5 +156,5 @@
       <origin xyz="0 0 -0.260" rpy="0 0 0"/>
       <axis xyz="0 1 0"/>
-      <limit lower="-1" upper="1" effort="50" velocity="1.0"/>
+      <limit lower="${arm_j5_lower_limit}" upper="${arm_j5_upper_limit}" effort="50" velocity="1.0"/>
     </joint>
     <joint name="arm_j6" type="revolute">
@@ -150,5 +163,5 @@
       <origin xyz="0.116 0 0" rpy="0 0 0"/>
       <axis xyz="1 0 0"/>
-      <limit lower="-1" upper="1" effort="50" velocity="1.0"/>
+      <limit lower="${arm_j6_lower_limit}" upper="${arm_j6_upper_limit}" effort="50" velocity="1.0"/>
     </joint>
   </xacro:macro>

Commit message: add manipulator mesh

File: src/mr2_rover_description/urdf/manipulator.xacro (robot description, xacro)
@@ -14,4 +14,11 @@
   <xacro:property name="arm_j6_lower_limit" value="-1"/>
   <xacro:property name="arm_j6_upper_limit" value="1"/>
+  <!-- Shared shaded material for STL visuals (prevents unlit white appearance) -->
+  <material name="ArmGrey">
+    <color rgba="0.6 0.6 0.6 1.0"/>
+  </material>
+  <!-- Use file:// URI for meshes so both RViz (resource_retriever) and Gazebo resolve correctly -->
+  <xacro:property name="manipulator_mesh_prefix" value="file://$(find mr2_rover_description)/meshes/manipulator"/>
+  <xacro:property name="manipulator_mesh_scale" value="0.001"/>
   <xacro:macro name="manipulator" params="length:=0.73 width:=0.49 height:=0.19">
     <link name="arm_l1">
@@ -22,7 +29,9 @@
       <visual>
         <geometry>
-          <cylinder radius="0.15" length="0.1"/>
+          <mesh filename="${manipulator_mesh_prefix}/rover_manipulator_link1.stl"
+                scale="${manipulator_mesh_scale} ${manipulator_mesh_scale} ${manipulator_mesh_scale}"/>
         </geometry>
-        <origin xyz="0 0 0.05"/>
+        <origin xyz="0 0 0.032" rpy="0 0 3.1415926536"/>
+        <material name="ArmGrey"/>
       </visual>
       <collision>
@@ -40,7 +49,9 @@
       <visual>
         <geometry>
-          <cylinder radius="0.02" length="0.4"/>
+          <mesh filename="${manipulator_mesh_prefix}/rover_manipulator_link2.stl"
+                scale="${manipulator_mesh_scale} ${manipulator_mesh_scale} ${manipulator_mesh_scale}"/>
         </geometry>
-        <origin xyz="0 0 0.2"/>
+        <origin xyz="-0.070 0 -0.104" rpy="0 0 3.1415926536"/>
+        <material name="ArmGrey"/>
       </visual>
       <collision>
@@ -58,7 +69,9 @@
       <visual>
         <geometry>
-          <cylinder radius="0.05" length="0.05"/>
+          <mesh filename="${manipulator_mesh_prefix}/rover_manipulator_link3.stl"
+                scale="${manipulator_mesh_scale} ${manipulator_mesh_scale} ${manipulator_mesh_scale}"/>
         </geometry>
-        <origin xyz="0.025 0 0" rpy="0 -1.571 0"/>
+        <origin xyz="-0.070 0.0001 -0.599" rpy="0 0 3.1415926536"/>
+        <material name="ArmGrey"/>
       </visual>
       <collision>
@@ -76,7 +89,9 @@
       <visual>
         <geometry>
-          <cylinder radius="0.02" length="0.2"/>
+          <mesh filename="${manipulator_mesh_prefix}/rover_manipulator_link4.stl"
+                scale="${manipulator_mesh_scale} ${manipulator_mesh_scale} ${manipulator_mesh_scale}"/>
         </geometry>
-        <origin xyz="0 0 -0.1"/>
+        <origin xyz="-0.140 0.000 -0.461" rpy="0 0 3.1415926536"/>
+        <material name="ArmGrey"/>
       </visual>
       <collision>
@@ -94,7 +109,9 @@
       <visual>
         <geometry>
-          <cylinder radius="0.05" length="0.1"/>
+          <mesh filename="${manipulator_mesh_prefix}/rover_manipulator_link5.stl"
+                scale="${manipulator_mesh_scale} ${manipulator_mesh_scale} ${manipulator_mesh_scale}"/>
         </geometry>
-        <origin xyz="0.05 0 0" rpy="0 -1.571 0"/>
+        <origin xyz="-0.140 0.000 -0.201" rpy="0 0 3.1415926536"/>
+        <material name="ArmGrey"/>
       </visual>
       <collision>
@@ -115,4 +132,5 @@
         </geometry>
         <origin xyz="0.05 0 0" rpy="0 0 0"/>
+        <material name="ArmGrey"/>
       </visual>
       <collision>
