Commit message: Update rover description for sim

File: src/mr2_rover_description/ros2_control/rover_can.ros2_control.xacro (robot description, xacro)
@@ -1,5 +1,5 @@
 <?xml version="1.0"?>
 <robot xmlns:xacro="http://www.ros.org/wiki/xacro">
-  <xacro:macro name="manipulator_ak_can_ros2_control" params="name can_iface:=can0">
+  <xacro:macro name="rover_can_ros2_control" params="name can_iface:=can0">
     <ros2_control name="${name}" type="system">
       <hardware>

File: src/mr2_rover_description/urdf/manipulator_ak_can.urdf.xacro (robot description, xacro)
@@ -4,6 +4,6 @@
   <link name="base_link"/>
   <xacro:include filename="manipulator.xacro"/>
-  <xacro:include filename="$(find mr2_rover_description)/ros2_control/manipulator_ak_can.ros2_control.xacro"/>
+  <xacro:include filename="$(find mr2_rover_description)/ros2_control/rover_can.ros2_control.xacro"/>
   <xacro:manipulator/>
-  <xacro:manipulator_ak_can_ros2_control name="ArmCanSystem" can_iface="$(arg can_iface)"/>
+  <xacro:rover_can_ros2_control name="ArmCanSystem" can_iface="$(arg can_iface)"/>
 </robot>

File: src/mr2_rover_description/urdf/rover.urdf.xacro (robot description, xacro)
@@ -2,8 +2,19 @@
 <robot xmlns:xacro="http://www.ros.org/wiki/xacro" name="rover">
   <xacro:arg name="can_iface" default="can0"/>
+  <xacro:arg name="ros2_control_mode" default="gazebo"/>
+  <xacro:arg name="ros2_control_config" default="$(find mr2_rover_description)/config/controllers/rover_controllers.yaml"/>
+  <xacro:property name="ros2_control_mode_value" value="$(arg ros2_control_mode)"/>
+  <xacro:property name="ros2_control_config_value" value="$(arg ros2_control_config)"/>
+  <xacro:property name="can_iface_value" value="$(arg can_iface)"/>
+  <material name="Rubber">
+    <color rgba="0.05 0.05 0.05 1.0"/>
+  </material>
   <!-- Include component macros -->
   <xacro:include filename="$(find mr2_rover_description)/urdf/rover_base.xacro"/>
   <xacro:include filename="$(find mr2_rover_description)/urdf/swerve_module.xacro"/>
   <xacro:include filename="$(find mr2_rover_description)/urdf/manipulator.xacro"/>
+  <xacro:include filename="$(find mr2_rover_description)/ros2_control/rover_can.ros2_control.xacro"/>
+  <xacro:include filename="$(find mr2_rover_description)/ros2_control/rover_gazebo.ros2_control.xacro"/>
+  <xacro:include filename="$(find mr2_rover_description)/urdf/rover_gazebo_sensors.xacro"/>
   <!-- Chassis -->
   <xacro:rover_base/>
@@ -15,177 +26,10 @@
   <!-- Manipulator -->
   <xacro:manipulator/>
-  <!-- ros2_control plugin that loads the TwistToCommands controller -->
-  <gazebo>
-    <plugin filename="gz_ros2_control-system" name="gz_ros2_control::GazeboSimROS2ControlPlugin">
-      <robot_param>robot_description</robot_param>
-      <robot_param_node>robot_state_publisher</robot_param_node>
-      <parameters>$(find mr2_rover_description)/config/controllers.yaml</parameters>
-    </plugin>
-  </gazebo>
-  <gazebo reference="left_gnss">
-    <sensor name="left_gnss_sensor" type="navsat">
-      <always_on>1</always_on>
-      <update_rate>1</update_rate>
-      <visualize>true</visualize>
-      <topic>left_gnss/navsat</topic>
-      <ignition_frame_id>left_gnss</ignition_frame_id>
-    </sensor>
-  </gazebo>
-  <gazebo reference="right_gnss">
-    <sensor name="right_gnss_sensor" type="navsat">
-      <always_on>1</always_on>
-      <update_rate>1</update_rate>
-      <visualize>true</visualize>
-      <topic>right_gnss/navsat</topic>
-      <ignition_frame_id>right_gnss</ignition_frame_id>
-    </sensor>
-  </gazebo>
-  <gazebo reference="front_camera">
-    <sensor name="front_camera_sensor" type="rgbd_camera">
-	<update_rate>60</update_rate>
-	<always_on>1</always_on>
-        <visualize>true</visualize>
-	<topic>rgbd_camera</topic>
-        <ignition_frame_id>front_camera</ignition_frame_id>
-        <camera>
-          <horizontal_fov>1.0472</horizontal_fov>
-          <lens>
-            <intrinsics>
-              <!-- fx = fy = width / ( 2 * tan (hfov / 2 ) ) -->
-              <fx>554.25469</fx>
-              <fy>554.25469</fy>
-              <!-- cx = ( width + 1 ) / 2 -->
-              <cx>320.5</cx>
-              <!-- cy = ( height + 1 ) / 2 -->
-              <cy>240.5</cy>
-              <s>0</s>
-            </intrinsics>
-          </lens>
-          <distortion>
-            <k1>0.0</k1>
-            <k2>0.0</k2>
-            <k3>0.0</k3>
-            <p1>0.0</p1>
-            <p2>0.0</p2>
-            <center>0.5 0.5</center>
-          </distortion>
-          <image>
-            <width>640</width>
-            <height>480</height>
-            <format>R8G8B8</format>
-          </image>
-          <clip>
-            <near>0.01</near>
-            <far>300</far>
-          </clip>
-          <depth_camera>
-            <clip>
-              <near>0.1</near>
-              <far>10</far>
-            </clip>
-          </depth_camera>
-          <noise>
-            <type>gaussian</type>
-            <mean>0</mean>
-            <stddev>0.007</stddev>
-          </noise>
-        </camera>
-    </sensor>
-  </gazebo>
-  <gazebo reference="imu_link">
-    <sensor name="imu_sensor" type="imu">
-      <always_on>1</always_on>
-      <update_rate>100</update_rate>
-      <visualize>false</visualize>
-      <topic>imu</topic>
-      <ignition_frame_id>imu_link</ignition_frame_id>
-    </sensor>
-  </gazebo>
-  <ros2_control name="GazeboSimSystem" type="system">
-    <hardware>
-      <plugin>gz_ros2_control/GazeboSimSystem</plugin>
-    </hardware>
-    <!-- Mimic Joint -->
-    <joint name="left_rocker_joint">
-      <state_interface name="position"/>
-      <state_interface name="velocity"/>
-      <state_interface name="effort"/>
-    </joint>
-    <joint name="right_rocker_joint">
-      <param name="mimic">left_rocker_joint</param>
-      <param name="multiplier">-1</param>
-      <state_interface name="position"/>
-      <state_interface name="velocity"/>
-      <state_interface name="effort"/>
-    </joint>
-    <!-- Steering position interfaces -->
-    <joint name="fl_steering_joint">
-      <command_interface name="position"/>
-      <state_interface name="position"/>
-    </joint>
-    <joint name="fr_steering_joint">
-      <command_interface name="position"/>
-      <state_interface name="position"/>
-    </joint>
-    <joint name="rl_steering_joint">
-      <command_interface name="position"/>
-      <state_interface name="position"/>
-    </joint>
-    <joint name="rr_steering_joint">
-      <command_interface name="position"/>
-      <state_interface name="position"/>
-    </joint>
-    <!-- Wheel velocity interfaces -->
-    <joint name="fl_wheel_joint">
-      <command_interface name="velocity"/>
-      <state_interface name="velocity"/>
-      <state_interface name="position"/>
-    </joint>
-    <joint name="fr_wheel_joint">
-      <command_interface name="velocity"/>
-      <state_interface name="velocity"/>
-      <state_interface name="position"/>
-    </joint>
-    <joint name="rl_wheel_joint">
-      <command_interface name="velocity"/>
-      <state_interface name="velocity"/>
-      <state_interface name="position"/>
-    </joint>
-    <joint name="rr_wheel_joint">
-      <command_interface name="velocity"/>
-      <state_interface name="velocity"/>
-      <state_interface name="position"/>
-    </joint>
-    <!-- Arm joint interfaces -->
-    <joint name="arm_j1">
-      <command_interface name="position"/>
-      <state_interface name="position"/>
-      <state_interface name="velocity"/>
-    </joint>
-    <joint name="arm_j2">
-      <command_interface name="position"/>
-      <state_interface name="position"/>
-      <state_interface name="velocity"/>
-    </joint>
-    <joint name="arm_j3">
-      <command_interface name="position"/>
-      <state_interface name="position"/>
-      <state_interface name="velocity"/>
-    </joint>
-    <joint name="arm_j4">
-      <command_interface name="position"/>
-      <state_interface name="position"/>
-      <state_interface name="velocity"/>
-    </joint>
-    <joint name="arm_j5">
-      <command_interface name="position"/>
-      <state_interface name="position"/>
-      <state_interface name="velocity"/>
-    </joint>
-    <joint name="arm_j6">
-      <command_interface name="position"/>
-      <state_interface name="position"/>
-      <state_interface name="velocity"/>
-    </joint>
-  </ros2_control>
+  <xacro:if value="${ros2_control_mode_value == 'gazebo'}">
+    <xacro:rover_gazebo_sensors ros2_control_config="${ros2_control_config_value}"/>
+    <xacro:rover_gazebo_ros2_control name="GazeboSimSystem"/>
+  </xacro:if>
+  <xacro:if value="${ros2_control_mode_value == 'real_hardware'}">
+    <xacro:rover_can_ros2_control name="RoverCanSystem" can_iface="${can_iface_value}"/>
+  </xacro:if>
 </robot>

File: src/mr2_rover_description/urdf/rover_base.xacro (robot description, xacro)
@@ -2,5 +2,6 @@
 <robot xmlns:xacro="http://www.ros.org/wiki/xacro">
   <xacro:macro name="rover_base" params="length:=0.73 width:=0.49 height:=0.19 mass:=10 rocker_size:=0.1 rocker_mass:=0.5 joint_effort:=50 joint_vel:=2.0 joint_lim:=1.57 front_camera_pitch:=0.3491">
-    <link name="base_link">
+    <link name="base_link"/>
+    <link name="base_chassis">
       <inertial>
         <mass value="${mass}"/>
@@ -20,4 +21,9 @@
       </collision>
     </link>
+    <joint name="base_link_to_chassis" type="fixed">
+      <parent link="base_link"/>
+      <child link="base_chassis"/>
+      <origin xyz="0 0 0"/>
+    </joint>
     <link name="left_rocker">
       <inertial>
@@ -40,5 +46,5 @@
     </link>
     <joint name="left_rocker_joint" type="revolute">
-      <parent link="base_link"/>
+      <parent link="base_chassis"/>
       <child link="left_rocker"/>
       <origin xyz="0 -${width/2.0} 0" rpy="0 0 0"/>
@@ -67,5 +73,5 @@
     </link>
     <joint name="right_rocker_joint" type="revolute">
-      <parent link="base_link"/>
+      <parent link="base_chassis"/>
       <child link="right_rocker"/>
       <origin xyz="0 ${width/2.0} 0" rpy="0 0 0"/>
@@ -76,5 +82,5 @@
     </joint>
     <joint name="right_rocker_joint_mimic" type="fixed">
-      <parent link="base_link" />
+      <parent link="base_chassis" />
       <child link="dummy_link" />
     </joint>
@@ -83,5 +89,5 @@
     <joint name="base_to_left_gnss" type="fixed">
       <origin xyz="0 ${-width/2.0} 0" rpy="0 0 0"/>
-      <parent link="base_link"/>
+      <parent link="base_chassis"/>
       <child link="left_gnss"/>
     </joint>
@@ -89,5 +95,5 @@
     <joint name="base_to_right_gnss" type="fixed">
       <origin xyz="0 ${width/2.0} 0" rpy="0 0 0"/>
-      <parent link="base_link"/>
+      <parent link="base_chassis"/>
       <child link="right_gnss"/>
     </joint>
@@ -95,5 +101,5 @@
     <joint name="base_to_front_camera" type="fixed">
             <origin xyz="${length/2.0} 0 ${height}" rpy="0 ${front_camera_pitch} 0"/>
-      <parent link="base_link"/>
+      <parent link="base_chassis"/>
       <child link="front_camera"/>
     </joint>
@@ -102,5 +108,5 @@
     <joint name="base_to_imu" type="fixed">
       <origin xyz="0 0 ${height}" rpy="0 0 0"/>
-      <parent link="base_link"/>
+      <parent link="base_chassis"/>
       <child link="imu_link"/>
     </joint>

Commit message: polished ak motor driver

File: src/mr2_rover_description/ros2_control/rover_can.ros2_control.xacro (robot description, xacro)
@@ -83,6 +83,4 @@
         <param name="can_id">0x181</param>
         <param name="state_name">arm_j2_limit_switch</param>
-        <param name="counter_name">arm_j2_limit_counter</param>
-        <param name="timestamp_name">arm_j2_limit_timestamp_ms</param>
         <param name="edge_name">arm_j2_limit_edge</param>
         <param name="active_high">true</param>

File: src/mr2_rover_description/urdf/single_joint.urdf.xacro (robot description, xacro)
@@ -2,4 +2,6 @@
 <robot xmlns:xacro="http://www.ros.org/wiki/xacro" name="single_joint">
   <xacro:arg name="can_iface" default="can0"/>
+  <xacro:arg name="motor_id" default="4"/>
+  <xacro:property name="actuator_name" value="motor$(arg motor_id)"/>
   <link name="base_link">
     <visual>
@@ -40,12 +42,31 @@
       <state_interface name="velocity"/>
       <state_interface name="effort"/>
-      <param name="actuator">motor4</param>
+      <param name="actuator">${actuator_name}</param>
       <param name="device_plugin">mr2_devices_ak_servo/AkServoDevice</param>
-      <param name="motor_id">4</param>
+      <param name="motor_id">$(arg motor_id)</param>
       <param name="can_iface">$(arg can_iface)</param>
     </joint>
+    <gpio name="joint1_aux_encoder">
+      <param name="device_plugin">mr2_devices_sensors/AbsoluteEncoderDevice</param>
+      <param name="can_iface">$(arg can_iface)</param>
+      <param name="can_id">0x180</param>
+      <param name="ticks_per_rev">4096</param>
+      <param name="direction">1.0</param>
+      <param name="zero_offset_deg">0.0</param>
+      <param name="state_name">joint1/encoder_aux_angle</param>
+      <param name="raw_name">joint1/encoder_aux_raw</param>
+      <param name="flags_name">joint1/encoder_aux_flags</param>
+    </gpio>
+    <gpio name="joint1_limit_switch">
+      <param name="device_plugin">mr2_devices_sensors/LimitSwitchDevice</param>
+      <param name="can_iface">$(arg can_iface)</param>
+      <param name="can_id">0x181</param>
+      <param name="state_name">joint1/limit_switch_state</param>
+      <param name="edge_name">joint1/limit_switch_edge</param>
+      <param name="active_high">true</param>
+    </gpio>
     <transmission name="joint1_transmission">
       <plugin>transmission_interface/SimpleTransmission</plugin>
-      <actuator name="motor4" role="motor4">
+      <actuator name="${actuator_name}" role="${actuator_name}">
         <command_interface name="position"/>
         <state_interface name="position"/>
