Commit message: Fix sim ros2_control config and MoveIt Servo bringup

File: src/mr2_moveit/config/rover.ros2_control.xacro (robot description, xacro)
@@ -2,5 +2,5 @@
 <robot xmlns:xacro="http://www.ros.org/wiki/xacro">
     <xacro:macro name="rover_ros2_control" params="name initial_positions_file">
-        <xacro:property name="initial_positions" value="${load_yaml(initial_positions_file)['initial_positions']}"/>
+        <xacro:property name="initial_positions" value="${xacro.load_yaml(initial_positions_file)['initial_positions']}"/>
         <ros2_control name="${name}" type="system">
             <hardware>

File: src/mr2_rover_description/ros2_control/rover_gazebo.ros2_control.xacro (robot description, xacro)
@@ -1,8 +1,11 @@
 <?xml version="1.0"?>
 <robot xmlns:xacro="http://www.ros.org/wiki/xacro">
-  <xacro:macro name="rover_gazebo_ros2_control" params="name">
+  <xacro:macro name="rover_gazebo_ros2_control" params="name ros2_control_config">
     <ros2_control name="${name}" type="system">
       <hardware>
         <plugin>gz_ros2_control/GazeboSimSystem</plugin>
+        <param name="parameters">${ros2_control_config}</param>
+        <!-- Increase position loop gain so simulated joints actually chase commanded setpoints -->
+        <param name="position_proportional_gain">50.0</param>
       </hardware>
       <!-- Mimic Joint -->

File: src/mr2_rover_description/urdf/rover.urdf.xacro (robot description, xacro)
@@ -28,5 +28,5 @@
   <xacro:if value="${ros2_control_mode_value == 'gazebo'}">
     <xacro:rover_gazebo_sensors ros2_control_config="${ros2_control_config_value}"/>
-    <xacro:rover_gazebo_ros2_control name="GazeboSimSystem"/>
+    <xacro:rover_gazebo_ros2_control name="GazeboSimSystem" ros2_control_config="${ros2_control_config_value}"/>
   </xacro:if>
   <xacro:if value="${ros2_control_mode_value == 'real_hardware'}">
