Commit message: adjust geometry

File: ros2_ws/src/mr2_rover_description/urdf/rover.urdf.xacro (robot description, xacro)
@@ -7,4 +7,6 @@
   <xacro:property name="ros2_control_config_value" value="$(arg ros2_control_config)"/>
   <xacro:property name="can_iface_value" value="$(arg can_iface)"/>
+  <xacro:property name="rover_mesh_prefix" value="file://$(find mr2_rover_description)/meshes/rover"/>
+  <xacro:property name="rover_mesh_scale" value="0.01"/>
   <material name="Rubber">
     <color rgba="0.05 0.05 0.05 1.0"/>
@@ -20,8 +22,8 @@
   <xacro:rover_base/>
   <!-- Four modules -->
-  <xacro:swerve_module prefix="fl" parent="left_rocker" xyz=" 0.47 -0.08 -0.18"/>
-  <xacro:swerve_module prefix="fr" parent="right_rocker" xyz=" 0.47 0.08 -0.18"/>
-  <xacro:swerve_module prefix="rl" parent="left_rocker" xyz="-0.47 -0.08 -0.18"/>
-  <xacro:swerve_module prefix="rr" parent="right_rocker" xyz="-0.47 0.08 -0.18"/>
+  <xacro:swerve_module prefix="fr" parent="right_rocker" xyz=" 0.476931 -0.0797 -0.18" direction="1"/>
+  <xacro:swerve_module prefix="fl" parent="left_rocker" xyz=" 0.476931 0.0797 -0.18" direction="-1"/>
+  <xacro:swerve_module prefix="rr" parent="right_rocker" xyz="-0.476931 -0.0797 -0.18" direction="1"/>
+  <xacro:swerve_module prefix="rl" parent="left_rocker" xyz="-0.476931 0.0797 -0.18" direction="-1"/>
   <!-- Manipulator -->
   <xacro:manipulator/>

File: ros2_ws/src/mr2_rover_description/urdf/rover_base.xacro (robot description, xacro)
@@ -1,5 +1,5 @@
 <?xml version="1.0"?>
 <robot xmlns:xacro="http://www.ros.org/wiki/xacro">
-  <xacro:macro name="rover_base" params="length:=0.73 width:=0.49 height:=0.19 mass:=10 rocker_size:=0.1 rocker_mass:=0.5 joint_effort:=50 joint_vel:=2.0 joint_lim:=1.57 front_camera_pitch:=0.3491">
+  <xacro:macro name="rover_base" params="length:=0.73 width:=0.491 height:=0.19 mass:=10 rocker_size:=0.1 rocker_mass:=0.5 joint_effort:=50 joint_vel:=2.0 joint_lim:=1.57 front_camera_pitch:=0.3491">
     <link name="base_link"/>
     <link name="base_chassis">
@@ -26,5 +26,5 @@
       <origin xyz="0 0 0"/>
     </joint>
-    <link name="left_rocker">
+    <link name="right_rocker">
       <inertial>
         <origin xyz="0 -${width/2.0} 0"/>
@@ -34,7 +34,37 @@
       <visual>
         <geometry>
+          <mesh filename="${rover_mesh_prefix}/rocker.obj"
+                scale="${rover_mesh_scale} ${rover_mesh_scale} ${rover_mesh_scale}"/>
+        </geometry>
+        <origin xyz="0 ${width/2.0} -0.01"/>
+      </visual>
+      <collision>
+        <geometry>
           <box size="${rocker_size} ${rocker_size} ${rocker_size}"/>
         </geometry>
         <origin xyz="0 0 ${rocker_size/2.0}"/>
+      </collision>
+    </link>
+    <joint name="right_rocker_joint" type="revolute">
+      <parent link="base_chassis"/>
+      <child link="right_rocker"/>
+      <origin xyz="0 -${width/2.0} 0.06" rpy="0 0 0"/>
+      <axis xyz="0 1 0"/>
+      <dynamics damping="0.1" friction="0.0"/>
+      <limit lower="-${joint_lim}" upper="${joint_lim}" effort="${joint_effort}" velocity="${joint_vel}"/>
+      <mimic joint="left_rocker_joint" multiplier="-1" offset="0"/>
+    </joint>
+    <link name="left_rocker">
+      <inertial>
+        <origin xyz="0 ${width/2.0} 0"/>
+        <mass value="${rocker_mass}"/>
+        <inertia ixx="1e-3" ixy="0" ixz="0" iyy="1e-3" iyz="0" izz="1e-3"/>
+      </inertial>
+      <visual>
+        <geometry>
+          <mesh filename="${rover_mesh_prefix}/rocker.obj"
+                scale="${rover_mesh_scale} ${rover_mesh_scale} ${rover_mesh_scale}"/>
+        </geometry>
+	<origin xyz="0 ${-width/2.0} -0.01" rpy="0 0 3.141592"/>
       </visual>
       <collision>
@@ -48,36 +78,8 @@
       <parent link="base_chassis"/>
       <child link="left_rocker"/>
-      <origin xyz="0 -${width/2.0} 0" rpy="0 0 0"/>
+      <origin xyz="0 ${width/2.0} 0.06" rpy="0 0 0"/>
       <axis xyz="0 1 0"/>
       <dynamics damping="0.1" friction="0.0"/>
       <limit lower="-${joint_lim}" upper="${joint_lim}" effort="${joint_effort}" velocity="${joint_vel}"/>
-    </joint>
-    <link name="right_rocker">
-      <inertial>
-        <origin xyz="0 ${width/2.0} 0"/>
-        <mass value="${rocker_mass}"/>
-        <inertia ixx="1e-3" ixy="0" ixz="0" iyy="1e-3" iyz="0" izz="1e-3"/>
-      </inertial>
-      <visual>
-        <geometry>
-          <box size="${rocker_size} ${rocker_size} ${rocker_size}"/>
-        </geometry>
-        <origin xyz="0 0 ${rocker_size/2.0}"/>
-      </visual>
-      <collision>
-        <geometry>
-          <box size="${rocker_size} ${rocker_size} ${rocker_size}"/>
-        </geometry>
-        <origin xyz="0 0 ${rocker_size/2.0}"/>
-      </collision>
-    </link>
-    <joint name="right_rocker_joint" type="revolute">
-      <parent link="base_chassis"/>
-      <child link="right_rocker"/>
-      <origin xyz="0 ${width/2.0} 0" rpy="0 0 0"/>
-      <axis xyz="0 1 0"/>
-      <dynamics damping="0.1" friction="0.0"/>
-      <limit lower="-${joint_lim}" upper="${joint_lim}" effort="${joint_effort}" velocity="${joint_vel}"/>
-      <mimic joint="left_rocker_joint" multiplier="-1" offset="0"/>
     </joint>
     <joint name="right_rocker_joint_mimic" type="fixed">
@@ -86,19 +88,19 @@
     </joint>
     <link name="dummy_link"/>
+    <link name="right_gnss"/>
+    <joint name="base_to_right_gnss" type="fixed">
+      <origin xyz="0 ${-width/2.0} 0" rpy="0 0 0"/>
+      <parent link="base_chassis"/>
+      <child link="right_gnss"/>
+    </joint>
     <link name="left_gnss"/>
     <joint name="base_to_left_gnss" type="fixed">
-      <origin xyz="0 ${-width/2.0} 0" rpy="0 0 0"/>
+      <origin xyz="0 ${width/2.0} 0" rpy="0 0 0"/>
       <parent link="base_chassis"/>
       <child link="left_gnss"/>
     </joint>
-    <link name="right_gnss"/>
-    <joint name="base_to_right_gnss" type="fixed">
-      <origin xyz="0 ${width/2.0} 0" rpy="0 0 0"/>
-      <parent link="base_chassis"/>
-      <child link="right_gnss"/>
-    </joint>
     <link name="front_camera"/>
     <joint name="base_to_front_camera" type="fixed">
-            <origin xyz="${length/2.0} 0 ${height}" rpy="0 ${front_camera_pitch} 0"/>
+      <origin xyz="${length/2.0} 0 ${height}" rpy="0 ${front_camera_pitch} 0"/>
       <parent link="base_chassis"/>
       <child link="front_camera"/>
@@ -107,5 +109,5 @@
     <link name="imu_link"/>
     <joint name="base_to_imu" type="fixed">
-      <origin xyz="0 0 ${height}" rpy="0 0 0"/>
+      <origin xyz="0 0 0" rpy="0 0 0"/>
       <parent link="base_chassis"/>
       <child link="imu_link"/>

File: ros2_ws/src/mr2_rover_description/urdf/swerve_module.xacro (robot description, xacro)
@@ -1,9 +1,9 @@
 <?xml version="1.0"?>
 <robot xmlns:xacro="http://www.ros.org/wiki/xacro">
-  <xacro:macro name="swerve_module" params="prefix parent xyz">
+  <xacro:macro name="swerve_module" params="prefix parent xyz direction">
     <!-- local constants -->
     <xacro:property name="steer_limit" value="3.14"/>
     <xacro:property name="wheel_limit" value="20.0"/>
-    <xacro:property name="wheel_radius" value="0.11"/>
+    <xacro:property name="wheel_radius" value="0.125"/>
     <xacro:property name="wheel_width" value="0.11"/>
     <!-- Steering link -->
@@ -15,6 +15,8 @@
       <visual>
         <geometry>
-          <cylinder radius="0.11" length="0.02"/>
+          <mesh filename="${rover_mesh_prefix}/giuk.obj"
+                scale="${rover_mesh_scale} ${-rover_mesh_scale * direction} ${rover_mesh_scale}"/>
         </geometry>
+	<origin xyz="-0.47931 ${0.3252*direction} 0.17" rpy="0 0 0"/>
       </visual>
       <collision>
@@ -31,9 +33,9 @@
       </inertial>
       <visual>
-        <origin xyz="0 0 0" rpy="1.5708 0 0"/>
         <geometry>
-          <cylinder radius="${wheel_radius}" length="${wheel_width}"/>
+          <mesh filename="${rover_mesh_prefix}/wheel.obj"
+                scale="${rover_mesh_scale} ${-rover_mesh_scale * direction} ${rover_mesh_scale}"/>
         </geometry>
-        <material name="Rubber"/>
+	<origin xyz="-0.47931 ${0.3252*direction} 0.348457" rpy="0 0 0"/>
       </visual>
       <collision>
@@ -56,5 +58,5 @@
       <parent link="${prefix}_mount"/>
       <child link="${prefix}_wheel"/>
-      <origin xyz="0 0 -${wheel_radius}" rpy="0 0 0"/>
+      <origin xyz="0 0 -0.178457" rpy="0 0 0"/>
       <axis xyz="0 1 0"/>
       <limit effort="5" velocity="${wheel_limit}"/>
