Commit message: fix collision geometry of base

File: ros2_ws/src/mr2_rover_description/urdf/rover_base.xacro (robot description, xacro)
@@ -10,7 +10,7 @@
       <visual>
         <geometry>
-          <box size="${length} ${width} ${height}"/>
+	<box size="${length/2.0} ${width} ${height}"/>
         </geometry>
-        <origin xyz="0 0 ${height/2.0}"/>
+        <origin xyz="${-length/4.0} 0 ${height/2.0}"/>
       </visual>
       <collision>

Commit message: fix realsense shit

File: ros2_ws/src/mr2_rover_description/urdf/rover_base.xacro (robot description, xacro)
@@ -1,5 +1,5 @@
 <?xml version="1.0"?>
 <robot xmlns:xacro="http://www.ros.org/wiki/xacro">
-  <xacro:macro name="rover_base" params="length:=0.73 width:=0.491 height:=0.19 mass:=10 rocker_size:=0.1 rocker_mass:=0.5 joint_effort:=50 joint_vel:=2.0 joint_lim:=1.57 front_camera_pitch:=0.3491">
+  <xacro:macro name="rover_base" params="length:=0.73 width:=0.491 height:=0.19 mass:=10 rocker_size:=0.1 rocker_mass:=0.5 joint_effort:=50 joint_vel:=2.0 joint_lim:=1.57 front_camera_pitch:=0.523599">
     <link name="base_link"/>
     <link name="base_chassis">

Commit message: add ntrip server

File: ros2_ws/src/mr2_rover_description/urdf/rover_base.xacro (robot description, xacro)
@@ -102,5 +102,5 @@
     <link name="front_camera"/>
     <joint name="base_to_front_camera" type="fixed">
-      <origin xyz="${length/2.0} 0 ${height}" rpy="0 ${front_camera_pitch} 0"/>
+      <origin xyz="${length/2.0} 0 0" rpy="0 ${front_camera_pitch} 0"/>
       <parent link="base_chassis"/>
       <child link="front_camera"/>
