Commit message: what the fuck is wrong with codex

File: ros2_ws/src/mr2_rover_description/urdf/manipulator.xacro (robot description, xacro)
@@ -2,8 +2,8 @@
 <robot xmlns:xacro="http://www.ros.org/wiki/xacro">
   <!-- Joint limits (shared with ros2_control config) -->
-  <xacro:property name="arm_j1_lower_limit" value="-100"/>
-  <xacro:property name="arm_j1_upper_limit" value="100"/>
-  <xacro:property name="arm_j2_lower_limit" value="-100"/>
-  <xacro:property name="arm_j2_upper_limit" value="100"/>
+  <xacro:property name="arm_j1_lower_limit" value="-4"/>
+  <xacro:property name="arm_j1_upper_limit" value="4"/>
+  <xacro:property name="arm_j2_lower_limit" value="-0.645"/>
+  <xacro:property name="arm_j2_upper_limit" value="1.57"/>
   <xacro:property name="arm_j3_lower_limit" value="-100"/>
   <xacro:property name="arm_j3_upper_limit" value="100"/>

File: ros2_ws/src/mr2_rover_description/urdf/rover_gazebo_sensors.xacro (robot description, xacro)
@@ -30,5 +30,5 @@
     <gazebo reference="front_camera">
       <sensor name="front_camera_sensor" type="rgbd_camera">
-        <update_rate>60</update_rate>
+        <update_rate>30</update_rate>
         <always_on>1</always_on>
         <visualize>true</visualize>
@@ -36,5 +36,5 @@
         <ignition_frame_id>front_camera</ignition_frame_id>
         <camera>
-          <horizontal_fov>1.0472</horizontal_fov>
+          <horizontal_fov>1.5184</horizontal_fov>
           <lens>
             <intrinsics>
@@ -59,5 +59,5 @@
           <image>
             <width>320</width>
-            <height>240</height>
+            <height>180</height>
 	    <anti_aliasing>4</anti_aliasing>
             <format>R8G8B8</format>
@@ -84,5 +84,5 @@
       <sensor name="imu_sensor" type="imu">
         <always_on>1</always_on>
-        <update_rate>100</update_rate>
+        <update_rate>60</update_rate>
         <visualize>false</visualize>
         <topic>imu</topic>

Commit message: arm works

File: ros2_ws/src/mr2_rover_description/urdf/manipulator.xacro (robot description, xacro)
@@ -2,14 +2,14 @@
 <robot xmlns:xacro="http://www.ros.org/wiki/xacro">
   <!-- Joint limits (shared with ros2_control config) -->
-  <!-- <xacro:property name="arm_j1_lower_limit" value="-4"/> -->
-  <!-- <xacro:property name="arm_j1_upper_limit" value="4"/> -->
-  <xacro:property name="arm_j1_lower_limit" value="-100"/>
-  <xacro:property name="arm_j1_upper_limit" value="100"/>
+  <xacro:property name="arm_j1_lower_limit" value="-4"/>
+  <xacro:property name="arm_j1_upper_limit" value="4"/>
+  <!-- <xacro:property name="arm_j1_lower_limit" value="-100"/> -->
+  <!-- <xacro:property name="arm_j1_upper_limit" value="100"/> -->
   <xacro:property name="arm_j2_lower_limit" value="-0.645"/>
   <xacro:property name="arm_j2_upper_limit" value="1.57"/>
-  <!-- <xacro:property name="arm_j3_lower_limit" value="-2"/> -->
-  <!-- <xacro:property name="arm_j3_upper_limit" value="-0.2"/> -->
-  <xacro:property name="arm_j3_lower_limit" value="-100"/>
-  <xacro:property name="arm_j3_upper_limit" value="100"/>
+  <xacro:property name="arm_j3_lower_limit" value="-2"/>
+  <xacro:property name="arm_j3_upper_limit" value="-0.1"/>
+  <!-- <xacro:property name="arm_j3_lower_limit" value="-100"/> -->
+  <!-- <xacro:property name="arm_j3_upper_limit" value="100"/> -->
   <xacro:property name="arm_j4_lower_limit" value="-3.5"/>
   <xacro:property name="arm_j4_upper_limit" value="3.5"/>
