Commit message: haha

File: ros2_ws/src/mr2_rover_description/ros2_control/rover_can.ros2_control.xacro (robot description, xacro)
@@ -6,22 +6,23 @@
         <plugin>mr2_can_hardware_interface/CanHW</plugin>
       </hardware>
-      <joint name="arm_j1">
-        <command_interface name="position"/>
-        <state_interface name="position"/>
-        <state_interface name="velocity"/>
-        <state_interface name="effort"/>
-        <param name="actuator">motor1</param>
-        <param name="device_plugin">mr2_devices_ak_servo/AkServoDevice</param>
-        <param name="motor_id">1</param>
-        <param name="can_iface">${can_iface}</param>
-        <param name="joint_lower_limit">${arm_j1_lower_limit}</param>
-        <param name="joint_upper_limit">${arm_j1_upper_limit}</param>
-        <param name="homing_plugin">mr2_can_hardware_interface/AbsoluteEncoderPolicy</param>
-        <param name="homing_device_can_iface">${can_iface}</param>
-        <param name="homing_device_can_id">0x180</param>
-        <param name="homing_device_state_name">arm_j1_abs</param>
-        <param name="homing_device_flags_name">arm_j1_abs_flags</param>
-        <param name="homing_device_ticks_per_rev">4096</param>
-      </joint>
+      <!-- <joint name="arm_j1"> -->
+      <!--   <command_interface name="position"/> -->
+      <!--   <state_interface name="position"/> -->
+      <!--   <state_interface name="velocity"/> -->
+      <!--   <state_interface name="effort"/> -->
+      <!--   <param name="actuator">motor1</param> -->
+      <!--   <param name="device_plugin">mr2_devices_ak_servo/AkServoDevice</param> -->
+      <!--   <param name="motor_id">101</param> -->
+      <!--   <param name="can_iface">${can_iface}</param> -->
+      <!--   <param name="joint_lower_limit">${arm_j1_lower_limit}</param> -->
+      <!--   <param name="joint_upper_limit">${arm_j1_upper_limit}</param> -->
+      <!--   <param name="homing_plugin">mr2_can_hardware_interface/AbsoluteEncoderPolicy</param> -->
+      <!--   <param name="homing_device_can_iface">${can_iface}</param> -->
+      <!--   <param name="homing_device_can_id">201</param> -->
+      <!--   <param name="homing_device_state_name">arm_j1_abs</param> -->
+      <!--   <param name="homing_device_flags_name">arm_j1_abs_flags</param> -->
+      <!--   <param name="homing_device_ticks_per_rev">4096</param> -->
+      <!-- </joint> -->
+      <!---->
       <joint name="arm_j2">
         <command_interface name="position"/>
@@ -31,5 +32,5 @@
         <param name="actuator">motor2</param>
         <param name="device_plugin">mr2_devices_ak_servo/AkServoDevice</param>
-        <param name="motor_id">2</param>
+        <param name="motor_id">102</param>
         <param name="can_iface">${can_iface}</param>
         <param name="joint_lower_limit">${arm_j2_lower_limit}</param>
@@ -37,6 +38,47 @@
         <param name="homing_plugin">mr2_can_hardware_interface/LimitSwitchPolicy</param>
         <param name="homing_device_can_iface">${can_iface}</param>
-        <param name="homing_device_can_id">0x181</param>
+        <param name="homing_device_can_id">202</param>
         <param name="homing_device_state_name">arm_j2_limit_switch</param>
+        <param name="homing_device_active_high">true</param>
+        <param name="homing_search_direction">negative</param>
+        <param name="homing_approach_speed">0.1</param>
+        <param name="homing_fine_speed">0.02</param>
+        <param name="homing_backoff_distance">0.05</param>
+      </joint>
+      <joint name="arm_j3">
+        <command_interface name="position"/>
+        <state_interface name="position"/>
+        <state_interface name="velocity"/>
+        <state_interface name="effort"/>
+        <param name="actuator">motor3</param>
+        <param name="device_plugin">mr2_devices_ak_servo/AkServoDevice</param>
+        <param name="motor_id">103</param>
+        <param name="can_iface">${can_iface}</param>
+        <param name="joint_lower_limit">${arm_j3_lower_limit}</param>
+        <param name="joint_upper_limit">${arm_j3_upper_limit}</param>
+        <param name="homing_plugin">mr2_can_hardware_interface/AbsoluteEncoderPolicy</param>
+        <param name="homing_offset">-5.6</param>
+        <param name="homing_device_can_iface">${can_iface}</param>
+        <param name="homing_device_can_id">203</param>
+        <param name="homing_device_state_name">arm_j3_abs</param>
+        <param name="homing_device_flags_name">arm_j3_abs_flags</param>
+        <param name="homing_device_ticks_per_rev">4096</param>
+      </joint>
+      <joint name="arm_j4">
+        <command_interface name="position"/>
+        <state_interface name="position"/>
+        <state_interface name="velocity"/>
+        <state_interface name="effort"/>
+        <param name="actuator">motor4</param>
+        <param name="device_plugin">mr2_devices_ak_servo/AkServoDevice</param>
+        <param name="motor_id">104</param>
+        <param name="can_iface">${can_iface}</param>
+        <param name="joint_lower_limit">${arm_j4_lower_limit}</param>
+        <param name="joint_upper_limit">${arm_j4_upper_limit}</param>
+        <param name="homing_plugin">mr2_can_hardware_interface/LimitSwitchPolicy</param>
+        <param name="homing_position">-2.55</param>
+        <param name="homing_device_can_iface">${can_iface}</param>
+        <param name="homing_device_can_id">204</param>
+        <param name="homing_device_state_name">arm_j4_limit_switch</param>
         <param name="homing_device_active_high">true</param>
         <param name="homing_search_direction">negative</param>
@@ -45,34 +87,4 @@
         <param name="homing_backoff_distance">0.12</param>
       </joint>
-      <joint name="arm_j3">
-        <command_interface name="position"/>
-        <state_interface name="position"/>
-        <state_interface name="velocity"/>
-        <state_interface name="effort"/>
-        <param name="actuator">motor3</param>
-        <param name="device_plugin">mr2_devices_ak_servo/AkServoDevice</param>
-        <param name="motor_id">3</param>
-        <param name="can_iface">${can_iface}</param>
-        <param name="joint_lower_limit">${arm_j3_lower_limit}</param>
-        <param name="joint_upper_limit">${arm_j3_upper_limit}</param>
-        <param name="homing_plugin">mr2_can_hardware_interface/AbsoluteEncoderPolicy</param>
-        <param name="homing_device_can_iface">${can_iface}</param>
-        <param name="homing_device_can_id">0x182</param>
-        <param name="homing_device_state_name">arm_j3_abs</param>
-        <param name="homing_device_flags_name">arm_j3_abs_flags</param>
-        <param name="homing_device_ticks_per_rev">4096</param>
-      </joint>
-      <joint name="arm_j4">
-        <command_interface name="position"/>
-        <state_interface name="position"/>
-        <state_interface name="velocity"/>
-        <state_interface name="effort"/>
-        <param name="actuator">motor4</param>
-        <param name="device_plugin">mr2_devices_ak_servo/AkServoDevice</param>
-        <param name="motor_id">4</param>
-        <param name="can_iface">${can_iface}</param>
-        <param name="joint_lower_limit">${arm_j4_lower_limit}</param>
-        <param name="joint_upper_limit">${arm_j4_upper_limit}</param>
-      </joint>
       <joint name="arm_j5">
         <command_interface name="position"/>
@@ -82,8 +94,16 @@
         <param name="actuator">motor5</param>
         <param name="device_plugin">mr2_devices_ak_servo/AkServoDevice</param>
-        <param name="motor_id">5</param>
+        <param name="motor_id">105</param>
         <param name="can_iface">${can_iface}</param>
         <param name="joint_lower_limit">${arm_j5_lower_limit}</param>
         <param name="joint_upper_limit">${arm_j5_upper_limit}</param>
+        <param name="homing_plugin">mr2_can_hardware_interface/AbsoluteEncoderPolicy</param>
+        <param name="homing_offset">2.53</param>
+        <param name="homing_encoder_direction">-1.0</param>
+        <param name="homing_device_can_iface">${can_iface}</param>
+        <param name="homing_device_can_id">205</param>
+        <param name="homing_device_state_name">arm_j5_abs</param>
+        <param name="homing_device_flags_name">arm_j5_abs_flags</param>
+        <param name="homing_device_ticks_per_rev">4096</param>
       </joint>
       <joint name="arm_j6">
@@ -94,21 +114,31 @@
         <param name="actuator">motor6</param>
         <param name="device_plugin">mr2_devices_ak_servo/AkServoDevice</param>
-        <param name="motor_id">6</param>
+        <param name="motor_id">106</param>
         <param name="can_iface">${can_iface}</param>
         <param name="joint_lower_limit">${arm_j6_lower_limit}</param>
         <param name="joint_upper_limit">${arm_j6_upper_limit}</param>
-      </joint>
-      <transmission name="arm_j1_transmission">
-        <plugin>transmission_interface/SimpleTransmission</plugin>
-        <actuator name="motor1" role="motor1">
-          <command_interface name="position"/>
-          <state_interface name="position"/>
-          <state_interface name="velocity"/>
-          <state_interface name="effort"/>
-        </actuator>
-        <joint name="arm_j1" role="arm_j1">
-          <mechanical_reduction>3.0</mechanical_reduction>
-        </joint>
-      </transmission>
+        <param name="homing_plugin">mr2_can_hardware_interface/LimitSwitchPolicy</param>
+        <param name="homing_device_can_id">206</param>
+        <param name="homing_device_can_iface">${can_iface}</param>
+        <param name="homing_position">-3.03</param>
+        <param name="homing_device_state_name">arm_j6_limit_switch</param>
+        <param name="homing_device_active_high">true</param>
+        <param name="homing_search_direction">negative</param>
+        <param name="homing_approach_speed">0.35</param>
+        <param name="homing_fine_speed">0.05</param>
+        <param name="homing_backoff_distance">0.12</param>
+      </joint>
+      <!-- <transmission name="arm_j1_transmission"> -->
+      <!--   <plugin>transmission_interface/SimpleTransmission</plugin> -->
+      <!--   <actuator name="motor1" role="motor1"> -->
+      <!--     <command_interface name="position"/> -->
+      <!--     <state_interface name="position"/> -->
+      <!--     <state_interface name="velocity"/> -->
+      <!--     <state_interface name="effort"/> -->
+      <!--   </actuator> -->
+      <!--   <joint name="arm_j1" role="arm_j1"> -->
+      <!--     <mechanical_reduction>3.0</mechanical_reduction> -->
+      <!--   </joint> -->
+      <!-- </transmission> -->
       <transmission name="arm_j2_j3_transmission">
         <plugin>transmission_interface/FourBarLinkageTransmission</plugin>
@@ -128,5 +158,5 @@
         </actuator>
         <joint name="arm_j2" role="arm_j2">
-          <mechanical_reduction>1.0</mechanical_reduction>
+          <mechanical_reduction>-1.0</mechanical_reduction>
           <offset>0.0</offset>
         </joint>

File: ros2_ws/src/mr2_rover_description/urdf/manipulator.xacro (robot description, xacro)
@@ -4,14 +4,14 @@
   <xacro:property name="arm_j1_lower_limit" value="-1"/>
   <xacro:property name="arm_j1_upper_limit" value="1"/>
-  <xacro:property name="arm_j2_lower_limit" value="-1"/>
-  <xacro:property name="arm_j2_upper_limit" value="1"/>
-  <xacro:property name="arm_j3_lower_limit" value="-1"/>
-  <xacro:property name="arm_j3_upper_limit" value="1"/>
-  <xacro:property name="arm_j4_lower_limit" value="-1"/>
-  <xacro:property name="arm_j4_upper_limit" value="1"/>
-  <xacro:property name="arm_j5_lower_limit" value="-1"/>
-  <xacro:property name="arm_j5_upper_limit" value="1"/>
-  <xacro:property name="arm_j6_lower_limit" value="-1"/>
-  <xacro:property name="arm_j6_upper_limit" value="1"/>
+  <xacro:property name="arm_j2_lower_limit" value="-100"/>
+  <xacro:property name="arm_j2_upper_limit" value="100"/>
+  <xacro:property name="arm_j3_lower_limit" value="-100"/>
+  <xacro:property name="arm_j3_upper_limit" value="100"/>
+  <xacro:property name="arm_j4_lower_limit" value="-100"/>
+  <xacro:property name="arm_j4_upper_limit" value="100"/>
+  <xacro:property name="arm_j5_lower_limit" value="-100"/>
+  <xacro:property name="arm_j5_upper_limit" value="100"/>
+  <xacro:property name="arm_j6_lower_limit" value="-4"/>
+  <xacro:property name="arm_j6_upper_limit" value="4"/>
   <!-- Shared shaded material for STL visuals (prevents unlit white appearance) -->
   <material name="ArmGrey">

File: ros2_ws/src/mr2_rover_description/urdf/single_joint_limit_switch.urdf.xacro (robot description, xacro)
@@ -6,11 +6,12 @@
   <xacro:arg name="limit_switch_can_id" default="385"/>
   <xacro:arg name="limit_switch_active_high" default="true"/>
-  <xacro:arg name="joint_lower_limit" default="-3.14"/>
-  <xacro:arg name="joint_upper_limit" default="3.14"/>
+  <xacro:arg name="joint_lower_limit" default="-100"/>
+  <xacro:arg name="joint_upper_limit" default="100"/>
   <xacro:arg name="homing_search_direction" default="negative"/>
-  <xacro:arg name="homing_approach_speed" default="0.30"/>
-  <xacro:arg name="homing_backoff_speed" default="0.60"/>
-  <xacro:arg name="homing_fine_speed" default="0.03"/>
-  <xacro:arg name="homing_backoff_distance" default="0.10"/>
+  <xacro:arg name="homing_position" default="0.5"/>
+  <xacro:arg name="homing_approach_speed" default="0.05"/>
+  <xacro:arg name="homing_backoff_speed" default="0.05"/>
+  <xacro:arg name="homing_fine_speed" default="0.01"/>
+  <xacro:arg name="homing_backoff_distance" default="0.05"/>
   <xacro:property name="actuator_name" value="motor$(arg motor_id)"/>
   <link name="base_link">
@@ -63,5 +64,7 @@
       <param name="homing_device_state_name">joint1/limit_switch_state</param>
       <param name="homing_device_active_high">$(arg limit_switch_active_high)</param>
+      <param name="homing_device_active_high">$(arg limit_switch_active_high)</param>
       <param name="homing_search_direction">$(arg homing_search_direction)</param>
+      <param name="homing_position">$(arg homing_position)</param>
       <param name="homing_approach_speed">$(arg homing_approach_speed)</param>
       <param name="homing_backoff_speed">$(arg homing_backoff_speed)</param>
@@ -78,5 +81,5 @@
       </actuator>
       <joint name="joint1" role="joint1">
-        <mechanical_reduction>20.0</mechanical_reduction>
+        <mechanical_reduction>1.0</mechanical_reduction>
       </joint>
     </transmission>
