Commit message: add servo driver

File: ros2_ws/src/mr2_rover_description/ros2_control/rover_can.ros2_control.xacro (robot description, xacro)
@@ -6,4 +6,39 @@
         <plugin>mr2_can_hardware_interface/CanHW</plugin>
       </hardware>
+      <!-- <joint name="fl_steering_joint"> -->
+      <!--   <command_interface name="position"/> -->
+      <!--   <state_interface name="position"/> -->
+      <!--   <param name="actuator">steering_fl</param> -->
+      <!--   <param name="device_plugin">mr2_devices_steering_servo/SteeringServoDevice</param> -->
+      <!--   <param name="node_id">1</param> -->
+      <!--   <param name="can_iface">${can_iface}</param> -->
+      <!-- </joint> -->
+      <!---->
+      <!-- <joint name="fr_steering_joint"> -->
+      <!--   <command_interface name="position"/> -->
+      <!--   <state_interface name="position"/> -->
+      <!--   <param name="actuator">steering_fr</param> -->
+      <!--   <param name="device_plugin">mr2_devices_steering_servo/SteeringServoDevice</param> -->
+      <!--   <param name="node_id">2</param> -->
+      <!--   <param name="can_iface">${can_iface}</param> -->
+      <!-- </joint> -->
+      <!---->
+      <!-- <joint name="rl_steering_joint"> -->
+      <!--   <command_interface name="position"/> -->
+      <!--   <state_interface name="position"/> -->
+      <!--   <param name="actuator">steering_rl</param> -->
+      <!--   <param name="device_plugin">mr2_devices_steering_servo/SteeringServoDevice</param> -->
+      <!--   <param name="node_id">3</param> -->
+      <!--   <param name="can_iface">${can_iface}</param> -->
+      <!-- </joint> -->
+      <!---->
+      <!-- <joint name="rr_steering_joint"> -->
+      <!--   <command_interface name="position"/> -->
+      <!--   <state_interface name="position"/> -->
+      <!--   <param name="actuator">steering_rr</param> -->
+      <!--   <param name="device_plugin">mr2_devices_steering_servo/SteeringServoDevice</param> -->
+      <!--   <param name="node_id">4</param> -->
+      <!--   <param name="can_iface">${can_iface}</param> -->
+      <!-- </joint> -->
       <joint name="arm_j1">
         <command_interface name="position"/>
@@ -127,4 +162,47 @@
         <param name="homing_backoff_distance">0.12</param>
       </joint>
+      <!-- <transmission name="fl_steering_transmission"> -->
+      <!--   <plugin>transmission_interface/SimpleTransmission</plugin> -->
+      <!--   <actuator name="steering_fl" role="steering_fl"> -->
+      <!--     <command_interface name="position"/> -->
+      <!--     <state_interface name="position"/> -->
+      <!--   </actuator> -->
+      <!--   <joint name="fl_steering_joint" role="fl_steering_joint"> -->
+      <!--     <mechanical_reduction>1.0</mechanical_reduction> -->
+      <!--   </joint> -->
+      <!-- </transmission> -->
+      <!---->
+      <!-- <transmission name="fr_steering_transmission"> -->
+      <!--   <plugin>transmission_interface/SimpleTransmission</plugin> -->
+      <!--   <actuator name="steering_fr" role="steering_fr"> -->
+      <!--     <command_interface name="position"/> -->
+      <!--     <state_interface name="position"/> -->
+      <!--   </actuator> -->
+      <!--   <joint name="fr_steering_joint" role="fr_steering_joint"> -->
+      <!--     <mechanical_reduction>1.0</mechanical_reduction> -->
+      <!--   </joint> -->
+      <!-- </transmission> -->
+      <!---->
+      <!-- <transmission name="rl_steering_transmission"> -->
+      <!--   <plugin>transmission_interface/SimpleTransmission</plugin> -->
+      <!--   <actuator name="steering_rl" role="steering_rl"> -->
+      <!--     <command_interface name="position"/> -->
+      <!--     <state_interface name="position"/> -->
+      <!--   </actuator> -->
+      <!--   <joint name="rl_steering_joint" role="rl_steering_joint"> -->
+      <!--     <mechanical_reduction>1.0</mechanical_reduction> -->
+      <!--   </joint> -->
+      <!-- </transmission> -->
+      <!---->
+      <!-- <transmission name="rr_steering_transmission"> -->
+      <!--   <plugin>transmission_interface/SimpleTransmission</plugin> -->
+      <!--   <actuator name="steering_rr" role="steering_rr"> -->
+      <!--     <command_interface name="position"/> -->
+      <!--     <state_interface name="position"/> -->
+      <!--   </actuator> -->
+      <!--   <joint name="rr_steering_joint" role="rr_steering_joint"> -->
+      <!--     <mechanical_reduction>1.0</mechanical_reduction> -->
+      <!--   </joint> -->
+      <!-- </transmission> -->
       <transmission name="arm_j1_transmission">
         <plugin>transmission_interface/SimpleTransmission</plugin>
