Commit message: 2026 auto (#43)
* Merge origin/2026; add traversability pipeline; keep homing topic fixes

* Enable SiK bridge sim by default; remove toggle

* Refine sim SiK and traversability launch configs; add homing topic docs

* Fix SiK sim launch substitution; add grid_map_core deps

* Fix grid_map include path and aligned allocator for heightmap

* Add fullscreen toggle and stabilize ROS topic cleanup

* Add arm servo joystick control and steering updates

* Skip joint limits during homing

* Add arm servo card to delivery panel

* Add follow rover toggle on map

* update transitive packages

* good.

* add aruco

* add texture to mdrs mesh

* add sky

* adjust geometry

* update wheel encoder odom node, integrate to ros2_control

* Successfully integrated C++ implementation of pc2 -> traversability occupancy grid pipeline

* minute cleanup

* enable double battery

* Backup: <is battery monitor can id configurable>

* PC2 -> Nav2 pipeline via grid_map library

* fix PC2 -> Nav2

* fix pc2 -> nav2

* fix pc2 -> nav2

* Remove src/mr2_autonomous

* Backup; prepare for navigation.launch.py cleanup

* Clean-up for navigation.launch.py; Now fixing Nav2 pipeline...

* good tuning

* fix use_sim_time default_value bug

* what the fuck is wrong with codex

* calibration done

* fix collision geometry of base

* add servo driver

* fix encoder shit

* add udev rules

* add docker files

* kinda fix ublox / realsense launches

* fix pointcloud pipeline

* fix realsense shit

* add ntrip server

* fix homing

* arm works

* add base station code

* added base station arduino interface

* add base station arduino udev rules

* update nginx comand

* add udev ublox rules for the base station

* fix sik bridge serial port

* location telemetry is sent by the sik bridge

* add robot_localization to launch file

* fix tf nan issue

* set datum from base station location

* fix datum setting in robot localization

* set datum

* adjust qos

* adjust qos once more

* fix datum

* add cyclonedds config

* disable arduino reset on start

* rtcm / svin data via sik

* sik bridge rtcm packet limit fix

* add options to adjust surveying accuracy

---------

Co-authored-by: Jaeuk Kim <159106973+pianojay@users.noreply.github.com>

File: ros2_ws/src/mr2_rover_description/ros2_control/rover_can.ros2_control.xacro (robot description, xacro)
@@ -6,4 +6,36 @@
         <plugin>mr2_can_hardware_interface/CanHW</plugin>
       </hardware>
+      <joint name="fl_steering_joint">
+        <command_interface name="position"/>
+        <state_interface name="position"/>
+        <param name="actuator">steering_fl</param>
+        <param name="device_plugin">mr2_devices_steering_servo/SteeringServoDevice</param>
+        <param name="node_id">2</param>
+        <param name="can_iface">${can_iface}</param>
+      </joint>
+      <joint name="fr_steering_joint">
+        <command_interface name="position"/>
+        <state_interface name="position"/>
+        <param name="actuator">steering_fr</param>
+        <param name="device_plugin">mr2_devices_steering_servo/SteeringServoDevice</param>
+        <param name="node_id">3</param>
+        <param name="can_iface">${can_iface}</param>
+      </joint>
+      <joint name="rl_steering_joint">
+        <command_interface name="position"/>
+        <state_interface name="position"/>
+        <param name="actuator">steering_rl</param>
+        <param name="device_plugin">mr2_devices_steering_servo/SteeringServoDevice</param>
+        <param name="node_id">4</param>
+        <param name="can_iface">${can_iface}</param>
+      </joint>
+      <joint name="rr_steering_joint">
+        <command_interface name="position"/>
+        <state_interface name="position"/>
+        <param name="actuator">steering_rr</param>
+        <param name="device_plugin">mr2_devices_steering_servo/SteeringServoDevice</param>
+        <param name="node_id">1</param>
+        <param name="can_iface">${can_iface}</param>
+      </joint>
       <!-- <joint name="arm_j1"> -->
       <!--   <command_interface name="position"/> -->
@@ -19,118 +51,157 @@
       <!--   <param name="homing_plugin">mr2_can_hardware_interface/AbsoluteEncoderPolicy</param> -->
       <!--   <param name="homing_device_can_iface">${can_iface}</param> -->
+      <!--   <param name="homing_offset">-4.70</param> -->
+      <!--   <param name="homing_split_angle">2.43</param> -->
+      <!--   <param name="homing_encoder_direction">1.0</param> -->
+      <!--   <param name="homing_device_can_iface">${can_iface}</param> -->
       <!--   <param name="homing_device_can_id">201</param> -->
-      <!--   <param name="homing_device_state_name">arm_j1_abs</param> -->
-      <!--   <param name="homing_device_flags_name">arm_j1_abs_flags</param> -->
       <!--   <param name="homing_device_ticks_per_rev">4096</param> -->
       <!-- </joint> -->
       <!---->
-      <joint name="arm_j2">
-        <command_interface name="position"/>
-        <state_interface name="position"/>
-        <state_interface name="velocity"/>
-        <state_interface name="effort"/>
-        <param name="actuator">motor2</param>
-        <param name="device_plugin">mr2_devices_ak_servo/AkServoDevice</param>
-        <param name="motor_id">102</param>
-        <param name="can_iface">${can_iface}</param>
-        <param name="joint_lower_limit">${arm_j2_lower_limit}</param>
-        <param name="joint_upper_limit">${arm_j2_upper_limit}</param>
-        <param name="homing_plugin">mr2_can_hardware_interface/LimitSwitchPolicy</param>
-        <param name="homing_position">-0.69</param>
-        <param name="homing_device_can_iface">${can_iface}</param>
-        <param name="homing_device_can_id">202</param>
-        <param name="homing_device_state_name">arm_j2_limit_switch</param>
-        <param name="homing_device_active_high">true</param>
-        <param name="homing_search_direction">negative</param>
-        <param name="homing_approach_speed">0.1</param>
-        <param name="homing_fine_speed">0.02</param>
-        <param name="homing_backoff_distance">0.05</param>
-      </joint>
-      <joint name="arm_j3">
-        <command_interface name="position"/>
-        <state_interface name="position"/>
-        <state_interface name="velocity"/>
-        <state_interface name="effort"/>
-        <param name="actuator">motor3</param>
-        <param name="device_plugin">mr2_devices_ak_servo/AkServoDevice</param>
-        <param name="motor_id">103</param>
-        <param name="can_iface">${can_iface}</param>
-        <param name="joint_lower_limit">${arm_j3_lower_limit}</param>
-        <param name="joint_upper_limit">${arm_j3_upper_limit}</param>
-        <param name="homing_plugin">mr2_can_hardware_interface/AbsoluteEncoderPolicy</param>
-        <param name="homing_offset">5.05</param>
-        <param name="homing_split_angle">2.7</param>
-        <param name="homing_encoder_direction">-1.0</param>
-        <param name="homing_device_can_iface">${can_iface}</param>
-        <param name="homing_device_can_id">203</param>
-        <param name="homing_device_state_name">arm_j3_abs</param>
-        <param name="homing_device_flags_name">arm_j3_abs_flags</param>
-        <param name="homing_device_ticks_per_rev">4096</param>
-      </joint>
-      <joint name="arm_j4">
-        <command_interface name="position"/>
-        <state_interface name="position"/>
-        <state_interface name="velocity"/>
-        <state_interface name="effort"/>
-        <param name="actuator">motor4</param>
-        <param name="device_plugin">mr2_devices_ak_servo/AkServoDevice</param>
-        <param name="motor_id">104</param>
-        <param name="can_iface">${can_iface}</param>
-        <param name="joint_lower_limit">${arm_j4_lower_limit}</param>
-        <param name="joint_upper_limit">${arm_j4_upper_limit}</param>
-        <param name="homing_plugin">mr2_can_hardware_interface/LimitSwitchPolicy</param>
-        <param name="homing_position">-2.55</param>
-        <param name="homing_device_can_iface">${can_iface}</param>
-        <param name="homing_device_can_id">204</param>
-        <param name="homing_device_state_name">arm_j4_limit_switch</param>
-        <param name="homing_device_active_high">true</param>
-        <param name="homing_search_direction">negative</param>
-        <param name="homing_approach_speed">0.35</param>
-        <param name="homing_fine_speed">0.05</param>
-        <param name="homing_backoff_distance">0.12</param>
-      </joint>
-      <joint name="arm_j5">
-        <command_interface name="position"/>
-        <state_interface name="position"/>
-        <state_interface name="velocity"/>
-        <state_interface name="effort"/>
-        <param name="actuator">motor5</param>
-        <param name="device_plugin">mr2_devices_ak_servo/AkServoDevice</param>
-        <param name="motor_id">105</param>
-        <param name="can_iface">${can_iface}</param>
-        <param name="joint_lower_limit">${arm_j5_lower_limit}</param>
-        <param name="joint_upper_limit">${arm_j5_upper_limit}</param>
-        <param name="homing_plugin">mr2_can_hardware_interface/AbsoluteEncoderPolicy</param>
-        <param name="homing_offset">2.53</param>
-        <param name="homing_split_angle">0.98</param>
-        <param name="homing_encoder_direction">-1.0</param>
-        <param name="homing_device_can_iface">${can_iface}</param>
-        <param name="homing_device_can_id">205</param>
-        <param name="homing_device_state_name">arm_j5_abs</param>
-        <param name="homing_device_flags_name">arm_j5_abs_flags</param>
-        <param name="homing_device_ticks_per_rev">4096</param>
-      </joint>
-      <joint name="arm_j6">
-        <command_interface name="position"/>
-        <state_interface name="position"/>
-        <state_interface name="velocity"/>
-        <state_interface name="effort"/>
-        <param name="actuator">motor6</param>
-        <param name="device_plugin">mr2_devices_ak_servo/AkServoDevice</param>
-        <param name="motor_id">106</param>
-        <param name="can_iface">${can_iface}</param>
-        <param name="joint_lower_limit">${arm_j6_lower_limit}</param>
-        <param name="joint_upper_limit">${arm_j6_upper_limit}</param>
-        <param name="homing_plugin">mr2_can_hardware_interface/LimitSwitchPolicy</param>
-        <param name="homing_device_can_id">206</param>
-        <param name="homing_device_can_iface">${can_iface}</param>
-        <param name="homing_position">-3.03</param>
-        <param name="homing_device_state_name">arm_j6_limit_switch</param>
-        <param name="homing_device_active_high">true</param>
-        <param name="homing_search_direction">negative</param>
-        <param name="homing_approach_speed">0.35</param>
-        <param name="homing_fine_speed">0.05</param>
-        <param name="homing_backoff_distance">0.12</param>
-      </joint>
+      <!-- <joint name="arm_j2"> -->
+      <!--   <command_interface name="position"/> -->
+      <!--   <state_interface name="position"/> -->
+      <!--   <state_interface name="velocity"/> -->
+      <!--   <state_interface name="effort"/> -->
+      <!--   <param name="actuator">motor2</param> -->
+      <!--   <param name="device_plugin">mr2_devices_ak_servo/AkServoDevice</param> -->
+      <!--   <param name="motor_id">102</param> -->
+      <!--   <param name="can_iface">${can_iface}</param> -->
+      <!--   <param name="joint_lower_limit">${arm_j2_lower_limit}</param> -->
+      <!--   <param name="joint_upper_limit">${arm_j2_upper_limit}</param> -->
+      <!--   <param name="homing_plugin">mr2_can_hardware_interface/LimitSwitchPolicy</param> -->
+      <!--   <param name="homing_position">-0.69</param> -->
+      <!--   <param name="homing_device_can_iface">${can_iface}</param> -->
+      <!--   <param name="homing_device_can_id">202</param> -->
+      <!--   <param name="homing_device_active_high">true</param> -->
+      <!--   <param name="homing_search_direction">negative</param> -->
+      <!--   <param name="homing_approach_speed">0.1</param> -->
+      <!--   <param name="homing_fine_speed">0.02</param> -->
+      <!--   <param name="homing_backoff_distance">0.05</param> -->
+      <!-- </joint> -->
+      <!---->
+      <!-- <joint name="arm_j3"> -->
+      <!--   <command_interface name="position"/> -->
+      <!--   <state_interface name="position"/> -->
+      <!--   <state_interface name="velocity"/> -->
+      <!--   <state_interface name="effort"/> -->
+      <!--   <param name="actuator">motor3</param> -->
+      <!--   <param name="device_plugin">mr2_devices_ak_servo/AkServoDevice</param> -->
+      <!--   <param name="motor_id">103</param> -->
+      <!--   <param name="can_iface">${can_iface}</param> -->
+      <!--   <param name="joint_lower_limit">${arm_j3_lower_limit}</param> -->
+      <!--   <param name="joint_upper_limit">${arm_j3_upper_limit}</param> -->
+      <!--   <param name="homing_plugin">mr2_can_hardware_interface/AbsoluteEncoderPolicy</param> -->
+      <!--   <param name="homing_offset">-7.52</param> -->
+      <!--   <param name="homing_split_angle">3.4</param> -->
+      <!--   <param name="homing_encoder_direction">1.0</param> -->
+      <!--   <param name="homing_device_can_iface">${can_iface}</param> -->
+      <!--   <param name="homing_device_can_id">203</param> -->
+      <!--   <param name="homing_device_ticks_per_rev">4096</param> -->
+      <!-- </joint> -->
+      <!---->
+      <!-- <joint name="arm_j4"> -->
+      <!--   <command_interface name="position"/> -->
+      <!--   <state_interface name="position"/> -->
+      <!--   <state_interface name="velocity"/> -->
+      <!--   <state_interface name="effort"/> -->
+      <!--   <param name="actuator">motor4</param> -->
+      <!--   <param name="device_plugin">mr2_devices_ak_servo/AkServoDevice</param> -->
+      <!--   <param name="motor_id">104</param> -->
+      <!--   <param name="can_iface">${can_iface}</param> -->
+      <!--   <param name="joint_lower_limit">${arm_j4_lower_limit}</param> -->
+      <!--   <param name="joint_upper_limit">${arm_j4_upper_limit}</param> -->
+      <!--   <param name="homing_plugin">mr2_can_hardware_interface/LimitSwitchPolicy</param> -->
+      <!--   <param name="homing_position">-2.55</param> -->
+      <!--   <param name="homing_device_can_iface">${can_iface}</param> -->
+      <!--   <param name="homing_device_can_id">204</param> -->
+      <!--   <param name="homing_device_active_high">true</param> -->
+      <!--   <param name="homing_search_direction">negative</param> -->
+      <!--   <param name="homing_approach_speed">0.35</param> -->
+      <!--   <param name="homing_fine_speed">0.05</param> -->
+      <!--   <param name="homing_backoff_distance">0.12</param> -->
+      <!-- </joint> -->
+      <!---->
+      <!-- <joint name="arm_j5"> -->
+      <!--   <command_interface name="position"/> -->
+      <!--   <state_interface name="position"/> -->
+      <!--   <state_interface name="velocity"/> -->
+      <!--   <state_interface name="effort"/> -->
+      <!--   <param name="actuator">motor5</param> -->
+      <!--   <param name="device_plugin">mr2_devices_ak_servo/AkServoDevice</param> -->
+      <!--   <param name="motor_id">105</param> -->
+      <!--   <param name="can_iface">${can_iface}</param> -->
+      <!--   <param name="joint_lower_limit">${arm_j5_lower_limit}</param> -->
+      <!--   <param name="joint_upper_limit">${arm_j5_upper_limit}</param> -->
+      <!--   <param name="homing_plugin">mr2_can_hardware_interface/AbsoluteEncoderPolicy</param> -->
+      <!--   <param name="homing_offset">-2.46</param> -->
+      <!--   <param name="homing_split_angle">0.98</param> -->
+      <!--   <param name="homing_encoder_direction">1.0</param> -->
+      <!--   <param name="homing_device_can_iface">${can_iface}</param> -->
+      <!--   <param name="homing_device_can_id">205</param> -->
+      <!--   <param name="homing_device_ticks_per_rev">4096</param> -->
+      <!-- </joint> -->
+      <!---->
+      <!-- <joint name="arm_j6"> -->
+      <!--   <command_interface name="position"/> -->
+      <!--   <state_interface name="position"/> -->
+      <!--   <state_interface name="velocity"/> -->
+      <!--   <state_interface name="effort"/> -->
+      <!--   <param name="actuator">motor6</param> -->
+      <!--   <param name="device_plugin">mr2_devices_ak_servo/AkServoDevice</param> -->
+      <!--   <param name="motor_id">106</param> -->
+      <!--   <param name="can_iface">${can_iface}</param> -->
+      <!--   <param name="joint_lower_limit">${arm_j6_lower_limit}</param> -->
+      <!--   <param name="joint_upper_limit">${arm_j6_upper_limit}</param> -->
+      <!--   <param name="homing_plugin">mr2_can_hardware_interface/LimitSwitchPolicy</param> -->
+      <!--   <param name="homing_device_can_id">206</param> -->
+      <!--   <param name="homing_device_can_iface">${can_iface}</param> -->
+      <!--   <param name="homing_position">-3.03</param> -->
+      <!--   <param name="homing_device_active_high">true</param> -->
+      <!--   <param name="homing_search_direction">negative</param> -->
+      <!--   <param name="homing_approach_speed">0.35</param> -->
+      <!--   <param name="homing_fine_speed">0.05</param> -->
+      <!--   <param name="homing_backoff_distance">0.12</param> -->
+      <!-- </joint> -->
+      <transmission name="fl_steering_transmission">
+        <plugin>transmission_interface/SimpleTransmission</plugin>
+        <actuator name="steering_fl" role="steering_fl">
+          <command_interface name="position"/>
+          <state_interface name="position"/>
+        </actuator>
+        <joint name="fl_steering_joint" role="fl_steering_joint">
+          <mechanical_reduction>1.0</mechanical_reduction>
+        </joint>
+      </transmission>
+      <transmission name="fr_steering_transmission">
+        <plugin>transmission_interface/SimpleTransmission</plugin>
+        <actuator name="steering_fr" role="steering_fr">
+          <command_interface name="position"/>
+          <state_interface name="position"/>
+        </actuator>
+        <joint name="fr_steering_joint" role="fr_steering_joint">
+          <mechanical_reduction>1.0</mechanical_reduction>
+        </joint>
+      </transmission>
+      <transmission name="rl_steering_transmission">
+        <plugin>transmission_interface/SimpleTransmission</plugin>
+        <actuator name="steering_rl" role="steering_rl">
+          <command_interface name="position"/>
+          <state_interface name="position"/>
+        </actuator>
+        <joint name="rl_steering_joint" role="rl_steering_joint">
+          <mechanical_reduction>1.0</mechanical_reduction>
+        </joint>
+      </transmission>
+      <transmission name="rr_steering_transmission">
+        <plugin>transmission_interface/SimpleTransmission</plugin>
+        <actuator name="steering_rr" role="steering_rr">
+          <command_interface name="position"/>
+          <state_interface name="position"/>
+        </actuator>
+        <joint name="rr_steering_joint" role="rr_steering_joint">
+          <mechanical_reduction>1.0</mechanical_reduction>
+        </joint>
+      </transmission>
       <!-- <transmission name="arm_j1_transmission"> -->
       <!--   <plugin>transmission_interface/SimpleTransmission</plugin> -->
@@ -142,68 +213,72 @@
       <!--   </actuator> -->
       <!--   <joint name="arm_j1" role="arm_j1"> -->
-      <!--     <mechanical_reduction>3.0</mechanical_reduction> -->
-      <!--   </joint> -->
-      <!-- </transmission> -->
-      <transmission name="arm_j2_j3_transmission">
-        <plugin>transmission_interface/FourBarLinkageTransmission</plugin>
-        <actuator name="motor2" role="motor2">
-          <command_interface name="position"/>
-          <state_interface name="position"/>
-          <state_interface name="velocity"/>
-          <state_interface name="effort"/>
-          <mechanical_reduction>50.0</mechanical_reduction>
-        </actuator>
-        <actuator name="motor3" role="motor3">
-          <command_interface name="position"/>
-          <state_interface name="position"/>
-          <state_interface name="velocity"/>
-          <state_interface name="effort"/>
-          <mechanical_reduction>50.0</mechanical_reduction>
-        </actuator>
-        <joint name="arm_j2" role="arm_j2">
-          <mechanical_reduction>-1.0</mechanical_reduction>
-          <offset>0.0</offset>
-        </joint>
-        <joint name="arm_j3" role="arm_j3">
-          <mechanical_reduction>1.0</mechanical_reduction>
-          <offset>0.0</offset>
-        </joint>
-      </transmission>
-      <transmission name="arm_j4_transmission">
-        <plugin>transmission_interface/SimpleTransmission</plugin>
-        <actuator name="motor4" role="motor4">
-          <command_interface name="position"/>
-          <state_interface name="position"/>
-          <state_interface name="velocity"/>
-          <state_interface name="effort"/>
-        </actuator>
-        <joint name="arm_j4" role="arm_j4">
-          <mechanical_reduction>1.0</mechanical_reduction>
-        </joint>
-      </transmission>
-      <transmission name="arm_j5_transmission">
-        <plugin>transmission_interface/SimpleTransmission</plugin>
-        <actuator name="motor5" role="motor5">
-          <command_interface name="position"/>
-          <state_interface name="position"/>
-          <state_interface name="velocity"/>
-          <state_interface name="effort"/>
-        </actuator>
-        <joint name="arm_j5" role="arm_j5">
-          <mechanical_reduction>1.0</mechanical_reduction>
-        </joint>
-      </transmission>
-      <transmission name="arm_j6_transmission">
-        <plugin>transmission_interface/SimpleTransmission</plugin>
-        <actuator name="motor6" role="motor6">
-          <command_interface name="position"/>
-          <state_interface name="position"/>
-          <state_interface name="velocity"/>
-          <state_interface name="effort"/>
-        </actuator>
-        <joint name="arm_j6" role="arm_j6">
-          <mechanical_reduction>1.0</mechanical_reduction>
-        </joint>
-      </transmission>
+      <!--     <mechanical_reduction>-3.0</mechanical_reduction> -->
+      <!--   </joint> -->
+      <!-- </transmission> -->
+      <!---->
+      <!-- <transmission name="arm_j2_j3_transmission"> -->
+      <!--   <plugin>transmission_interface/FourBarLinkageTransmission</plugin> -->
+      <!--   <actuator name="motor2" role="motor2"> -->
+      <!--     <command_interface name="position"/> -->
+      <!--     <state_interface name="position"/> -->
+      <!--     <state_interface name="velocity"/> -->
+      <!--     <state_interface name="effort"/> -->
+      <!--     <mechanical_reduction>50.0</mechanical_reduction> -->
+      <!--   </actuator> -->
+      <!--   <actuator name="motor3" role="motor3"> -->
+      <!--     <command_interface name="position"/> -->
+      <!--     <state_interface name="position"/> -->
+      <!--     <state_interface name="velocity"/> -->
+      <!--     <state_interface name="effort"/> -->
+      <!--     <mechanical_reduction>50.0</mechanical_reduction> -->
+      <!--   </actuator> -->
+      <!--   <joint name="arm_j2" role="arm_j2"> -->
+      <!--     <mechanical_reduction>-1.0</mechanical_reduction> -->
+      <!--     <offset>0.0</offset> -->
+      <!--   </joint> -->
+      <!--   <joint name="arm_j3" role="arm_j3"> -->
+      <!--     <mechanical_reduction>1.0</mechanical_reduction> -->
+      <!--     <offset>0.0</offset> -->
+      <!--   </joint> -->
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