Commit message: 2026 auto (#43)
* Merge origin/2026; add traversability pipeline; keep homing topic fixes

* Enable SiK bridge sim by default; remove toggle

* Refine sim SiK and traversability launch configs; add homing topic docs

* Fix SiK sim launch substitution; add grid_map_core deps

* Fix grid_map include path and aligned allocator for heightmap

* Add fullscreen toggle and stabilize ROS topic cleanup

* Add arm servo joystick control and steering updates

* Skip joint limits during homing

* Add arm servo card to delivery panel

* Add follow rover toggle on map

* update transitive packages

* good.

* add aruco

* add texture to mdrs mesh

* add sky

* adjust geometry

* update wheel encoder odom node, integrate to ros2_control

* Successfully integrated C++ implementation of pc2 -> traversability occupancy grid pipeline

* minute cleanup

* enable double battery

* Backup: <is battery monitor can id configurable>

* PC2 -> Nav2 pipeline via grid_map library

* fix PC2 -> Nav2

* fix pc2 -> nav2

* fix pc2 -> nav2

* Remove src/mr2_autonomous

* Backup; prepare for navigation.launch.py cleanup

* Clean-up for navigation.launch.py; Now fixing Nav2 pipeline...

* good tuning

* fix use_sim_time default_value bug

* what the fuck is wrong with codex

* calibration done

* fix collision geometry of base

* add servo driver

* fix encoder shit

* add udev rules

* add docker files

* kinda fix ublox / realsense launches

* fix pointcloud pipeline

* fix realsense shit

* add ntrip server

* fix homing

* arm works

* add base station code

* added base station arduino interface

* add base station arduino udev rules

* update nginx comand

* add udev ublox rules for the base station

* fix sik bridge serial port

* location telemetry is sent by the sik bridge

* add robot_localization to launch file

* fix tf nan issue

* set datum from base station location

* fix datum setting in robot localization

* set datum

* adjust qos

* adjust qos once more

* fix datum

* add cyclonedds config

* disable arduino reset on start

* rtcm / svin data via sik

* sik bridge rtcm packet limit fix

* add options to adjust surveying accuracy

---------

Co-authored-by: Jaeuk Kim <159106973+pianojay@users.noreply.github.com>

File: ros2_ws/src/mr2_rover_description/urdf/manipulator.xacro (robot description, xacro)
@@ -2,14 +2,18 @@
 <robot xmlns:xacro="http://www.ros.org/wiki/xacro">
   <!-- Joint limits (shared with ros2_control config) -->
-  <xacro:property name="arm_j1_lower_limit" value="-1"/>
-  <xacro:property name="arm_j1_upper_limit" value="1"/>
-  <xacro:property name="arm_j2_lower_limit" value="-100"/>
-  <xacro:property name="arm_j2_upper_limit" value="100"/>
-  <xacro:property name="arm_j3_lower_limit" value="-100"/>
-  <xacro:property name="arm_j3_upper_limit" value="100"/>
-  <xacro:property name="arm_j4_lower_limit" value="-100"/>
-  <xacro:property name="arm_j4_upper_limit" value="100"/>
-  <xacro:property name="arm_j5_lower_limit" value="-100"/>
-  <xacro:property name="arm_j5_upper_limit" value="100"/>
+  <xacro:property name="arm_j1_lower_limit" value="-4"/>
+  <xacro:property name="arm_j1_upper_limit" value="4"/>
+  <!-- <xacro:property name="arm_j1_lower_limit" value="-100"/> -->
+  <!-- <xacro:property name="arm_j1_upper_limit" value="100"/> -->
+  <xacro:property name="arm_j2_lower_limit" value="-0.645"/>
+  <xacro:property name="arm_j2_upper_limit" value="1.57"/>
+  <xacro:property name="arm_j3_lower_limit" value="-2"/>
+  <xacro:property name="arm_j3_upper_limit" value="-0.1"/>
+  <!-- <xacro:property name="arm_j3_lower_limit" value="-100"/> -->
+  <!-- <xacro:property name="arm_j3_upper_limit" value="100"/> -->
+  <xacro:property name="arm_j4_lower_limit" value="-3.5"/>
+  <xacro:property name="arm_j4_upper_limit" value="3.5"/>
+  <xacro:property name="arm_j5_lower_limit" value="-0.12"/>
+  <xacro:property name="arm_j5_upper_limit" value="3.65"/>
   <xacro:property name="arm_j6_lower_limit" value="-4"/>
   <xacro:property name="arm_j6_upper_limit" value="4"/>

File: ros2_ws/src/mr2_rover_description/urdf/rover_base.xacro (robot description, xacro)
@@ -1,5 +1,5 @@
 <?xml version="1.0"?>
 <robot xmlns:xacro="http://www.ros.org/wiki/xacro">
-  <xacro:macro name="rover_base" params="length:=0.73 width:=0.49 height:=0.19 mass:=10 rocker_size:=0.1 rocker_mass:=0.5 joint_effort:=50 joint_vel:=2.0 joint_lim:=1.57 front_camera_pitch:=0.3491">
+  <xacro:macro name="rover_base" params="length:=0.73 width:=0.491 height:=0.19 mass:=10 rocker_size:=0.1 rocker_mass:=0.5 joint_effort:=50 joint_vel:=2.0 joint_lim:=1.57 front_camera_pitch:=0.523599">
     <link name="base_link"/>
     <link name="base_chassis">
@@ -10,7 +10,7 @@
       <visual>
         <geometry>
-          <box size="${length} ${width} ${height}"/>
+	<box size="${length/2.0} ${width} ${height}"/>
         </geometry>
-        <origin xyz="0 0 ${height/2.0}"/>
+        <origin xyz="${-length/4.0} 0 ${height/2.0}"/>
       </visual>
       <collision>
@@ -26,5 +26,5 @@
       <origin xyz="0 0 0"/>
     </joint>
-    <link name="left_rocker">
+    <link name="right_rocker">
       <inertial>
         <origin xyz="0 -${width/2.0} 0"/>
@@ -34,7 +34,37 @@
       <visual>
         <geometry>
+          <mesh filename="${rover_mesh_prefix}/rocker.obj"
+                scale="${rover_mesh_scale} ${rover_mesh_scale} ${rover_mesh_scale}"/>
+        </geometry>
+        <origin xyz="0 ${width/2.0} -0.01"/>
+      </visual>
+      <collision>
+        <geometry>
           <box size="${rocker_size} ${rocker_size} ${rocker_size}"/>
         </geometry>
         <origin xyz="0 0 ${rocker_size/2.0}"/>
+      </collision>
+    </link>
+    <joint name="right_rocker_joint" type="revolute">
+      <parent link="base_chassis"/>
+      <child link="right_rocker"/>
+      <origin xyz="0 -${width/2.0} 0.06" rpy="0 0 0"/>
+      <axis xyz="0 1 0"/>
+      <dynamics damping="0.1" friction="0.0"/>
+      <limit lower="-${joint_lim}" upper="${joint_lim}" effort="${joint_effort}" velocity="${joint_vel}"/>
+      <mimic joint="left_rocker_joint" multiplier="-1" offset="0"/>
+    </joint>
+    <link name="left_rocker">
+      <inertial>
+        <origin xyz="0 ${width/2.0} 0"/>
+        <mass value="${rocker_mass}"/>
+        <inertia ixx="1e-3" ixy="0" ixz="0" iyy="1e-3" iyz="0" izz="1e-3"/>
+      </inertial>
+      <visual>
+        <geometry>
+          <mesh filename="${rover_mesh_prefix}/rocker.obj"
+                scale="${rover_mesh_scale} ${rover_mesh_scale} ${rover_mesh_scale}"/>
+        </geometry>
+	<origin xyz="0 ${-width/2.0} -0.01" rpy="0 0 3.141592"/>
       </visual>
       <collision>
@@ -48,36 +78,8 @@
       <parent link="base_chassis"/>
       <child link="left_rocker"/>
-      <origin xyz="0 -${width/2.0} 0" rpy="0 0 0"/>
+      <origin xyz="0 ${width/2.0} 0.06" rpy="0 0 0"/>
       <axis xyz="0 1 0"/>
       <dynamics damping="0.1" friction="0.0"/>
       <limit lower="-${joint_lim}" upper="${joint_lim}" effort="${joint_effort}" velocity="${joint_vel}"/>
-    </joint>
-    <link name="right_rocker">
-      <inertial>
-        <origin xyz="0 ${width/2.0} 0"/>
-        <mass value="${rocker_mass}"/>
-        <inertia ixx="1e-3" ixy="0" ixz="0" iyy="1e-3" iyz="0" izz="1e-3"/>
-      </inertial>
-      <visual>
-        <geometry>
-          <box size="${rocker_size} ${rocker_size} ${rocker_size}"/>
-        </geometry>
-        <origin xyz="0 0 ${rocker_size/2.0}"/>
-      </visual>
-      <collision>
-        <geometry>
-          <box size="${rocker_size} ${rocker_size} ${rocker_size}"/>
-        </geometry>
-        <origin xyz="0 0 ${rocker_size/2.0}"/>
-      </collision>
-    </link>
-    <joint name="right_rocker_joint" type="revolute">
-      <parent link="base_chassis"/>
-      <child link="right_rocker"/>
-      <origin xyz="0 ${width/2.0} 0" rpy="0 0 0"/>
-      <axis xyz="0 1 0"/>
-      <dynamics damping="0.1" friction="0.0"/>
-      <limit lower="-${joint_lim}" upper="${joint_lim}" effort="${joint_effort}" velocity="${joint_vel}"/>
-      <mimic joint="left_rocker_joint" multiplier="-1" offset="0"/>
     </joint>
     <joint name="right_rocker_joint_mimic" type="fixed">
@@ -86,19 +88,19 @@
     </joint>
     <link name="dummy_link"/>
+    <link name="right_gnss"/>
+    <joint name="base_to_right_gnss" type="fixed">
+      <origin xyz="0 ${-width/2.0} 0" rpy="0 0 0"/>
+      <parent link="base_chassis"/>
+      <child link="right_gnss"/>
+    </joint>
     <link name="left_gnss"/>
     <joint name="base_to_left_gnss" type="fixed">
-      <origin xyz="0 ${-width/2.0} 0" rpy="0 0 0"/>
+      <origin xyz="0 ${width/2.0} 0" rpy="0 0 0"/>
       <parent link="base_chassis"/>
       <child link="left_gnss"/>
     </joint>
-    <link name="right_gnss"/>
-    <joint name="base_to_right_gnss" type="fixed">
-      <origin xyz="0 ${width/2.0} 0" rpy="0 0 0"/>
-      <parent link="base_chassis"/>
-      <child link="right_gnss"/>
-    </joint>
     <link name="front_camera"/>
     <joint name="base_to_front_camera" type="fixed">
-            <origin xyz="${length/2.0} 0 ${height}" rpy="0 ${front_camera_pitch} 0"/>
+      <origin xyz="${length/2.0} 0 0" rpy="0 ${front_camera_pitch} 0"/>
       <parent link="base_chassis"/>
       <child link="front_camera"/>
@@ -107,5 +109,5 @@
     <link name="imu_link"/>
     <joint name="base_to_imu" type="fixed">
-      <origin xyz="0 0 ${height}" rpy="0 0 0"/>
+      <origin xyz="0 0 0" rpy="0 0 0"/>
       <parent link="base_chassis"/>
       <child link="imu_link"/>

File: ros2_ws/src/mr2_rover_description/urdf/single_joint_limit_switch.urdf.xacro (robot description, xacro)
@@ -6,6 +6,6 @@
   <xacro:arg name="limit_switch_can_id" default="385"/>
   <xacro:arg name="limit_switch_active_high" default="true"/>
-  <xacro:arg name="joint_lower_limit" default="-100"/>
-  <xacro:arg name="joint_upper_limit" default="100"/>
+  <xacro:arg name="joint_lower_limit" default="-4"/>
+  <xacro:arg name="joint_upper_limit" default="4"/>
   <xacro:arg name="homing_search_direction" default="negative"/>
   <xacro:arg name="homing_position" default="0.5"/>
@@ -62,5 +62,4 @@
       <param name="homing_device_can_iface">$(arg can_iface)</param>
       <param name="homing_device_can_id">$(arg limit_switch_can_id)</param>
-      <param name="homing_device_state_name">joint1/limit_switch_state</param>
       <param name="homing_device_active_high">$(arg limit_switch_active_high)</param>
       <param name="homing_device_active_high">$(arg limit_switch_active_high)</param>
