Commit message: Fix topic name of sim to respect real; Ad hoc fix for realistic camera position definition

File: rover/ros2_ws/src/mr2_rover_description/urdf/rover_base.xacro (robot description, xacro)
@@ -2,4 +2,5 @@
 <robot xmlns:xacro="http://www.ros.org/wiki/xacro">
   <xacro:macro name="rover_base" params="length:=0.73 width:=0.491 height:=0.19 mass:=10 rocker_size:=0.1 rocker_mass:=0.5 joint_effort:=50 joint_vel:=2.0 joint_lim:=1.57 front_camera_pitch:=0.523599">
+    <!-- TODO: set as real dimension of the rover (#34) -->
     <link name="base_link"/>
     <link name="base_chassis">
@@ -102,5 +103,5 @@
     <link name="front_camera"/>
     <joint name="base_to_front_camera" type="fixed">
-      <origin xyz="${length/2.0} 0 0" rpy="0 ${front_camera_pitch} 0"/>
+      <origin xyz="${length/2.0 + 0.14} 0 0" rpy="0 ${front_camera_pitch} 0"/>
       <parent link="base_chassis"/>
       <child link="front_camera"/>

File: rover/ros2_ws/src/mr2_rover_description/urdf/rover_gazebo_sensors.xacro (robot description, xacro)
@@ -69,6 +69,6 @@
           <depth_camera>
             <clip>
-              <near>0.1</near>
-              <far>10</far>
+              <near>0.3</near>
+              <far>3.0</far>
             </clip>
           </depth_camera>

Commit message: Save new Realsense pitch

File: rover/ros2_ws/src/mr2_rover_description/urdf/rover_base.xacro (robot description, xacro)
@@ -1,5 +1,5 @@
 <?xml version="1.0"?>
 <robot xmlns:xacro="http://www.ros.org/wiki/xacro">
-  <xacro:macro name="rover_base" params="length:=0.73 width:=0.491 height:=0.19 mass:=10 rocker_size:=0.1 rocker_mass:=0.5 joint_effort:=50 joint_vel:=2.0 joint_lim:=1.57 front_camera_pitch:=0.523599">
+  <xacro:macro name="rover_base" params="length:=0.73 width:=0.491 height:=0.19 mass:=10 rocker_size:=0.1 rocker_mass:=0.5 joint_effort:=50 joint_vel:=2.0 joint_lim:=1.57 front_camera_pitch:=0.349066">
     <link name="base_link"/>
     <link name="base_chassis">

Commit message: fix aruco detection pipeline / realsense framerate configurations

File: rover/ros2_ws/src/mr2_rover_description/urdf/rover_base.xacro (robot description, xacro)
@@ -100,9 +100,22 @@
       <child link="left_gnss"/>
     </joint>
+    <link name="rgbd_camera"/>
+    <joint name="base_to_rgbd_camera" type="fixed">
+      <origin xyz="${length/2.0} 0 0" rpy="0 ${front_camera_pitch} 0"/>
+      <parent link="base_chassis"/>
+      <child link="rgbd_camera"/>
+    </joint>
     <link name="front_camera"/>
     <joint name="base_to_front_camera" type="fixed">
-      <origin xyz="${length/2.0} 0 0" rpy="0 ${front_camera_pitch} 0"/>
-      <parent link="base_chassis"/>
+      <origin xyz="${length/2.0} 0 0.5" rpy="0 0 0"/>
+      <parent link="base_link"/>
       <child link="front_camera"/>
+    </joint>
+    <!-- Optical frame for the front UVC camera (REP 103): x right, y down, z forward -->
+    <link name="front_camera_optical_frame"/>
+    <joint name="front_camera_to_optical" type="fixed">
+      <origin xyz="0 0 0" rpy="-1.57079632679 0 -1.57079632679"/>
+      <parent link="front_camera"/>
+      <child link="front_camera_optical_frame"/>
     </joint>
     <!-- IMU mounted at the top of the base box -->

File: rover/ros2_ws/src/mr2_rover_description/urdf/rover_gazebo_sensors.xacro (robot description, xacro)
@@ -28,11 +28,11 @@
       </sensor>
     </gazebo>
-    <gazebo reference="front_camera">
-      <sensor name="front_camera_sensor" type="rgbd_camera">
+    <gazebo reference="rgbd_camera">
+      <sensor name="rgbd_camera_sensor" type="rgbd_camera">
         <update_rate>30</update_rate>
         <always_on>1</always_on>
         <visualize>true</visualize>
         <topic>rgbd_camera</topic>
-        <ignition_frame_id>front_camera</ignition_frame_id>
+        <ignition_frame_id>rgbd_camera</ignition_frame_id>
         <camera>
           <horizontal_fov>1.5184</horizontal_fov>

Commit message: Connected vision pipeline sim to navigation for sim

File: rover/ros2_ws/src/mr2_rover_description/urdf/rover_base.xacro (robot description, xacro)
@@ -110,5 +110,5 @@
     <joint name="base_to_front_camera" type="fixed">
       <origin xyz="${length/2.0} 0 0.5" rpy="0 0 0"/>
-      <parent link="base_link"/>
+      <parent link="base_chassis"/>
       <child link="front_camera"/>
     </joint>

File: rover/ros2_ws/src/mr2_rover_description/urdf/rover_gazebo_sensors.xacro (robot description, xacro)
@@ -81,4 +81,57 @@
       </sensor>
     </gazebo>
+    <gazebo reference="front_camera">
+      <sensor name="front_camera_sensor" type="rgbd_camera">
+        <update_rate>30</update_rate>
+        <always_on>1</always_on>
+        <visualize>true</visualize>
+        <topic>front_camera</topic>
+        <ignition_frame_id>front_camera</ignition_frame_id>
+        <camera>
+          <horizontal_fov>1.5184</horizontal_fov>
+          <lens>
+            <intrinsics>
+              <!-- fx = fy = width / ( 2 * tan (hfov / 2 ) ) -->
+              <fx>277.12735</fx>
+              <fy>277.12735</fy>
+              <!-- cx = ( width + 1 ) / 2 -->
+              <cx>160.5</cx>
+              <!-- cy = ( height + 1 ) / 2 -->
+              <cy>120.5</cy>
+              <s>0</s>
+            </intrinsics>
+          </lens>
+          <distortion>
+            <k1>0.0</k1>
+            <k2>0.0</k2>
+            <k3>0.0</k3>
+            <p1>0.0</p1>
+            <p2>0.0</p2>
+            <center>0.5 0.5</center>
+          </distortion>
+          <image>
+            <width>320</width>
+            <height>180</height>
+            <anti_aliasing>4</anti_aliasing>
+            <format>R8G8B8</format>
+          </image>
+          <clip>
+            <near>0.3</near>
+            <far>3.0</far>
+          </clip>
+          <depth_camera>
+            <clip>
+              <near>0.3</near>
+              <far>3.0</far>
+            </clip>
+          </depth_camera>
+          <noise>
+            <type>gaussian</type>
+            <mean>0</mean>
+            <stddev>0.007</stddev>
+          </noise>
+        </camera>
+      </sensor>
+    </gazebo>
     <gazebo reference="imu_link">
       <sensor name="imu_sensor" type="imu">

Commit message: Save mr2-ubuntu (Jaeuk)

File: rover/ros2_ws/src/mr2_rover_description/urdf/rover_base.xacro (robot description, xacro)
@@ -114,5 +114,5 @@
     <link name="rgbd_camera"/>
     <joint name="base_to_rgbd_camera" type="fixed">
-      <origin xyz="${length/2.0 + 0.14} 0 0" rpy="0 ${front_camera_pitch} 0"/>
+      <origin xyz="${length/2.0 + 0.14} 0 0" rpy="0 ${front_camera_pitch} 0"/> <!-- For Gazebo rendering, add 1cm to 0.14 -->
       <parent link="base_chassis"/>
       <child link="rgbd_camera"/>
