Commit message: fix arm calibration values

File: rover/ros2_ws/src/mr2_rover_description/ros2_control/rover_can.ros2_control.xacro (robot description, xacro)
@@ -6,79 +6,72 @@
         <plugin>mr2_can_hardware_interface/CanHW</plugin>
       </hardware>
-      <!-- <joint name="fl_steering_joint"> -->
-      <!--   <command_interface name="position"/> -->
-      <!--   <state_interface name="position"/> -->
-      <!--   <param name="actuator">steering_fl</param> -->
-      <!--   <param name="device_plugin">mr2_devices_steering_servo/SteeringServoDevice</param> -->
-      <!--   <param name="node_id">2</param> -->
-      <!--   <param name="can_iface">${can_iface}</param> -->
-      <!-- </joint> -->
-      <!---->
-      <!-- <joint name="fr_steering_joint"> -->
-      <!--   <command_interface name="position"/> -->
-      <!--   <state_interface name="position"/> -->
-      <!--   <param name="actuator">steering_fr</param> -->
-      <!--   <param name="device_plugin">mr2_devices_steering_servo/SteeringServoDevice</param> -->
-      <!--   <param name="node_id">3</param> -->
-      <!--   <param name="can_iface">${can_iface}</param> -->
-      <!-- </joint> -->
-      <!---->
-      <!-- <joint name="rl_steering_joint"> -->
-      <!--   <command_interface name="position"/> -->
-      <!--   <state_interface name="position"/> -->
-      <!--   <param name="actuator">steering_rl</param> -->
-      <!--   <param name="device_plugin">mr2_devices_steering_servo/SteeringServoDevice</param> -->
-      <!--   <param name="node_id">4</param> -->
-      <!--   <param name="can_iface">${can_iface}</param> -->
-      <!-- </joint> -->
-      <!---->
-      <!-- <joint name="rr_steering_joint"> -->
-      <!--   <command_interface name="position"/> -->
-      <!--   <state_interface name="position"/> -->
-      <!--   <param name="actuator">steering_rr</param> -->
-      <!--   <param name="device_plugin">mr2_devices_steering_servo/SteeringServoDevice</param> -->
-      <!--   <param name="node_id">1</param> -->
-      <!--   <param name="can_iface">${can_iface}</param> -->
-      <!-- </joint> -->
-      <!---->
-      <!-- <joint name="fl_wheel_joint"> -->
-      <!--   <command_interface name="velocity"/> -->
-      <!--   <state_interface name="position"/> -->
-      <!--   <state_interface name="velocity"/> -->
-      <!--   <param name="actuator">drive_fl</param> -->
-      <!--   <param name="device_plugin">mr2_devices_drive_motor/DriveMotorDevice</param> -->
-      <!--   <param name="node_id">18</param> -->
-      <!--   <param name="can_iface">${can_iface}</param> -->
-      <!-- </joint> -->
-      <!---->
-      <!-- <joint name="fr_wheel_joint"> -->
-      <!--   <command_interface name="velocity"/> -->
-      <!--   <state_interface name="position"/> -->
-      <!--   <state_interface name="velocity"/> -->
-      <!--   <param name="actuator">drive_fr</param> -->
-      <!--   <param name="device_plugin">mr2_devices_drive_motor/DriveMotorDevice</param> -->
-      <!--   <param name="node_id">19</param> -->
-      <!--   <param name="can_iface">${can_iface}</param> -->
-      <!-- </joint> -->
-      <!---->
-      <!-- <joint name="rl_wheel_joint"> -->
-      <!--   <command_interface name="velocity"/> -->
-      <!--   <state_interface name="position"/> -->
-      <!--   <state_interface name="velocity"/> -->
-      <!--   <param name="actuator">drive_rl</param> -->
-      <!--   <param name="device_plugin">mr2_devices_drive_motor/DriveMotorDevice</param> -->
-      <!--   <param name="node_id">20</param> -->
-      <!--   <param name="can_iface">${can_iface}</param> -->
-      <!-- </joint> -->
-      <!---->
-      <!-- <joint name="rr_wheel_joint"> -->
-      <!--   <command_interface name="velocity"/> -->
-      <!--   <state_interface name="position"/> -->
-      <!--   <state_interface name="velocity"/> -->
-      <!--   <param name="actuator">drive_rr</param> -->
-      <!--   <param name="device_plugin">mr2_devices_drive_motor/DriveMotorDevice</param> -->
-      <!--   <param name="node_id">17</param> -->
-      <!--   <param name="can_iface">${can_iface}</param> -->
-      <!-- </joint> -->
+      <joint name="fl_steering_joint">
+        <command_interface name="position"/>
+        <state_interface name="position"/>
+        <param name="actuator">steering_fl</param>
+        <param name="device_plugin">mr2_devices_steering_servo/SteeringServoDevice</param>
+        <param name="node_id">2</param>
+        <param name="can_iface">${can_iface}</param>
+      </joint>
+      <joint name="fr_steering_joint">
+        <command_interface name="position"/>
+        <state_interface name="position"/>
+        <param name="actuator">steering_fr</param>
+        <param name="device_plugin">mr2_devices_steering_servo/SteeringServoDevice</param>
+        <param name="node_id">3</param>
+        <param name="can_iface">${can_iface}</param>
+      </joint>
+      <joint name="rl_steering_joint">
+        <command_interface name="position"/>
+        <state_interface name="position"/>
+        <param name="actuator">steering_rl</param>
+        <param name="device_plugin">mr2_devices_steering_servo/SteeringServoDevice</param>
+        <param name="node_id">4</param>
+        <param name="can_iface">${can_iface}</param>
+      </joint>
+      <joint name="rr_steering_joint">
+        <command_interface name="position"/>
+        <state_interface name="position"/>
+        <param name="actuator">steering_rr</param>
+        <param name="device_plugin">mr2_devices_steering_servo/SteeringServoDevice</param>
+        <param name="node_id">1</param>
+        <param name="can_iface">${can_iface}</param>
+      </joint>
+      <joint name="fl_wheel_joint">
+        <command_interface name="velocity"/>
+        <state_interface name="position"/>
+        <state_interface name="velocity"/>
+        <param name="actuator">drive_fl</param>
+        <param name="device_plugin">mr2_devices_drive_motor/DriveMotorDevice</param>
+        <param name="node_id">18</param>
+        <param name="can_iface">${can_iface}</param>
+      </joint>
+      <joint name="fr_wheel_joint">
+        <command_interface name="velocity"/>
+        <state_interface name="position"/>
+        <state_interface name="velocity"/>
+        <param name="actuator">drive_fr</param>
+        <param name="device_plugin">mr2_devices_drive_motor/DriveMotorDevice</param>
+        <param name="node_id">19</param>
+        <param name="can_iface">${can_iface}</param>
+      </joint>
+      <joint name="rl_wheel_joint">
+        <command_interface name="velocity"/>
+        <state_interface name="position"/>
+        <state_interface name="velocity"/>
+        <param name="actuator">drive_rl</param>
+        <param name="device_plugin">mr2_devices_drive_motor/DriveMotorDevice</param>
+        <param name="node_id">20</param>
+        <param name="can_iface">${can_iface}</param>
+      </joint>
+      <joint name="rr_wheel_joint">
+        <command_interface name="velocity"/>
+        <state_interface name="position"/>
+        <state_interface name="velocity"/>
+        <param name="actuator">drive_rr</param>
+        <param name="device_plugin">mr2_devices_drive_motor/DriveMotorDevice</param>
+        <param name="node_id">17</param>
+        <param name="can_iface">${can_iface}</param>
+      </joint>
       <joint name="arm_j1">
         <command_interface name="position"/>
@@ -134,7 +127,7 @@
         <param name="joint_upper_limit">${arm_j3_upper_limit}</param>
         <param name="homing_plugin">mr2_can_hardware_interface/AbsoluteEncoderPolicy</param>
-        <param name="homing_offset">-7.52</param>
+        <param name="homing_offset">4.91</param>
         <param name="homing_split_angle">3.4</param>
-        <param name="homing_encoder_direction">1.0</param>
+        <param name="homing_encoder_direction">-1.0</param>
         <param name="homing_device_can_iface">${can_iface}</param>
         <param name="homing_device_can_id">203</param>
@@ -211,95 +204,88 @@
         <param name="can_iface">${can_iface}</param>
       </joint>
-      <!-- <transmission name="fl_steering_transmission"> -->
-      <!--   <plugin>transmission_interface/SimpleTransmission</plugin> -->
-      <!--   <actuator name="steering_fl" role="steering_fl"> -->
-      <!--     <command_interface name="position"/> -->
-      <!--     <state_interface name="position"/> -->
-      <!--   </actuator> -->
-      <!--   <joint name="fl_steering_joint" role="fl_steering_joint"> -->
-      <!--     <mechanical_reduction>1.0</mechanical_reduction> -->
-      <!--   </joint> -->
-      <!-- </transmission> -->
-      <!---->
-      <!-- <transmission name="fr_steering_transmission"> -->
-      <!--   <plugin>transmission_interface/SimpleTransmission</plugin> -->
-      <!--   <actuator name="steering_fr" role="steering_fr"> -->
-      <!--     <command_interface name="position"/> -->
-      <!--     <state_interface name="position"/> -->
-      <!--   </actuator> -->
-      <!--   <joint name="fr_steering_joint" role="fr_steering_joint"> -->
-      <!--     <mechanical_reduction>1.0</mechanical_reduction> -->
-      <!--   </joint> -->
-      <!-- </transmission> -->
-      <!---->
-      <!-- <transmission name="rl_steering_transmission"> -->
-      <!--   <plugin>transmission_interface/SimpleTransmission</plugin> -->
-      <!--   <actuator name="steering_rl" role="steering_rl"> -->
-      <!--     <command_interface name="position"/> -->
-      <!--     <state_interface name="position"/> -->
-      <!--   </actuator> -->
-      <!--   <joint name="rl_steering_joint" role="rl_steering_joint"> -->
-      <!--     <mechanical_reduction>1.0</mechanical_reduction> -->
-      <!--   </joint> -->
-      <!-- </transmission> -->
-      <!---->
-      <!-- <transmission name="rr_steering_transmission"> -->
-      <!--   <plugin>transmission_interface/SimpleTransmission</plugin> -->
-      <!--   <actuator name="steering_rr" role="steering_rr"> -->
-      <!--     <command_interface name="position"/> -->
-      <!--     <state_interface name="position"/> -->
-      <!--   </actuator> -->
-      <!--   <joint name="rr_steering_joint" role="rr_steering_joint"> -->
-      <!--     <mechanical_reduction>1.0</mechanical_reduction> -->
-      <!--   </joint> -->
-      <!-- </transmission> -->
-      <!---->
-      <!-- <transmission name="fl_drive_transmission"> -->
-      <!--   <plugin>transmission_interface/SimpleTransmission</plugin> -->
-      <!--   <actuator name="drive_fl" role="drive_fl"> -->
-      <!--     <command_interface name="velocity"/> -->
-      <!--     <state_interface name="position"/> -->
-      <!--     <state_interface name="velocity"/> -->
-      <!--   </actuator> -->
-      <!--   <joint name="fl_wheel_joint" role="fl_wheel_joint"> -->
-      <!--     <mechanical_reduction>-1.0</mechanical_reduction> -->
-      <!--   </joint> -->
-      <!-- </transmission> -->
-      <!---->
-      <!-- <transmission name="fr_drive_transmission"> -->
-      <!--   <plugin>transmission_interface/SimpleTransmission</plugin> -->
-      <!--   <actuator name="drive_fr" role="drive_fr"> -->
-      <!--     <command_interface name="velocity"/> -->
-      <!--     <state_interface name="position"/> -->
-      <!--     <state_interface name="velocity"/> -->
-      <!--   </actuator> -->
-      <!--   <joint name="fr_wheel_joint" role="fr_wheel_joint"> -->
-      <!--     <mechanical_reduction>1.0</mechanical_reduction> -->
-      <!--   </joint> -->
-      <!-- </transmission> -->
-      <!---->
-      <!-- <transmission name="rl_drive_transmission"> -->
-      <!--   <plugin>transmission_interface/SimpleTransmission</plugin> -->
-      <!--   <actuator name="drive_rl" role="drive_rl"> -->
-      <!--     <command_interface name="velocity"/> -->
-      <!--     <state_interface name="position"/> -->
-      <!--     <state_interface name="velocity"/> -->
-      <!--   </actuator> -->
-      <!--   <joint name="rl_wheel_joint" role="rl_wheel_joint"> -->
-      <!--     <mechanical_reduction>-1.0</mechanical_reduction> -->
-      <!--   </joint> -->
-      <!-- </transmission> -->
-      <!---->
-      <!-- <transmission name="rr_drive_transmission"> -->
-      <!--   <plugin>transmission_interface/SimpleTransmission</plugin> -->
-      <!--   <actuator name="drive_rr" role="drive_rr"> -->
-      <!--     <command_interface name="velocity"/> -->
-      <!--     <state_interface name="position"/> -->
-      <!--     <state_interface name="velocity"/> -->
-      <!--   </actuator> -->
-      <!--   <joint name="rr_wheel_joint" role="rr_wheel_joint"> -->
-      <!--     <mechanical_reduction>-1.0</mechanical_reduction> -->
-      <!--   </joint> -->
-      <!-- </transmission> -->
+      <transmission name="fl_steering_transmission">
+        <plugin>transmission_interface/SimpleTransmission</plugin>
+        <actuator name="steering_fl" role="steering_fl">
+          <command_interface name="position"/>
+          <state_interface name="position"/>
+        </actuator>
+        <joint name="fl_steering_joint" role="fl_steering_joint">
+          <mechanical_reduction>1.0</mechanical_reduction>
+        </joint>
+      </transmission>
+      <transmission name="fr_steering_transmission">
+        <plugin>transmission_interface/SimpleTransmission</plugin>
+        <actuator name="steering_fr" role="steering_fr">
+          <command_interface name="position"/>
+          <state_interface name="position"/>
+        </actuator>
+        <joint name="fr_steering_joint" role="fr_steering_joint">
+          <mechanical_reduction>1.0</mechanical_reduction>
+        </joint>
+      </transmission>
+      <transmission name="rl_steering_transmission">
+        <plugin>transmission_interface/SimpleTransmission</plugin>
+        <actuator name="steering_rl" role="steering_rl">
+          <command_interface name="position"/>
+          <state_interface name="position"/>
+        </actuator>
+        <joint name="rl_steering_joint" role="rl_steering_joint">
+          <mechanical_reduction>1.0</mechanical_reduction>
+        </joint>
+      </transmission>
+      <transmission name="rr_steering_transmission">
+        <plugin>transmission_interface/SimpleTransmission</plugin>
+        <actuator name="steering_rr" role="steering_rr">
+          <command_interface name="position"/>
+          <state_interface name="position"/>
+        </actuator>
+        <joint name="rr_steering_joint" role="rr_steering_joint">
+          <mechanical_reduction>1.0</mechanical_reduction>
+        </joint>
+      </transmission>
+      <transmission name="fl_drive_transmission">
+        <plugin>transmission_interface/SimpleTransmission</plugin>
+        <actuator name="drive_fl" role="drive_fl">
+          <command_interface name="velocity"/>
+          <state_interface name="position"/>
+          <state_interface name="velocity"/>
+        </actuator>
+        <joint name="fl_wheel_joint" role="fl_wheel_joint">
+          <mechanical_reduction>-1.0</mechanical_reduction>
+        </joint>
+      </transmission>
+      <transmission name="fr_drive_transmission">
+        <plugin>transmission_interface/SimpleTransmission</plugin>
+        <actuator name="drive_fr" role="drive_fr">
+          <command_interface name="velocity"/>
+          <state_interface name="position"/>
+          <state_interface name="velocity"/>
+        </actuator>
+        <joint name="fr_wheel_joint" role="fr_wheel_joint">
+          <mechanical_reduction>1.0</mechanical_reduction>
+        </joint>
+      </transmission>
+      <transmission name="rl_drive_transmission">
+        <plugin>transmission_interface/SimpleTransmission</plugin>
+        <actuator name="drive_rl" role="drive_rl">
+          <command_interface name="velocity"/>
+          <state_interface name="position"/>
+          <state_interface name="velocity"/>
+        </actuator>
+        <joint name="rl_wheel_joint" role="rl_wheel_joint">
+          <mechanical_reduction>-1.0</mechanical_reduction>
+        </joint>
+      </transmission>
+      <transmission name="rr_drive_transmission">
+        <plugin>transmission_interface/SimpleTransmission</plugin>
+        <actuator name="drive_rr" role="drive_rr">
+          <command_interface name="velocity"/>
+          <state_interface name="position"/>
+          <state_interface name="velocity"/>
+        </actuator>
+        <joint name="rr_wheel_joint" role="rr_wheel_joint">
+          <mechanical_reduction>-1.0</mechanical_reduction>
+        </joint>
+      </transmission>
       <transmission name="arm_j1_transmission">
         <plugin>transmission_interface/SimpleTransmission</plugin>
@@ -311,5 +297,5 @@
         </actuator>
         <joint name="arm_j1" role="arm_j1">
-          <mechanical_reduction>-3.0</mechanical_reduction>
+          <mechanical_reduction>-2.0</mechanical_reduction>
         </joint>
       </transmission>

File: rover/ros2_ws/src/mr2_rover_description/urdf/manipulator.xacro (robot description, xacro)
@@ -2,28 +2,28 @@
 <robot xmlns:xacro="http://www.ros.org/wiki/xacro">
   <!-- Joint limits (shared with ros2_control config) -->
-  <!-- <xacro:property name="arm_j1_lower_limit" value="-4"/> -->
-  <!-- <xacro:property name="arm_j1_upper_limit" value="4"/> -->
-  <xacro:property name="arm_j1_lower_limit" value="-100"/>
-  <xacro:property name="arm_j1_upper_limit" value="100"/>
-  <!-- <xacro:property name="arm_j2_lower_limit" value="-0.645"/> -->
-  <!-- <xacro:property name="arm_j2_upper_limit" value="1.57"/> -->
-  <xacro:property name="arm_j2_lower_limit" value="-100"/>
-  <xacro:property name="arm_j2_upper_limit" value="100"/>
-  <!-- <xacro:property name="arm_j3_lower_limit" value="-2"/> -->
-  <!-- <xacro:property name="arm_j3_upper_limit" value="-0.1"/> -->
-  <xacro:property name="arm_j3_lower_limit" value="-100"/>
-  <xacro:property name="arm_j3_upper_limit" value="100"/>
-  <!-- <xacro:property name="arm_j4_lower_limit" value="-3.5"/> -->
-  <!-- <xacro:property name="arm_j4_upper_limit" value="3.5"/> -->
-  <xacro:property name="arm_j4_lower_limit" value="-100"/>
-  <xacro:property name="arm_j4_upper_limit" value="100"/>
-  <!-- <xacro:property name="arm_j5_lower_limit" value="-0.12"/> -->
-  <!-- <xacro:property name="arm_j5_upper_limit" value="3.65"/> -->
-  <xacro:property name="arm_j5_lower_limit" value="-100"/>
-  <xacro:property name="arm_j5_upper_limit" value="100"/>
-  <!-- <xacro:property name="arm_j6_lower_limit" value="-4"/> -->
-  <!-- <xacro:property name="arm_j6_upper_limit" value="4"/> -->
-  <xacro:property name="arm_j6_lower_limit" value="-100"/>
-  <xacro:property name="arm_j6_upper_limit" value="100"/>
+  <xacro:property name="arm_j1_lower_limit" value="-4"/>
+  <xacro:property name="arm_j1_upper_limit" value="4"/>
+  <!-- <xacro:property name="arm_j1_lower_limit" value="-100"/> -->
+  <!-- <xacro:property name="arm_j1_upper_limit" value="100"/> -->
+  <xacro:property name="arm_j2_lower_limit" value="-0.645"/>
+  <xacro:property name="arm_j2_upper_limit" value="1.57"/>
+  <!-- <xacro:property name="arm_j2_lower_limit" value="-100"/> -->
+  <!-- <xacro:property name="arm_j2_upper_limit" value="100"/> -->
+  <xacro:property name="arm_j3_lower_limit" value="-2"/>
+  <xacro:property name="arm_j3_upper_limit" value="-0.1"/>
+  <!-- <xacro:property name="arm_j3_lower_limit" value="-100"/> -->
+  <!-- <xacro:property name="arm_j3_upper_limit" value="100"/> -->
+  <xacro:property name="arm_j4_lower_limit" value="-3.5"/>
+  <xacro:property name="arm_j4_upper_limit" value="3.5"/>
+  <!-- <xacro:property name="arm_j4_lower_limit" value="-100"/> -->
+  <!-- <xacro:property name="arm_j4_upper_limit" value="100"/> -->
+  <xacro:property name="arm_j5_lower_limit" value="-0.12"/>
+  <xacro:property name="arm_j5_upper_limit" value="3.65"/>
+  <!-- <xacro:property name="arm_j5_lower_limit" value="-100"/> -->
+  <!-- <xacro:property name="arm_j5_upper_limit" value="100"/> -->
+  <xacro:property name="arm_j6_lower_limit" value="-4"/>
+  <xacro:property name="arm_j6_upper_limit" value="4"/>
+  <!-- <xacro:property name="arm_j6_lower_limit" value="-100"/> -->
+  <!-- <xacro:property name="arm_j6_upper_limit" value="100"/> -->
   <!-- Shared shaded material for STL visuals (prevents unlit white appearance) -->
   <material name="ArmGrey">
