Commit message: make manipulator optional

File: rover/ros2_ws/src/mr2_rover_description/ros2_control/rover_can.ros2_control.xacro (robot description, xacro)
@@ -1,5 +1,6 @@
 <?xml version="1.0"?>
 <robot xmlns:xacro="http://www.ros.org/wiki/xacro">n
-  <xacro:macro name="rover_can_ros2_control" params="name can_iface:=can0">
+  <xacro:macro name="rover_can_ros2_control" params="name can_iface:=can0 enable_manipulator:=true">
+    <xacro:property name="enable_manipulator_value" value="${enable_manipulator}"/>
     <ros2_control name="${name}" type="system">
       <hardware>
@@ -74,4 +75,5 @@
         <param name="can_iface">${can_iface}</param>
       </joint>
+      <xacro:if value="${enable_manipulator_value}">
       <joint name="arm_j1">
         <command_interface name="position"/>
@@ -204,4 +206,5 @@
         <param name="can_iface">${can_iface}</param>
       </joint>
+      </xacro:if>
       <transmission name="fl_steering_transmission">
         <plugin>transmission_interface/SimpleTransmission</plugin>
@@ -288,4 +291,5 @@
         </joint>
       </transmission>
+      <xacro:if value="${enable_manipulator_value}">
       <transmission name="arm_j1_transmission">
         <plugin>transmission_interface/SimpleTransmission</plugin>
@@ -371,4 +375,5 @@
         </joint>
       </transmission>
+      </xacro:if>
     </ros2_control>
   </xacro:macro>

File: rover/ros2_ws/src/mr2_rover_description/ros2_control/rover_gazebo.ros2_control.xacro (robot description, xacro)
@@ -1,5 +1,6 @@
 <?xml version="1.0"?>
 <robot xmlns:xacro="http://www.ros.org/wiki/xacro">
-  <xacro:macro name="rover_gazebo_ros2_control" params="name ros2_control_config">
+  <xacro:macro name="rover_gazebo_ros2_control" params="name ros2_control_config enable_manipulator:=true">
+    <xacro:property name="enable_manipulator_value" value="${enable_manipulator}"/>
     <ros2_control name="${name}" type="system">
       <hardware>
@@ -61,34 +62,36 @@
       </joint>
       <!-- Arm joint interfaces -->
-      <joint name="arm_j1">
-        <command_interface name="position"/>
-        <state_interface name="position"/>
-        <state_interface name="velocity"/>
-      </joint>
-      <joint name="arm_j2">
-        <command_interface name="position"/>
-        <state_interface name="position"/>
-        <state_interface name="velocity"/>
-      </joint>
-      <joint name="arm_j3">
-        <command_interface name="position"/>
-        <state_interface name="position"/>
-        <state_interface name="velocity"/>
-      </joint>
-      <joint name="arm_j4">
-        <command_interface name="position"/>
-        <state_interface name="position"/>
-        <state_interface name="velocity"/>
-      </joint>
-      <joint name="arm_j5">
-        <command_interface name="position"/>
-        <state_interface name="position"/>
-        <state_interface name="velocity"/>
-      </joint>
-      <joint name="arm_j6">
-        <command_interface name="position"/>
-        <state_interface name="position"/>
-        <state_interface name="velocity"/>
-      </joint>
+      <xacro:if value="${enable_manipulator_value}">
+        <joint name="arm_j1">
+          <command_interface name="position"/>
+          <state_interface name="position"/>
+          <state_interface name="velocity"/>
+        </joint>
+        <joint name="arm_j2">
+          <command_interface name="position"/>
+          <state_interface name="position"/>
+          <state_interface name="velocity"/>
+        </joint>
+        <joint name="arm_j3">
+          <command_interface name="position"/>
+          <state_interface name="position"/>
+          <state_interface name="velocity"/>
+        </joint>
+        <joint name="arm_j4">
+          <command_interface name="position"/>
+          <state_interface name="position"/>
+          <state_interface name="velocity"/>
+        </joint>
+        <joint name="arm_j5">
+          <command_interface name="position"/>
+          <state_interface name="position"/>
+          <state_interface name="velocity"/>
+        </joint>
+        <joint name="arm_j6">
+          <command_interface name="position"/>
+          <state_interface name="position"/>
+          <state_interface name="velocity"/>
+        </joint>
+      </xacro:if>
     </ros2_control>
   </xacro:macro>

File: rover/ros2_ws/src/mr2_rover_description/urdf/rover.urdf.xacro (robot description, xacro)
@@ -4,7 +4,9 @@
   <xacro:arg name="ros2_control_mode" default="gazebo"/>
   <xacro:arg name="ros2_control_config" default="$(find mr2_rover_description)/config/controllers/rover_controllers.yaml"/>
+  <xacro:arg name="enable_manipulator" default="true"/>
   <xacro:property name="ros2_control_mode_value" value="$(arg ros2_control_mode)"/>
   <xacro:property name="ros2_control_config_value" value="$(arg ros2_control_config)"/>
   <xacro:property name="can_iface_value" value="$(arg can_iface)"/>
+  <xacro:property name="enable_manipulator_value" value="$(arg enable_manipulator)"/>
   <xacro:property name="rover_mesh_prefix" value="file://$(find mr2_rover_description)/meshes/rover"/>
   <xacro:property name="rover_mesh_scale" value="0.01"/>
@@ -27,11 +29,13 @@
   <xacro:swerve_module prefix="rl" parent="left_rocker" xyz="-0.476931 0.0797 -0.18" direction="-1"/>
   <!-- Manipulator -->
-  <xacro:manipulator/>
+  <xacro:if value="${enable_manipulator_value}">
+    <xacro:manipulator/>
+  </xacro:if>
   <xacro:if value="${ros2_control_mode_value == 'gazebo'}">
     <xacro:rover_gazebo_sensors ros2_control_config="${ros2_control_config_value}"/>
-    <xacro:rover_gazebo_ros2_control name="GazeboSimSystem" ros2_control_config="${ros2_control_config_value}"/>
+    <xacro:rover_gazebo_ros2_control name="GazeboSimSystem" ros2_control_config="${ros2_control_config_value}" enable_manipulator="${enable_manipulator_value}"/>
   </xacro:if>
   <xacro:if value="${ros2_control_mode_value == 'real_hardware'}">
-    <xacro:rover_can_ros2_control name="RoverCanSystem" can_iface="${can_iface_value}"/>
+    <xacro:rover_can_ros2_control name="RoverCanSystem" can_iface="${can_iface_value}" enable_manipulator="${enable_manipulator_value}"/>
   </xacro:if>
 </robot>

Commit message: 2026. 02. 09 save (Jaeuk Kim)

File: rover/ros2_ws/src/mr2_rover_description/ros2_control/rover_can.ros2_control.xacro (robot description, xacro)
@@ -87,12 +87,12 @@
         <param name="joint_lower_limit">${arm_j1_lower_limit}</param>
         <param name="joint_upper_limit">${arm_j1_upper_limit}</param>
-        <param name="homing_plugin">mr2_can_hardware_interface/AbsoluteEncoderPolicy</param>
-        <param name="homing_device_can_iface">${can_iface}</param>
-        <param name="homing_offset">-4.70</param>
-        <param name="homing_split_angle">2.43</param>
-        <param name="homing_encoder_direction">1.0</param>
-        <param name="homing_device_can_iface">${can_iface}</param>
-        <param name="homing_device_can_id">201</param>
-        <param name="homing_device_ticks_per_rev">4096</param>
+        <!-- <param name="homing_plugin">mr2_can_hardware_interface/AbsoluteEncoderPolicy</param> -->
+        <!-- <param name="homing_device_can_iface">${can_iface}</param> -->
+        <!-- <param name="homing_offset">-4.70</param> -->
+        <!-- <param name="homing_split_angle">2.43</param> -->
+        <!-- <param name="homing_encoder_direction">1.0</param> -->
+        <!-- <param name="homing_device_can_iface">${can_iface}</param> -->
+        <!-- <param name="homing_device_can_id">201</param> -->
+        <!-- <param name="homing_device_ticks_per_rev">4096</param> -->
       </joint>
       <joint name="arm_j2">
@@ -107,13 +107,13 @@
         <param name="joint_lower_limit">${arm_j2_lower_limit}</param>
         <param name="joint_upper_limit">${arm_j2_upper_limit}</param>
-        <param name="homing_plugin">mr2_can_hardware_interface/LimitSwitchPolicy</param>
-        <param name="homing_position">-0.69</param>
-        <param name="homing_device_can_iface">${can_iface}</param>
-        <param name="homing_device_can_id">202</param>
-        <param name="homing_device_active_high">true</param>
-        <param name="homing_search_direction">negative</param>
-        <param name="homing_approach_speed">0.1</param>
-        <param name="homing_fine_speed">0.02</param>
-        <param name="homing_backoff_distance">0.05</param>
+        <!-- <param name="homing_plugin">mr2_can_hardware_interface/LimitSwitchPolicy</param> -->
+        <!-- <param name="homing_position">-0.69</param> -->
+        <!-- <param name="homing_device_can_iface">${can_iface}</param> -->
+        <!-- <param name="homing_device_can_id">202</param> -->
+        <!-- <param name="homing_device_active_high">true</param> -->
+        <!-- <param name="homing_search_direction">negative</param> -->
+        <!-- <param name="homing_approach_speed">0.1</param> -->
+        <!-- <param name="homing_fine_speed">0.02</param> -->
+        <!-- <param name="homing_backoff_distance">0.05</param> -->
       </joint>
       <joint name="arm_j3">
@@ -128,11 +128,11 @@
         <param name="joint_lower_limit">${arm_j3_lower_limit}</param>
         <param name="joint_upper_limit">${arm_j3_upper_limit}</param>
-        <param name="homing_plugin">mr2_can_hardware_interface/AbsoluteEncoderPolicy</param>
-        <param name="homing_offset">4.91</param>
-        <param name="homing_split_angle">3.4</param>
-        <param name="homing_encoder_direction">-1.0</param>
-        <param name="homing_device_can_iface">${can_iface}</param>
-        <param name="homing_device_can_id">203</param>
-        <param name="homing_device_ticks_per_rev">4096</param>
+        <!-- <param name="homing_plugin">mr2_can_hardware_interface/AbsoluteEncoderPolicy</param> -->
+        <!-- <param name="homing_offset">4.91</param> -->
+        <!-- <param name="homing_split_angle">3.4</param> -->
+        <!-- <param name="homing_encoder_direction">-1.0</param> -->
+        <!-- <param name="homing_device_can_iface">${can_iface}</param> -->
+        <!-- <param name="homing_device_can_id">203</param> -->
+        <!-- <param name="homing_device_ticks_per_rev">4096</param> -->
       </joint>
       <joint name="arm_j4">
@@ -147,13 +147,13 @@
         <param name="joint_lower_limit">${arm_j4_lower_limit}</param>
         <param name="joint_upper_limit">${arm_j4_upper_limit}</param>
-        <param name="homing_plugin">mr2_can_hardware_interface/LimitSwitchPolicy</param>
-        <param name="homing_position">-2.55</param>
-        <param name="homing_device_can_iface">${can_iface}</param>
-        <param name="homing_device_can_id">204</param>
-        <param name="homing_device_active_high">true</param>
-        <param name="homing_search_direction">negative</param>
-        <param name="homing_approach_speed">0.35</param>
-        <param name="homing_fine_speed">0.05</param>
-        <param name="homing_backoff_distance">0.12</param>
+        <!-- <param name="homing_plugin">mr2_can_hardware_interface/LimitSwitchPolicy</param> -->
+        <!-- <param name="homing_position">-2.55</param> -->
+        <!-- <param name="homing_device_can_iface">${can_iface}</param> -->
+        <!-- <param name="homing_device_can_id">204</param> -->
+        <!-- <param name="homing_device_active_high">true</param> -->
+        <!-- <param name="homing_search_direction">negative</param> -->
+        <!-- <param name="homing_approach_speed">0.35</param> -->
+        <!-- <param name="homing_fine_speed">0.05</param> -->
+        <!-- <param name="homing_backoff_distance">0.12</param> -->
       </joint>
       <joint name="arm_j5">
@@ -168,11 +168,11 @@
         <param name="joint_lower_limit">${arm_j5_lower_limit}</param>
         <param name="joint_upper_limit">${arm_j5_upper_limit}</param>
-        <param name="homing_plugin">mr2_can_hardware_interface/AbsoluteEncoderPolicy</param>
-        <param name="homing_offset">-2.46</param>
-        <param name="homing_split_angle">0.98</param>
-        <param name="homing_encoder_direction">1.0</param>
-        <param name="homing_device_can_iface">${can_iface}</param>
-        <param name="homing_device_can_id">205</param>
-        <param name="homing_device_ticks_per_rev">4096</param>
+        <!-- <param name="homing_plugin">mr2_can_hardware_interface/AbsoluteEncoderPolicy</param> -->
+        <!-- <param name="homing_offset">-2.46</param> -->
+        <!-- <param name="homing_split_angle">0.98</param> -->
+        <!-- <param name="homing_encoder_direction">1.0</param> -->
+        <!-- <param name="homing_device_can_iface">${can_iface}</param> -->
+        <!-- <param name="homing_device_can_id">205</param> -->
+        <!-- <param name="homing_device_ticks_per_rev">4096</param> -->
       </joint>
       <joint name="arm_j6">
@@ -187,13 +187,13 @@
         <param name="joint_lower_limit">${arm_j6_lower_limit}</param>
         <param name="joint_upper_limit">${arm_j6_upper_limit}</param>
-        <param name="homing_plugin">mr2_can_hardware_interface/LimitSwitchPolicy</param>
-        <param name="homing_device_can_id">206</param>
-        <param name="homing_device_can_iface">${can_iface}</param>
-        <param name="homing_position">-3.03</param>
-        <param name="homing_device_active_high">true</param>
-        <param name="homing_search_direction">negative</param>
-        <param name="homing_approach_speed">0.35</param>
-        <param name="homing_fine_speed">0.05</param>
-        <param name="homing_backoff_distance">0.12</param>
+        <!-- <param name="homing_plugin">mr2_can_hardware_interface/LimitSwitchPolicy</param> -->
+        <!-- <param name="homing_device_can_id">206</param> -->
+        <!-- <param name="homing_device_can_iface">${can_iface}</param> -->
+        <!-- <param name="homing_position">-3.03</param> -->
+        <!-- <param name="homing_device_active_high">true</param> -->
+        <!-- <param name="homing_search_direction">negative</param> -->
+        <!-- <param name="homing_approach_speed">0.35</param> -->
+        <!-- <param name="homing_fine_speed">0.05</param> -->
+        <!-- <param name="homing_backoff_distance">0.12</param> -->
       </joint>
       <!-- Gripper motor using steering-style centi-degree CAN protocol -->

File: rover/ros2_ws/src/mr2_rover_description/urdf/manipulator.xacro (robot description, xacro)
@@ -2,28 +2,28 @@
 <robot xmlns:xacro="http://www.ros.org/wiki/xacro">
   <!-- Joint limits (shared with ros2_control config) -->
-  <xacro:property name="arm_j1_lower_limit" value="-4"/>
-  <xacro:property name="arm_j1_upper_limit" value="4"/>
-  <!-- <xacro:property name="arm_j1_lower_limit" value="-100"/> -->
-  <!-- <xacro:property name="arm_j1_upper_limit" value="100"/> -->
-  <xacro:property name="arm_j2_lower_limit" value="-0.645"/>
-  <xacro:property name="arm_j2_upper_limit" value="1.57"/>
-  <!-- <xacro:property name="arm_j2_lower_limit" value="-100"/> -->
-  <!-- <xacro:property name="arm_j2_upper_limit" value="100"/> -->
-  <xacro:property name="arm_j3_lower_limit" value="-2"/>
-  <xacro:property name="arm_j3_upper_limit" value="-0.1"/>
-  <!-- <xacro:property name="arm_j3_lower_limit" value="-100"/> -->
-  <!-- <xacro:property name="arm_j3_upper_limit" value="100"/> -->
-  <xacro:property name="arm_j4_lower_limit" value="-3.5"/>
-  <xacro:property name="arm_j4_upper_limit" value="3.5"/>
-  <!-- <xacro:property name="arm_j4_lower_limit" value="-100"/> -->
-  <!-- <xacro:property name="arm_j4_upper_limit" value="100"/> -->
-  <xacro:property name="arm_j5_lower_limit" value="-0.12"/>
-  <xacro:property name="arm_j5_upper_limit" value="3.65"/>
-  <!-- <xacro:property name="arm_j5_lower_limit" value="-100"/> -->
-  <!-- <xacro:property name="arm_j5_upper_limit" value="100"/> -->
-  <xacro:property name="arm_j6_lower_limit" value="-4"/>
-  <xacro:property name="arm_j6_upper_limit" value="4"/>
-  <!-- <xacro:property name="arm_j6_lower_limit" value="-100"/> -->
-  <!-- <xacro:property name="arm_j6_upper_limit" value="100"/> -->
+  <!-- <xacro:property name="arm_j1_lower_limit" value="-4"/> -->
+  <!-- <xacro:property name="arm_j1_upper_limit" value="4"/> -->
+  <xacro:property name="arm_j1_lower_limit" value="-100"/>
+  <xacro:property name="arm_j1_upper_limit" value="100"/>
+  <!-- <xacro:property name="arm_j2_lower_limit" value="-0.645"/> -->
+  <!-- <xacro:property name="arm_j2_upper_limit" value="1.57"/> -->
+  <xacro:property name="arm_j2_lower_limit" value="-100"/>
+  <xacro:property name="arm_j2_upper_limit" value="100"/>
+  <!-- <xacro:property name="arm_j3_lower_limit" value="-2"/> -->
+  <!-- <xacro:property name="arm_j3_upper_limit" value="-0.1"/> -->
+  <xacro:property name="arm_j3_lower_limit" value="-100"/>
+  <xacro:property name="arm_j3_upper_limit" value="100"/>
+  <!-- <xacro:property name="arm_j4_lower_limit" value="-3.5"/> -->
+  <!-- <xacro:property name="arm_j4_upper_limit" value="3.5"/> -->
+  <xacro:property name="arm_j4_lower_limit" value="-100"/>
+  <xacro:property name="arm_j4_upper_limit" value="100"/>
+  <!-- <xacro:property name="arm_j5_lower_limit" value="-0.12"/> -->
+  <!-- <xacro:property name="arm_j5_upper_limit" value="3.65"/> -->
+  <xacro:property name="arm_j5_lower_limit" value="-100"/>
+  <xacro:property name="arm_j5_upper_limit" value="100"/>
+  <!-- <xacro:property name="arm_j6_lower_limit" value="-4"/> -->
+  <!-- <xacro:property name="arm_j6_upper_limit" value="4"/> -->
+  <xacro:property name="arm_j6_lower_limit" value="-100"/>
+  <xacro:property name="arm_j6_upper_limit" value="100"/>
   <!-- Shared shaded material for STL visuals (prevents unlit white appearance) -->
   <material name="ArmGrey">
