Commit message: fix urdf and add autonomous module

File: rover/ros2_ws/src/mr2_rover_description/ros2_control/rover_can.ros2_control.xacro (robot description, xacro)
@@ -1,6 +1,6 @@
 <?xml version="1.0"?>
 <robot xmlns:xacro="http://www.ros.org/wiki/xacro">n
-  <xacro:macro name="rover_can_ros2_control" params="name can_iface:=can0 enable_manipulator:=true">
-    <xacro:property name="enable_manipulator_value" value="${enable_manipulator}"/>
+  <xacro:macro name="rover_can_ros2_control" params="name can_iface:=can0 enable_manipulator_module:=true">
+    <xacro:property name="enable_manipulator_module_value" value="${enable_manipulator_module}"/>
     <ros2_control name="${name}" type="system">
       <hardware>
@@ -75,5 +75,5 @@
         <param name="can_iface">${can_iface}</param>
       </joint>
-      <xacro:if value="${enable_manipulator_value}">
+      <xacro:if value="${enable_manipulator_module_value}">
       <joint name="arm_j1">
         <command_interface name="position"/>
@@ -291,5 +291,5 @@
         </joint>
       </transmission>
-      <xacro:if value="${enable_manipulator_value}">
+      <xacro:if value="${enable_manipulator_module_value}">
       <transmission name="arm_j1_transmission">
         <plugin>transmission_interface/SimpleTransmission</plugin>

File: rover/ros2_ws/src/mr2_rover_description/ros2_control/rover_gazebo.ros2_control.xacro (robot description, xacro)
@@ -1,6 +1,6 @@
 <?xml version="1.0"?>
 <robot xmlns:xacro="http://www.ros.org/wiki/xacro">
-  <xacro:macro name="rover_gazebo_ros2_control" params="name ros2_control_config enable_manipulator:=true">
-    <xacro:property name="enable_manipulator_value" value="${enable_manipulator}"/>
+  <xacro:macro name="rover_gazebo_ros2_control" params="name ros2_control_config enable_manipulator_module:=true">
+    <xacro:property name="enable_manipulator_module_value" value="${enable_manipulator_module}"/>
     <ros2_control name="${name}" type="system">
       <hardware>
@@ -62,5 +62,5 @@
       </joint>
       <!-- Arm joint interfaces -->
-      <xacro:if value="${enable_manipulator_value}">
+      <xacro:if value="${enable_manipulator_module_value}">
         <joint name="arm_j1">
           <command_interface name="position"/>

File: rover/ros2_ws/src/mr2_rover_description/urdf/rover.urdf.xacro (robot description, xacro)
@@ -4,9 +4,11 @@
   <xacro:arg name="ros2_control_mode" default="gazebo"/>
   <xacro:arg name="ros2_control_config" default="$(find mr2_rover_description)/config/controllers/rover_controllers.yaml"/>
-  <xacro:arg name="enable_manipulator" default="true"/>
+  <xacro:arg name="enable_manipulator_module" default="true"/>
+  <xacro:arg name="enable_autonomous_module" default="true"/>
   <xacro:property name="ros2_control_mode_value" value="$(arg ros2_control_mode)"/>
   <xacro:property name="ros2_control_config_value" value="$(arg ros2_control_config)"/>
   <xacro:property name="can_iface_value" value="$(arg can_iface)"/>
-  <xacro:property name="enable_manipulator_value" value="$(arg enable_manipulator)"/>
+  <xacro:property name="enable_manipulator_module_value" value="$(arg enable_manipulator_module)"/>
+  <xacro:property name="enable_autonomous_module_value" value="$(arg enable_autonomous_module)"/>
   <xacro:property name="rover_mesh_prefix" value="file://$(find mr2_rover_description)/meshes/rover"/>
   <xacro:property name="rover_mesh_scale" value="0.01"/>
@@ -22,5 +24,5 @@
   <xacro:include filename="$(find mr2_rover_description)/urdf/rover_gazebo_sensors.xacro"/>
   <!-- Chassis -->
-  <xacro:rover_base/>
+  <xacro:rover_base enable_autonomous_module="${enable_autonomous_module_value}"/>
   <!-- Four modules -->
   <xacro:swerve_module prefix="fr" parent="right_rocker" xyz=" 0.476931 -0.0797 -0.18" direction="1"/>
@@ -29,13 +31,13 @@
   <xacro:swerve_module prefix="rl" parent="left_rocker" xyz="-0.476931 0.0797 -0.18" direction="-1"/>
   <!-- Manipulator -->
-  <xacro:if value="${enable_manipulator_value}">
+  <xacro:if value="${enable_manipulator_module_value}">
     <xacro:manipulator/>
   </xacro:if>
   <xacro:if value="${ros2_control_mode_value == 'gazebo'}">
-    <xacro:rover_gazebo_sensors ros2_control_config="${ros2_control_config_value}"/>
-    <xacro:rover_gazebo_ros2_control name="GazeboSimSystem" ros2_control_config="${ros2_control_config_value}" enable_manipulator="${enable_manipulator_value}"/>
+    <xacro:rover_gazebo_sensors ros2_control_config="${ros2_control_config_value}" enable_autonomous_module="${enable_autonomous_module_value}"/>
+    <xacro:rover_gazebo_ros2_control name="GazeboSimSystem" ros2_control_config="${ros2_control_config_value}" enable_manipulator_module="${enable_manipulator_module_value}"/>
   </xacro:if>
   <xacro:if value="${ros2_control_mode_value == 'real_hardware'}">
-    <xacro:rover_can_ros2_control name="RoverCanSystem" can_iface="${can_iface_value}" enable_manipulator="${enable_manipulator_value}"/>
+    <xacro:rover_can_ros2_control name="RoverCanSystem" can_iface="${can_iface_value}" enable_manipulator_module="${enable_manipulator_module_value}"/>
   </xacro:if>
 </robot>

File: rover/ros2_ws/src/mr2_rover_description/urdf/rover_base.xacro (robot description, xacro)
@@ -1,5 +1,6 @@
 <?xml version="1.0"?>
 <robot xmlns:xacro="http://www.ros.org/wiki/xacro">
-  <xacro:macro name="rover_base" params="length:=0.73 width:=0.491 height:=0.19 mass:=10 rocker_size:=0.1 rocker_mass:=0.5 joint_effort:=50 joint_vel:=2.0 joint_lim:=1.57 front_camera_pitch:=0.349066">
+  <xacro:macro name="rover_base" params="length:=0.73 width:=0.491 height:=0.19 mass:=10 rocker_size:=0.1 rocker_mass:=0.5 joint_effort:=50 joint_vel:=2.0 joint_lim:=1.57 front_camera_pitch:=0.349066 enable_autonomous_module:=true">
+    <xacro:property name="enable_autonomous_module_value" value="${enable_autonomous_module}"/>
     <!-- TODO: set as real dimension of the rover (#34) -->
     <link name="base_link"/>
@@ -11,8 +12,18 @@
       <visual>
         <geometry>
-	<box size="${length/2.0} ${width} ${height}"/>
+          <mesh filename="${rover_mesh_prefix}/base.obj"
+                scale="${rover_mesh_scale} ${rover_mesh_scale} ${rover_mesh_scale}"/>
         </geometry>
-        <origin xyz="${-length/4.0} 0 ${height/2.0}"/>
+        <origin xyz="0 0 0.05"/>
       </visual>
+      <xacro:if value="${enable_autonomous_module_value}">
+        <visual>
+          <geometry>
+            <mesh filename="${rover_mesh_prefix}/autonomous_module.obj"
+                  scale="${rover_mesh_scale} ${rover_mesh_scale} ${rover_mesh_scale}"/>
+          </geometry>
+          <origin xyz="0 0 0.05"/>
+        </visual>
+      </xacro:if>
       <collision>
         <geometry>
@@ -107,17 +118,19 @@
       <child link="rgbd_camera"/>
     </joint>
-    <link name="front_camera"/>
-    <joint name="base_to_front_camera" type="fixed">
-      <origin xyz="${length/2.0} 0 0.5" rpy="0 0 0"/>
-      <parent link="base_chassis"/>
-      <child link="front_camera"/>
-    </joint>
-    <!-- Optical frame for the front UVC camera (REP 103): x right, y down, z forward -->
-    <link name="front_camera_optical_frame"/>
-    <joint name="front_camera_to_optical" type="fixed">
-      <origin xyz="0 0 0" rpy="-1.57079632679 0 -1.57079632679"/>
-      <parent link="front_camera"/>
-      <child link="front_camera_optical_frame"/>
-    </joint>
+    <xacro:if value="${enable_autonomous_module_value}">
+      <link name="front_camera"/>
+      <joint name="base_to_front_camera" type="fixed">
+        <origin xyz="0.3476 0 0.438" rpy="0 0 0"/>
+        <parent link="base_chassis"/>
+        <child link="front_camera"/>
+      </joint>
+      <!-- Optical frame for the front UVC camera (REP 103): x right, y down, z forward -->
+      <link name="front_camera_optical_frame"/>
+      <joint name="front_camera_to_optical" type="fixed">
+        <origin xyz="0 0 0" rpy="-1.57079632679 0 -1.57079632679"/>
+        <parent link="front_camera"/>
+        <child link="front_camera_optical_frame"/>
+      </joint>
+    </xacro:if>
     <!-- IMU mounted at the top of the base box -->
     <link name="imu_link"/>

File: rover/ros2_ws/src/mr2_rover_description/urdf/rover_gazebo_sensors.xacro (robot description, xacro)
@@ -1,5 +1,6 @@
 <?xml version="1.0"?>
 <robot xmlns:xacro="http://www.ros.org/wiki/xacro">
-  <xacro:macro name="rover_gazebo_sensors" params="ros2_control_config">
+  <xacro:macro name="rover_gazebo_sensors" params="ros2_control_config enable_autonomous_module:=true">
+    <xacro:property name="enable_autonomous_module_value" value="${enable_autonomous_module}"/>
     <!-- ros2_control plugin that loads the TwistToCommands controller -->
     <gazebo>
@@ -81,57 +82,59 @@
       </sensor>
     </gazebo>
-    <gazebo reference="front_camera">
-      <sensor name="front_camera_sensor" type="rgbd_camera">
-        <update_rate>30</update_rate>
-        <always_on>1</always_on>
-        <visualize>true</visualize>
-        <topic>front_camera</topic>
-        <ignition_frame_id>front_camera_optical_frame</ignition_frame_id>
-        <camera>
-          <horizontal_fov>1.5184</horizontal_fov>
-          <lens>
-            <intrinsics>
-              <!-- fx = fy = width / ( 2 * tan (hfov / 2 ) ) -->
-              <fx>277.12735</fx>
-              <fy>277.12735</fy>
-              <!-- cx = ( width + 1 ) / 2 -->
-              <cx>160.5</cx>
-              <!-- cy = ( height + 1 ) / 2 -->
-              <cy>120.5</cy>
-              <s>0</s>
-            </intrinsics>
-          </lens>
-          <distortion>
-            <k1>0.0</k1>
-            <k2>0.0</k2>
-            <k3>0.0</k3>
-            <p1>0.0</p1>
-            <p2>0.0</p2>
-            <center>0.5 0.5</center>
-          </distortion>
-          <image>
-            <width>320</width>
-            <height>180</height>
-            <anti_aliasing>4</anti_aliasing>
-            <format>R8G8B8</format>
-          </image>
-          <clip>
-            <near>0.3</near>
-            <far>3.0</far>
-          </clip>
-          <depth_camera>
+    <xacro:if value="${enable_autonomous_module_value}">
+      <gazebo reference="front_camera">
+        <sensor name="front_camera_sensor" type="rgbd_camera">
+          <update_rate>30</update_rate>
+          <always_on>1</always_on>
+          <visualize>true</visualize>
+          <topic>front_camera</topic>
+          <ignition_frame_id>front_camera_optical_frame</ignition_frame_id>
+          <camera>
+            <horizontal_fov>1.5184</horizontal_fov>
+            <lens>
+              <intrinsics>
+                <!-- fx = fy = width / ( 2 * tan (hfov / 2 ) ) -->
+                <fx>277.12735</fx>
+                <fy>277.12735</fy>
+                <!-- cx = ( width + 1 ) / 2 -->
+                <cx>160.5</cx>
+                <!-- cy = ( height + 1 ) / 2 -->
+                <cy>120.5</cy>
+                <s>0</s>
+              </intrinsics>
+            </lens>
+            <distortion>
+              <k1>0.0</k1>
+              <k2>0.0</k2>
+              <k3>0.0</k3>
+              <p1>0.0</p1>
+              <p2>0.0</p2>
+              <center>0.5 0.5</center>
+            </distortion>
+            <image>
+              <width>320</width>
+              <height>180</height>
+              <anti_aliasing>4</anti_aliasing>
+              <format>R8G8B8</format>
+            </image>
             <clip>
               <near>0.3</near>
               <far>3.0</far>
             </clip>
-          </depth_camera>
-          <noise>
-            <type>gaussian</type>
-            <mean>0</mean>
-            <stddev>0.007</stddev>
-          </noise>
-        </camera>
-      </sensor>
-    </gazebo>
+            <depth_camera>
+              <clip>
+                <near>0.3</near>
+                <far>3.0</far>
+              </clip>
+            </depth_camera>
+            <noise>
+              <type>gaussian</type>
+              <mean>0</mean>
+              <stddev>0.007</stddev>
+            </noise>
+          </camera>
+        </sensor>
+      </gazebo>
+    </xacro:if>
     <gazebo reference="imu_link">
       <sensor name="imu_sensor" type="imu">

Commit message: Align NoFW actuator mapping and publish status

File: rover/ros2_ws/src/mr2_rover_description/ros2_control/rover_can.ros2_control.xacro (robot description, xacro)
@@ -12,41 +12,49 @@
         <param name="actuator">steering_fl</param>
         <param name="device_plugin">mr2_devices_output_actuator/OutputActuatorDevice</param>
+        <param name="node_id">3</param>
+        <param name="can_iface">${can_iface}</param>
+        <param name="command_channel">angle</param>
+        <param name="desired_profile">As5600</param>
+        <param name="expected_output_min_deg">-120.0</param>
+        <param name="expected_output_max_deg">120.0</param>
+        <param name="auto_arm">true</param>
+      </joint>
+      <joint name="fr_steering_joint">
+        <command_interface name="position"/>
+        <state_interface name="position"/>
+        <param name="actuator">steering_fr</param>
+        <param name="device_plugin">mr2_devices_output_actuator/OutputActuatorDevice</param>
+        <param name="node_id">1</param>
+        <param name="can_iface">${can_iface}</param>
+        <param name="command_channel">angle</param>
+        <param name="desired_profile">As5600</param>
+        <param name="expected_output_min_deg">-120.0</param>
+        <param name="expected_output_max_deg">120.0</param>
+        <param name="auto_arm">true</param>
+      </joint>
+      <joint name="rl_steering_joint">
+        <command_interface name="position"/>
+        <state_interface name="position"/>
+        <param name="actuator">steering_rl</param>
+        <param name="device_plugin">mr2_devices_output_actuator/OutputActuatorDevice</param>
+        <param name="node_id">4</param>
+        <param name="can_iface">${can_iface}</param>
+        <param name="command_channel">angle</param>
+        <param name="desired_profile">As5600</param>
+        <param name="expected_output_min_deg">-120.0</param>
+        <param name="expected_output_max_deg">120.0</param>
+        <param name="auto_arm">true</param>
+      </joint>
+      <joint name="rr_steering_joint">
+        <command_interface name="position"/>
+        <state_interface name="position"/>
+        <param name="actuator">steering_rr</param>
+        <param name="device_plugin">mr2_devices_output_actuator/OutputActuatorDevice</param>
         <param name="node_id">2</param>
         <param name="can_iface">${can_iface}</param>
         <param name="command_channel">angle</param>
         <param name="desired_profile">As5600</param>
-        <param name="auto_arm">true</param>
-      </joint>
-      <joint name="fr_steering_joint">
-        <command_interface name="position"/>
-        <state_interface name="position"/>
-        <param name="actuator">steering_fr</param>
-        <param name="device_plugin">mr2_devices_output_actuator/OutputActuatorDevice</param>
-        <param name="node_id">3</param>
-        <param name="can_iface">${can_iface}</param>
-        <param name="command_channel">angle</param>
-        <param name="desired_profile">As5600</param>
-        <param name="auto_arm">true</param>
-      </joint>
-      <joint name="rl_steering_joint">
-        <command_interface name="position"/>
-        <state_interface name="position"/>
-        <param name="actuator">steering_rl</param>
-        <param name="device_plugin">mr2_devices_output_actuator/OutputActuatorDevice</param>
-        <param name="node_id">4</param>
-        <param name="can_iface">${can_iface}</param>
-        <param name="command_channel">angle</param>
-        <param name="desired_profile">As5600</param>
-        <param name="auto_arm">true</param>
-      </joint>
-      <joint name="rr_steering_joint">
-        <command_interface name="position"/>
-        <state_interface name="position"/>
-        <param name="actuator">steering_rr</param>
-        <param name="device_plugin">mr2_devices_output_actuator/OutputActuatorDevice</param>
-        <param name="node_id">1</param>
-        <param name="can_iface">${can_iface}</param>
-        <param name="command_channel">angle</param>
-        <param name="desired_profile">As5600</param>
+        <param name="expected_output_min_deg">-120.0</param>
+        <param name="expected_output_max_deg">120.0</param>
         <param name="auto_arm">true</param>
       </joint>
@@ -57,5 +65,5 @@
         <param name="actuator">drive_fl</param>
         <param name="device_plugin">mr2_devices_output_actuator/OutputActuatorDevice</param>
-        <param name="node_id">18</param>
+        <param name="node_id">7</param>
         <param name="can_iface">${can_iface}</param>
         <param name="command_channel">velocity</param>
@@ -69,5 +77,5 @@
         <param name="actuator">drive_fr</param>
         <param name="device_plugin">mr2_devices_output_actuator/OutputActuatorDevice</param>
-        <param name="node_id">19</param>
+        <param name="node_id">5</param>
         <param name="can_iface">${can_iface}</param>
         <param name="command_channel">velocity</param>
@@ -81,5 +89,5 @@
         <param name="actuator">drive_rl</param>
         <param name="device_plugin">mr2_devices_output_actuator/OutputActuatorDevice</param>
-        <param name="node_id">20</param>
+        <param name="node_id">8</param>
         <param name="can_iface">${can_iface}</param>
         <param name="command_channel">velocity</param>
@@ -93,5 +101,5 @@
         <param name="actuator">drive_rr</param>
         <param name="device_plugin">mr2_devices_output_actuator/OutputActuatorDevice</param>
-        <param name="node_id">17</param>
+        <param name="node_id">6</param>
         <param name="can_iface">${can_iface}</param>
         <param name="command_channel">velocity</param>
@@ -183,5 +191,5 @@
         <param name="actuator">gripper_motor</param>
         <param name="device_plugin">mr2_devices_output_actuator/OutputActuatorDevice</param>
-        <param name="node_id">7</param>
+        <param name="node_id">9</param>
         <param name="can_iface">${can_iface}</param>
         <param name="command_channel">angle</param>

Commit message: Fix MoveIt passive and gripper joints

File: rover/ros2_ws/src/mr2_rover_description/ros2_control/rover_can.ros2_control.xacro (robot description, xacro)
@@ -196,6 +196,6 @@
         <param name="desired_profile">DirectInput</param>
         <param name="require_limits_status">false</param>
-        <param name="joint_lower_limit">0.0</param>
-        <param name="joint_upper_limit">1.3089969390</param>
+        <param name="joint_lower_limit">${arm_gripper_lower_limit}</param>
+        <param name="joint_upper_limit">${arm_gripper_upper_limit}</param>
         <param name="auto_arm">true</param>
       </joint>

File: rover/ros2_ws/src/mr2_rover_description/urdf/manipulator.xacro (robot description, xacro)
@@ -26,4 +26,6 @@
   <!-- <xacro:property name="arm_j6_lower_limit" value="-100"/> -->
   <!-- <xacro:property name="arm_j6_upper_limit" value="100"/> -->
+  <xacro:property name="arm_gripper_lower_limit" value="0.0"/>
+  <xacro:property name="arm_gripper_upper_limit" value="1.3089969390"/>
   <!-- Shared shaded material for STL visuals (prevents unlit white appearance) -->
   <material name="ArmGrey">
@@ -201,4 +203,26 @@
       <origin xyz="0.215 0 0" rpy="0 0 0"/>
     </joint>
+    <link name="gripper_link">
+      <visual>
+        <geometry>
+          <box size="0.08 0.04 0.04"/>
+        </geometry>
+        <origin xyz="0.04 0 0" rpy="0 0 0"/>
+        <material name="ArmGrey"/>
+      </visual>
+      <collision>
+        <geometry>
+          <box size="0.08 0.04 0.04"/>
+        </geometry>
+        <origin xyz="0.04 0 0" rpy="0 0 0"/>
+      </collision>
+    </link>
+    <joint name="arm_gripper" type="revolute">
+      <parent link="eef_link"/>
+      <child link="gripper_link"/>
+      <origin xyz="0 0 0" rpy="0 0 0"/>
+      <axis xyz="0 0 1"/>
+      <limit lower="${arm_gripper_lower_limit}" upper="${arm_gripper_upper_limit}" effort="20" velocity="2.0"/>
+    </joint>
   </xacro:macro>
 </robot>
